File: jl142/jl142.kicad_pcb (KiCad board)
At the start: 2 copper layers, 302.1 x 127 mm, 86 parts, among them SW12 SWITCH_PUSH, SW13 SWITCH_PUSH, SW14 SWITCH_PUSH, SW17 SWITCH_PUSH, SW18 SWITCH_PUSH, SW19 SWITCH_PUSH, SW2 SWITCH_PUSH, SW20 SWITCH_PUSH, SW22 SWITCH_PUSH, SW23 SWITCH_PUSH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

Commit message: Moved libraries around.
Parts:
- U1: value Arduino Pro Micro -> ARDUINO_PRO_MICRO
