File: jl142/jl142.kicad_sch (KiCad schematic)
At the start: 86 parts, among them SW12 SWITCH_PUSH, SW13 SWITCH_PUSH, SW14 SWITCH_PUSH, SW17 SWITCH_PUSH, SW18 SWITCH_PUSH, SW19 SWITCH_PUSH, SW2 SWITCH_PUSH, SW20 SWITCH_PUSH, SW22 SWITCH_PUSH, SW23 SWITCH_PUSH, SW24 SWITCH_PUSH, SW25 SWITCH_PUSH, SW27 SWITCH_PUSH, SW28 SWITCH_PUSH, SW29 SWITCH_PUSH, SW3 SWITCH_PUSH, SW30 SWITCH_PUSH, SW34 SWITCH_PUSH, SW35 SWITCH_PUSH, SW36 SWITCH_PUSH, SW37 SWITCH_PUSH, SW39 SWITCH_PUSH, SW4 SWITCH_PUSH, SW40 SWITCH_PUSH, SW41 SWITCH_PUSH, SW42 SWITCH_PUSH, SW44 SWITCH_PUSH, SW45 SWITCH_PUSH, SW46 SWITCH_PUSH, SW47 SWITCH_PUSH, SW49 SWITCH_PUSH, SW50 SWITCH_PUSH, SW51 SWITCH_PUSH, SW54 SWITCH_PUSH, SW55 SWITCH_PUSH, SW56 SWITCH_PUSH, SW59 SWITCH_PUSH, SW60 SWITCH_PUSH, SW61 SWITCH_PUSH, SW7 SWITCH_PUSH, SW8 SWITCH_PUSH, SW9 SWITCH_PUSH, U1 ARDUINO_PRO_MICRO

Commit message: Renamed the kicad project to jl142.
Parts:
- D12, D13, D14, D17, D18, D19, D2, D20, D22, D23, D24, D25, D27, D28, D29, D3, D30, D34, D35, D36, D37, D39, D4, D40, D41, D42, D44, D45, D46, D47, D49, D50, D51, D54, D55, D56, D59, D60, D61, D7, D8, D9: symbol Diode:1N4148 -> symbols:1N4148
- SW-RST1, SW12, SW13, SW14, SW17, SW18, SW19, SW2, SW20, SW22, SW23, SW24, SW25, SW27, SW28, SW29, SW3, SW30, SW34, SW35, SW36, SW37, SW39, SW4, SW40, SW41, SW42, SW44, SW45, SW46, SW47, SW49, SW50, SW51, SW54, SW55, SW56, SW59, SW60, SW61, SW7, SW8, SW9: symbol Atreus62-rescue:SWITCH_PUSH -> symbols:SWITCH_PUSH
- U1: symbol Atreus62-rescue:ARDUINO_PRO_MICRO -> symbols:ARDUINO_PRO_MICRO

Commit message: Moved libraries around.
Parts:
- D12, D13, D14, D17, D18, D19, D2, D20, D22, D23, D24, D25, D27, D28, D29, D3, D30, D34, D35, D36, D37, D39, D4, D40, D41, D42, D44, D45, D46, D47, D49, D50, D51, D54, D55, D56, D59, D60, D61, D7, D8, D9: symbol symbols:1N4148 -> Diode:1N4148
