File: jl142/jl142_pcb/jl142_pcb.kicad_pcb (KiCad board)
At the start: 2 copper layers, 286.2 x 114.7 mm, 44 parts, among them SW12 SWITCH_PUSH, SW13 SWITCH_PUSH, SW14 SWITCH_PUSH, SW17 SWITCH_PUSH, SW18 SWITCH_PUSH, SW19 SWITCH_PUSH, SW2 SWITCH_PUSH, SW20 SWITCH_PUSH, SW22 SWITCH_PUSH, SW23 SWITCH_PUSH, SW24 SWITCH_PUSH, SW25 SWITCH_PUSH, SW27 SWITCH_PUSH, SW28 SWITCH_PUSH, SW29 SWITCH_PUSH, SW3 SWITCH_PUSH, SW30 SWITCH_PUSH, SW34 SWITCH_PUSH, SW35 SWITCH_PUSH, SW36 SWITCH_PUSH, SW37 SWITCH_PUSH, SW39 SWITCH_PUSH, SW4 SWITCH_PUSH, SW40 SWITCH_PUSH, SW41 SWITCH_PUSH, SW42 SWITCH_PUSH, SW44 SWITCH_PUSH, SW45 SWITCH_PUSH, SW46 SWITCH_PUSH, SW47 SWITCH_PUSH, SW49 SWITCH_PUSH, SW50 SWITCH_PUSH, SW51 SWITCH_PUSH, SW54 SWITCH_PUSH, SW55 SWITCH_PUSH, SW56 SWITCH_PUSH, SW59 SWITCH_PUSH, SW60 SWITCH_PUSH, SW61 SWITCH_PUSH, SW7 SWITCH_PUSH, SW8 SWITCH_PUSH, SW9 SWITCH_PUSH, U1 Arduino Pro Micro

Commit message: Changed the pro micro symbol.
Parts:
- removed SW2, SW3, SW4, SW59, SW60, SW61: SWITCH_PUSH, footprints:kailh_choc_with_diode
- moved SW37 27.4 mm to (170.5, 137.6)
- moved SW22 27.4 mm to (95.6, 69.7)
- moved SW19 27.4 mm to (66.2, 87.5)
- moved SW9 27.4 mm to (23.6, 88.7)
- moved SW7 27.4 mm to (39.7, 54.1)
- moved SW-RST1 27.4 mm to (138.2, 110.6)
- moved SW44 27.4 mm to (194.1, 53.0)
- moved SW46 27.4 mm to (210.2, 87.5)
- moved SW55 27.4 mm to (244.8, 71.4)
- moved SW24 27.4 mm to (79.5, 104.2)
- moved SW56 27.4 mm to (252.8, 88.7)
- moved SW45 27.4 mm to (202.2, 70.3)
- moved SW17 27.4 mm to (82.3, 53.0)
- moved SW18 27.4 mm to (74.2, 70.3)
- moved SW49 27.4 mm to (214.6, 51.8)
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Routing:
- net /COL0: track 39.5 -> 0.00 mm
- net /COL11: track 39.5 -> 0.00 mm
- net /ROW2: track 214.1 -> 176.0 mm
- net /ROW3: track 214.2 -> 176.1 mm
- net /ROW1: track 214.2 -> 176.1 mm
- net Net-(SW61-A): track 19.3 -> 0.00 mm
- net Net-(SW4-A): track 19.3 -> 0.00 mm
- net Net-(SW2-A): track 19.3 -> 0.00 mm
- net Net-(SW3-A): track 19.3 -> 0.00 mm
- net Net-(SW60-A): track 19.3 -> 0.00 mm
- net Net-(SW59-A): track 19.3 -> 0.00 mm
- net /COL5: track 71.7 -> 74.1 mm
Other:
- board size 286.2 x 114.7 mm -> 251.8 x 108.2 mm

Commit message: Routed rev2 of jl142.
Parts:
- added D1: IR204A, LED_THT:LED_D3.0mm_IRBlack, F.Cu at (134.0, 117.2)
- added D2: IR204A, LED_THT:LED_D3.0mm_IRBlack, F.Cu at (140.0, 117.2)
- added D3: IR204A, LED_THT:LED_D3.0mm_IRBlack, F.Cu at (146.0, 117.2)
- added R1: 330, Resistor_THT:R_Axial_DIN0207_L6.3mm_D2.5mm_P7.62mm_Horizontal, B.Cu at (136.0, 107.0)
- added R2: 330, Resistor_THT:R_Axial_DIN0207_L6.3mm_D2.5mm_P7.62mm_Horizontal, B.Cu at (140.0, 107.0)
- added R3: 330, Resistor_THT:R_Axial_DIN0207_L6.3mm_D2.5mm_P7.62mm_Horizontal, B.Cu at (144.0, 107.0)
- added REF**: MountingHole_4mm, MountingHole:MountingHole_4mm, F.Cu at (103.1, 123.4)
- added REF**: MountingHole_4mm, MountingHole:MountingHole_4mm, F.Cu at (176.9, 123.4)
- added REF**: MountingHole_4mm, MountingHole:MountingHole_4mm, F.Cu at (246.0, 91.2)
- added REF**: MountingHole_4mm, MountingHole:MountingHole_4mm, F.Cu at (101.9, 80.8)
- added REF**: MountingHole_4mm, MountingHole:MountingHole_4mm, F.Cu at (76.6, 90.0)
- added REF**: MountingHole_4mm, MountingHole:MountingHole_4mm, F.Cu at (225.8, 48.0)
- added REF**: MountingHole_4mm, MountingHole:MountingHole_4mm, F.Cu at (178.1, 80.8)
- added REF**: MountingHole_4mm, MountingHole:MountingHole_4mm, F.Cu at (54.2, 48.0)
- added REF**: MountingHole_4mm, MountingHole:MountingHole_4mm, F.Cu at (203.4, 90.0)
- added REF**: MountingHole_4mm, MountingHole:MountingHole_4mm, F.Cu at (34.0, 91.2)
- SW12, SW13, SW14, SW17, SW18, SW19, SW20, SW22, SW23, SW24, SW25, SW27, SW28, SW29, SW30, SW34, SW35, SW36, SW37, SW39, SW40, SW41, SW42, SW44, SW45, SW46, SW47, SW49, SW50, SW51, SW54, SW55, SW56, SW7, SW8, SW9: footprint footprints:kailh_choc_with_diode -> footprints:cherry_hotswap_with_diode
- U1: value Arduino Pro Micro -> ARDUINO_PRO_MICRO
- moved U1 3.91 mm to (140.0, 93.2)
- moved SW19 2.33 mm to (68.0, 86.0), turned to -25 degrees
- moved SW42 2.33 mm to (189.6, 128.0), turned to 25 degrees
- moved SW55 2.33 mm to (246.5, 69.9), turned to 25 degrees
- moved SW7 2.33 mm to (41.5, 52.6), turned to -25 degrees
- moved SW18 2.33 mm to (76.0, 68.8), turned to -25 degrees
- moved SW51 2.33 mm to (232.5, 84.9), turned to 25 degrees
- moved SW37 2.33 mm to (172.3, 136.1), turned to 25 degrees
- moved SW36 2.33 mm to (181.5, 110.7), turned to 25 degrees
- moved SW27 2.33 mm to (114.6, 76.2), turned to -25 degrees
- moved SW12 2.33 mm to (63.6, 50.3), turned to -25 degrees
- moved SW23 2.33 mm to (89.3, 85.4), turned to -25 degrees
- moved SW9 2.33 mm to (25.4, 87.2), turned to -25 degrees
- moved SW24 2.33 mm to (81.2, 102.7), turned to -25 degrees
- moved SW47 2.33 mm to (206.8, 120.0), turned to 25 degrees
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- renumbered SW-RST1 to RST1
Connections:
- RST1 pad 1: GND -> Net-(U1-RST)
- RST1 pad 2: Net-(U1-RST) -> GND
- U1 pad 10: /COL5 -> /COL6
- U1 pad 15: /COL6 -> /COL5
- U1 pad 16: /COL7 -> /COL4
- U1 pad 17: /COL8 -> /COL3
- U1 pad 18: /COL9 -> /COL2
- U1 pad 19: /COL10 -> /COL1
- U1 pad 2: unconnected-(U1-RX-Pad2) -> /LED2
- U1 pad 20: /COL11 -> /LED1
- U1 pad 5: /COL0 -> /LED3
- U1 pad 6: /COL1 -> /COL10
- U1 pad 7: /COL2 -> /COL9
- U1 pad 8: /COL3 -> /COL8
- U1 pad 9: /COL4 -> /COL7
Routing:
- net /COL10: track 39.5 -> 157.3 mm
- net /COL1: track 39.5 -> 151.9 mm
- net /ROW3: track 176.1 -> 281.6 mm
- net /ROW0: track 76.2 -> 174.7 mm
- net /ROW1: track 176.1 -> 271.7 mm
- net /COL9: track 39.5 -> 134.5 mm
- net /ROW2: track 176.0 -> 266.5 mm
- net /COL2: track 39.5 -> 122.7 mm
- net /COL8: track 75.9 -> 148.1 mm
- net /COL3: track 76.3 -> 139.5 mm
- net /COL7: track 68.8 -> 120.8 mm
- net /COL4: track 69.4 -> 115.3 mm
- net /COL6: track 68.8 -> 101.3 mm
- net Net-(U1-RST): track 0.00 -> 29.5 mm
- net /COL5: track 74.1 -> 97.5 mm
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- added copper zone on F.Cu, net GND
Other:
- board size 251.8 x 108.2 mm -> 253.1 x 110.2 mm
- board text removed: "Rev 2"
