File: kfs/kfs_pcb/kfs_pcb.kicad_sch (KiCad schematic)
At the start: 66 parts, among them SW1 SWITCH, SW10 SWITCH, SW11 SWITCH, SW12 SWITCH, SW13 SWITCH, SW14 SWITCH, SW15 SWITCH, SW16 SWITCH, SW17 SWITCH, SW18 SWITCH, SW19 SWITCH, SW2 SWITCH, SW20 SWITCH, SW21 SWITCH, SW22 SWITCH, SW23 SWITCH, SW24 SWITCH, SW25 SWITCH, SW26 SWITCH, SW27 SWITCH, SW28 SWITCH, SW29 SWITCH, SW3 SWITCH, SW30 SWITCH, SW31 SWITCH, SW32 SWITCH, SW33 SWITCH, SW34 SWITCH, SW35 SWITCH, SW36 SWITCH, SW37 SWITCH, SW38 SWITCH, SW39 SWITCH, SW4 SWITCH, SW41 SWITCH, SW42 SWITCH, SW43 SWITCH, SW44 SWITCH, SW45 SWITCH, SW46 SWITCH, SW47 SWITCH, SW48 SWITCH, SW49 SWITCH, SW5 SWITCH, SW50 SWITCH, SW51 SWITCH, SW52 SWITCH, SW53 SWITCH, SW54 SWITCH, SW55 SWITCH, SW56 SWITCH, SW57 SWITCH, SW58 SWITCH, SW59 SWITCH, SW6 SWITCH, SW60 SWITCH, SW61 SWITCH, SW62 SWITCH, SW63 SWITCH, SW64 SWITCH, SW65 SWITCH, SW7 SWITCH, SW8 SWITCH, SW9 SWITCH, U1 ARDUINO_PRO_MICRO

Commit message: Updates to kfs.
Parts:
- added H0, H1, H2, H3, H4, H5, H6: MountingHole_Pad, MountingHole:MountingHole_2.2mm_M2_ISO7380_Pad, symbol Mechanical:MountingHole_Pad
- added H10, H11, H12, H7, H8, H9: MountingHole, MountingHole:MountingHole_3.5mm, symbol Mechanical:MountingHole
- SW19: renamed from SW20; footprint footprints:cherry_hotswap_with_diode -> footprints:cherry_hotswap_with_diode_2u
- SW43: renamed from SW45; footprint footprints:cherry_hotswap_with_diode -> footprints:cherry_hotswap_with_diode_2u
- renumbered RST1 to RST0, SW1 to SW0, SW2 to SW1, SW11 to SW10, SW12 to SW11, SW13 to SW12, SW14 to SW13, SW15 to SW14, SW16 to SW15, SW17 to SW16, SW18 to SW17, SW19 to SW18, SW3 to SW2, SW21 to SW20, SW22 to SW21, SW23 to SW22, SW24 to SW23, SW25 to SW24, SW26 to SW25, SW27 to SW26, SW28 to SW27, SW29 to SW28, SW30 to SW29, SW4 to SW3, SW31 to SW30, SW32 to SW31, SW33 to SW32, SW34 to SW33, SW35 to SW34, SW36 to SW35, SW37 to SW36, SW38 to SW37, SW39 to SW38, SW41 to SW39, SW5 to SW4, SW42 to SW40, SW43 to SW41, SW44 to SW42, SW46 to SW44, SW47 to SW45, SW48 to SW46, SW49 to SW47, SW50 to SW48, SW51 to SW49, SW6 to SW5, SW52 to SW50, SW53 to SW51, SW54 to SW52, SW55 to SW53, SW56 to SW54, SW57 to SW55, SW58 to SW56, SW59 to SW57, SW60 to SW58, SW61 to SW59, SW7 to SW6, SW62 to SW60, SW63 to SW61, SW64 to SW62, SW65 to SW63, SW8 to SW7, SW9 to SW8, SW10 to SW9, U1 to U0
Connections:
- net GND: now also H0.1, H1.1, H2.1, H3.1, H4.1, H5.1, H6.1
