File: kfs/kfs_pcb/kfs_pcb.kicad_pcb (KiCad board)
At the start: 2 copper layers, 266.7 x 95.2 mm, 75 parts, among them SW1 SWITCH, SW10 SWITCH, SW11 SWITCH, SW12 SWITCH, SW13 SWITCH, SW14 SWITCH, SW15 SWITCH, SW16 SWITCH, SW17 SWITCH, SW18 SWITCH, SW19 SWITCH, SW2 SWITCH, SW20 SWITCH, SW21 SWITCH, SW22 SWITCH, SW23 SWITCH, SW24 SWITCH, SW25 SWITCH, SW26 SWITCH, SW27 SWITCH, SW28 SWITCH, SW29 SWITCH, SW3 SWITCH, SW30 SWITCH, SW31 SWITCH, SW32 SWITCH, SW33 SWITCH, SW34 SWITCH, SW35 SWITCH, SW36 SWITCH, SW37 SWITCH, SW38 SWITCH, SW39 SWITCH, SW4 SWITCH, SW41 SWITCH, SW42 SWITCH, SW43 SWITCH, SW44 SWITCH, SW45 SWITCH, SW46 SWITCH, SW47 SWITCH, SW48 SWITCH, SW49 SWITCH, SW5 SWITCH, SW50 SWITCH, SW51 SWITCH, SW52 SWITCH, SW53 SWITCH, SW54 SWITCH, SW55 SWITCH, SW56 SWITCH, SW57 SWITCH, SW58 SWITCH, SW59 SWITCH, SW6 SWITCH, SW60 SWITCH, SW61 SWITCH, SW62 SWITCH, SW63 SWITCH, SW64 SWITCH, SW65 SWITCH, SW7 SWITCH, SW8 SWITCH, SW9 SWITCH, U1 ARDUINO_PRO_MICRO

Commit message: Updates to kfs.
Parts:
- removed REF** (x9): MountingHole_3.5mm, MountingHole:MountingHole_3.5mm
- added H0: MountingHole_Pad, MountingHole:MountingHole_2.2mm_M2_ISO7380_Pad, F.Cu at (114.3, 47.6)
- added H1: MountingHole_Pad, MountingHole:MountingHole_2.2mm_M2_ISO7380_Pad, F.Cu at (114.3, 104.8)
- added H10: MountingHole, MountingHole:MountingHole_3.5mm, F.Cu at (266.7, 104.8)
- added H11: MountingHole, MountingHole:MountingHole_3.5mm, F.Cu at (156.4, 32.6)
- added H12: MountingHole, MountingHole:MountingHole_3.5mm, F.Cu at (129.3, 32.6)
- added H2: MountingHole_Pad, MountingHole:MountingHole_2.2mm_M2_ISO7380_Pad, F.Cu at (190.5, 47.6)
- added H3: MountingHole_Pad, MountingHole:MountingHole_2.2mm_M2_ISO7380_Pad, F.Cu at (209.6, 104.8)
- added H4: MountingHole_Pad, MountingHole:MountingHole_2.2mm_M2_ISO7380_Pad, F.Cu at (76.2, 66.7)
- added H5: MountingHole_Pad, MountingHole:MountingHole_2.2mm_M2_ISO7380_Pad, F.Cu at (152.4, 85.7)
- added H6: MountingHole_Pad, MountingHole:MountingHole_2.2mm_M2_ISO7380_Pad, F.Cu at (228.6, 66.7)
- added H7: MountingHole, MountingHole:MountingHole_3.5mm, F.Cu at (38.1, 47.6)
- added H8: MountingHole, MountingHole:MountingHole_3.5mm, F.Cu at (38.1, 104.8)
- added H9: MountingHole, MountingHole:MountingHole_3.5mm, F.Cu at (266.7, 47.6)
- SW19: renamed from SW20; footprint footprints:cherry_hotswap_with_diode -> footprints:cherry_hotswap_with_diode_2u
- SW43: renamed from SW45; footprint footprints:cherry_hotswap_with_diode -> footprints:cherry_hotswap_with_diode_2u
- moved U0 4.51 mm to (142.9, 50.1)
- renumbered RST1 to RST0, SW1 to SW0, SW2 to SW1, SW11 to SW10, SW12 to SW11, SW13 to SW12, SW14 to SW13, SW15 to SW14, SW16 to SW15, SW17 to SW16, SW18 to SW17, SW19 to SW18, SW3 to SW2, SW21 to SW20, SW22 to SW21, SW23 to SW22, SW24 to SW23, SW25 to SW24, SW26 to SW25, SW27 to SW26, SW28 to SW27, SW29 to SW28, SW30 to SW29, SW4 to SW3, SW31 to SW30, SW32 to SW31, SW33 to SW32, SW34 to SW33, SW35 to SW34, SW36 to SW35, SW37 to SW36, SW38 to SW37, SW39 to SW38, SW41 to SW39, SW5 to SW4, SW42 to SW40, SW43 to SW41, SW44 to SW42, SW46 to SW44, SW47 to SW45, SW48 to SW46, SW49 to SW47, SW50 to SW48, SW51 to SW49, SW6 to SW5, SW52 to SW50, SW53 to SW51, SW54 to SW52, SW55 to SW53, SW56 to SW54, SW57 to SW55, SW58 to SW56, SW59 to SW57, SW60 to SW58, SW61 to SW59, SW7 to SW6, SW62 to SW60, SW63 to SW61, SW64 to SW62, SW65 to SW63, SW8 to SW7, SW9 to SW8, SW10 to SW9, U1 to U0
Routing:
- net /ROW2: track 329.8 -> 311.9 mm
- net /ROW1: track 323.7 -> 314.7 mm
- net /ROW3: track 303.7 -> 296.2 mm
- net /ROW4: track 298.7 -> 292.1 mm
- net /COL12: track 214.0 -> 218.6 mm
- net /ROW0: track 316.7 -> 312.2 mm
- net /COL7: track 96.6 -> 100.0 mm
- net /COL4: track 139.2 -> 141.1 mm
- net /COL5: track 89.5 -> 87.6 mm
- net /COL0: track 182.6 -> 184.4 mm
- net /COL3: track 130.9 -> 132.8 mm
- net /COL1: track 164.2 -> 166.1 mm
- net /COL6: track 97.1 -> 95.2 mm
- net /COL9: track 153.5 -> 155.3 mm
- net /COL8: track 138.5 -> 140.4 mm
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- added copper zone on B.Cu, net GND

Commit message: Many updates to kfs. Now low profile.
Parts:
- removed H1: MountingHole_Pad, MountingHole:MountingHole_2.2mm_M2_ISO7380_Pad
- removed H11, H12: MountingHole, MountingHole:MountingHole_3.5mm
- H0, H2, H3, H4, H5, H6: value MountingHole_Pad -> MountingHole; footprint MountingHole:MountingHole_2.2mm_M2_ISO7380_Pad -> MountingHole:MountingHole_3.5mm
- RST0: moved to B.Cu
- SW0, SW1, SW10, SW11, SW12, SW13, SW14, SW15, SW16, SW17, SW18, SW2, SW20, SW21, SW22, SW23, SW24, SW25, SW26, SW27, SW28, SW29, SW3, SW30, SW31, SW32, SW33, SW34, SW35, SW36, SW37, SW38, SW39, SW4, SW40, SW41, SW42, SW44, SW45, SW46, SW47, SW48, SW49, SW5, SW50, SW51, SW52, SW53, SW54, SW55, SW56, SW57, SW58, SW59, SW6, SW60, SW61, SW62, SW63, SW7, SW8, SW9: footprint footprints:cherry_hotswap_with_diode -> footprints:kailh_choc_with_diode
- SW19, SW43: footprint footprints:cherry_hotswap_with_diode_2u -> footprints:kailh_choc_with_diode
- U0: value ARDUINO_PRO_MICRO -> Arduino Pro Micro
- moved H6 156.8 mm to (72.0, 59.5)
- moved H2 54.0 mm to (162.0, 93.5)
- moved H0 48.0 mm to (162.0, 42.5)
- moved H5 45.1 mm to (108.0, 93.5)
- moved H4 39.9 mm to (108.0, 42.5)
- moved H3 29.0 mm to (216.0, 76.5)
- moved SW63 27.2 mm to (252.0, 102.0)
- moved H9 26.6 mm to (252.0, 25.5)
- moved SW58 26.2 mm to (234.0, 102.0)
- moved SW53 25.3 mm to (216.0, 102.0)
- moved SW48 24.4 mm to (198.0, 102.0)
- moved H7 22.2 mm to (36.0, 25.5)
- moved SW43 19.4 mm to (175.5, 102.0)
- moved SW62 18.4 mm to (261.0, 85.0)
- moved SW57 17.5 mm to (243.0, 85.0)
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Connections:
- SW0 pad 1: /ROW4 -> /COL0
- SW0 pad 2: unconnected-(SW0-A-Pad2) -> Net-(SW0-A)
- SW0 pad 3: /COL0 -> /ROW4
- SW1 pad 1: /ROW3 -> /COL0
- SW1 pad 2: unconnected-(SW1-A-Pad2) -> Net-(SW1-A)
- SW1 pad 3: /COL0 -> /ROW3
- SW10 pad 1: /ROW4 -> /COL2
- SW10 pad 2: unconnected-(SW10-A-Pad2) -> Net-(SW10-A)
- SW10 pad 3: /COL2 -> /ROW4
- SW11 pad 1: /ROW3 -> /COL2
- SW11 pad 2: unconnected-(SW11-A-Pad2) -> Net-(SW11-A)
- SW11 pad 3: /COL2 -> /ROW3
- SW12 pad 1: /ROW2 -> /COL2
- SW12 pad 2: unconnected-(SW12-A-Pad2) -> Net-(SW12-A)
- SW12 pad 3: /COL2 -> /ROW2
- SW13 pad 1: /ROW1 -> /COL2
- SW13 pad 2: unconnected-(SW13-A-Pad2) -> Net-(SW13-A)
- SW13 pad 3: /COL2 -> /ROW1
- SW14 pad 1: /ROW0 -> /COL2
- SW14 pad 2: unconnected-(SW14-A-Pad2) -> Net-(SW14-A)
- SW14 pad 3: /COL2 -> /ROW0
- SW15 pad 1: /ROW4 -> /COL3
- SW15 pad 2: unconnected-(SW15-A-Pad2) -> Net-(SW15-A)
- SW15 pad 3: /COL3 -> /ROW4
- SW16 pad 1: /ROW3 -> /COL3
- SW16 pad 2: unconnected-(SW16-A-Pad2) -> Net-(SW16-A)
- SW16 pad 3: /COL3 -> /ROW3
- SW17 pad 1: /ROW2 -> /COL3
- SW17 pad 2: unconnected-(SW17-A-Pad2) -> Net-(SW17-A)
- SW17 pad 3: /COL3 -> /ROW2
- SW18 pad 1: /ROW1 -> /COL3
- SW18 pad 2: unconnected-(SW18-A-Pad2) -> Net-(SW18-A)
- SW18 pad 3: /COL3 -> /ROW1
- SW19 pad 1: /ROW0 -> /COL3
- SW19 pad 2: unconnected-(SW19-A-Pad2) -> Net-(SW19-A)
- SW19 pad 3: /COL3 -> /ROW0
- SW2 pad 1: /ROW2 -> /COL0
- SW2 pad 2: unconnected-(SW2-A-Pad2) -> Net-(SW2-A)
- SW2 pad 3: /COL0 -> /ROW2
- SW20 pad 1: /ROW4 -> /COL4
- SW20 pad 2: unconnected-(SW20-A-Pad2) -> Net-(SW20-A)
- SW20 pad 3: /COL4 -> /ROW4
- SW21 pad 1: /ROW3 -> /COL4
- SW21 pad 2: unconnected-(SW21-A-Pad2) -> Net-(SW21-A)
- SW21 pad 3: /COL4 -> /ROW3
- SW22 pad 1: /ROW2 -> /COL4
- SW22 pad 2: unconnected-(SW22-A-Pad2) -> Net-(SW22-A)
- SW22 pad 3: /COL4 -> /ROW2
- SW23 pad 1: /ROW1 -> /COL4
- SW23 pad 2: unconnected-(SW23-A-Pad2) -> Net-(SW23-A)
- SW23 pad 3: /COL4 -> /ROW1
- SW24 pad 1: /ROW0 -> /COL4
- SW24 pad 2: unconnected-(SW24-A-Pad2) -> Net-(SW24-A)
- SW24 pad 3: /COL4 -> /ROW0
- SW25 pad 1: /ROW4 -> /COL5
- SW25 pad 2: unconnected-(SW25-A-Pad2) -> Net-(SW25-A)
- SW25 pad 3: /COL5 -> /ROW4
- SW26 pad 1: /ROW3 -> /COL5
- SW26 pad 2: unconnected-(SW26-A-Pad2) -> Net-(SW26-A)
- SW26 pad 3: /COL5 -> /ROW3
- SW27 pad 1: /ROW2 -> /COL5
- SW27 pad 2: unconnected-(SW27-A-Pad2) -> Net-(SW27-A)
- SW27 pad 3: /COL5 -> /ROW2
- SW28 pad 1: /ROW1 -> /COL5
- SW28 pad 2: unconnected-(SW28-A-Pad2) -> Net-(SW28-A)
- SW28 pad 3: /COL5 -> /ROW1
- SW29 pad 1: /ROW0 -> /COL5
- SW29 pad 2: unconnected-(SW29-A-Pad2) -> Net-(SW29-A)
- SW29 pad 3: /COL5 -> /ROW0
- SW3 pad 1: /ROW1 -> /COL0
- SW3 pad 2: unconnected-(SW3-A-Pad2) -> Net-(SW3-A)
- SW3 pad 3: /COL0 -> /ROW1
- SW30 pad 1: /ROW4 -> /COL6
- SW30 pad 2: unconnected-(SW30-A-Pad2) -> Net-(SW30-A)
- SW30 pad 3: /COL6 -> /ROW4
- SW31 pad 1: /ROW3 -> /COL6
- SW31 pad 2: unconnected-(SW31-A-Pad2) -> Net-(SW31-A)
- SW31 pad 3: /COL6 -> /ROW3
- SW32 pad 1: /ROW2 -> /COL6
- SW32 pad 2: unconnected-(SW32-A-Pad2) -> Net-(SW32-A)
- SW32 pad 3: /COL6 -> /ROW2
- SW33 pad 1: /ROW1 -> /COL6
- SW33 pad 2: unconnected-(SW33-A-Pad2) -> Net-(SW33-A)
- SW33 pad 3: /COL6 -> /ROW1
- SW34 pad 1: /ROW0 -> /COL6
- SW34 pad 2: unconnected-(SW34-A-Pad2) -> Net-(SW34-A)
- SW34 pad 3: /COL6 -> /ROW0
- SW35 pad 1: /ROW4 -> /COL7
- SW35 pad 2: unconnected-(SW35-A-Pad2) -> Net-(SW35-A)
- SW35 pad 3: /COL7 -> /ROW4
- SW36 pad 1: /ROW3 -> /COL7
- SW36 pad 2: unconnected-(SW36-A-Pad2) -> Net-(SW36-A)
- SW36 pad 3: /COL7 -> /ROW3
- SW37 pad 1: /ROW2 -> /COL7
- SW37 pad 2: unconnected-(SW37-A-Pad2) -> Net-(SW37-A)
- SW37 pad 3: /COL7 -> /ROW2
- SW38 pad 1: /ROW1 -> /COL7
- SW38 pad 2: unconnected-(SW38-A-Pad2) -> Net-(SW38-A)
- SW38 pad 3: /COL7 -> /ROW1
- SW39 pad 1: /ROW4 -> /COL8
- SW39 pad 2: unconnected-(SW39-A-Pad2) -> Net-(SW39-A)
- SW39 pad 3: /COL8 -> /ROW4
- SW4 pad 1: /ROW0 -> /COL0
- SW4 pad 2: unconnected-(SW4-A-Pad2) -> Net-(SW4-A)
- SW4 pad 3: /COL0 -> /ROW0
- SW40 pad 1: /ROW3 -> /COL8
- SW40 pad 2: unconnected-(SW40-A-Pad2) -> Net-(SW40-A)
- SW40 pad 3: /COL8 -> /ROW3
- SW41 pad 1: /ROW2 -> /COL8
- SW41 pad 2: unconnected-(SW41-A-Pad2) -> Net-(SW41-A)
- SW41 pad 3: /COL8 -> /ROW2
- SW42 pad 1: /ROW1 -> /COL8
- SW42 pad 2: unconnected-(SW42-A-Pad2) -> Net-(SW42-A)
- SW42 pad 3: /COL8 -> /ROW1
- SW43 pad 1: /ROW0 -> /COL8
- SW43 pad 2: unconnected-(SW43-A-Pad2) -> Net-(SW43-A)
- SW43 pad 3: /COL8 -> /ROW0
- SW44 pad 1: /ROW4 -> /COL9
- SW44 pad 2: unconnected-(SW44-A-Pad2) -> Net-(SW44-A)
- SW44 pad 3: /COL9 -> /ROW4
- SW45 pad 1: /ROW3 -> /COL9
- SW45 pad 2: unconnected-(SW45-A-Pad2) -> Net-(SW45-A)
- SW45 pad 3: /COL9 -> /ROW3
- SW46 pad 1: /ROW2 -> /COL9
- SW46 pad 2: unconnected-(SW46-A-Pad2) -> Net-(SW46-A)
- SW46 pad 3: /COL9 -> /ROW2
- SW47 pad 1: /ROW1 -> /COL9
- SW47 pad 2: unconnected-(SW47-A-Pad2) -> Net-(SW47-A)
- SW47 pad 3: /COL9 -> /ROW1
- SW48 pad 1: /ROW0 -> /COL9
- SW48 pad 2: unconnected-(SW48-A-Pad2) -> Net-(SW48-A)
- SW48 pad 3: /COL9 -> /ROW0
- SW49 pad 1: /ROW4 -> /COL10
- SW49 pad 2: unconnected-(SW49-A-Pad2) -> Net-(SW49-A)
- SW49 pad 3: /COL10 -> /ROW4
- SW5 pad 1: /ROW4 -> /COL1
- SW5 pad 2: unconnected-(SW5-A-Pad2) -> Net-(SW5-A)
- SW5 pad 3: /COL1 -> /ROW4
- SW50 pad 1: /ROW3 -> /COL10
- SW50 pad 2: unconnected-(SW50-A-Pad2) -> Net-(SW50-A)
- SW50 pad 3: /COL10 -> /ROW3
- SW51 pad 1: /ROW2 -> /COL10
- SW51 pad 2: unconnected-(SW51-A-Pad2) -> Net-(SW51-A)
- SW51 pad 3: /COL10 -> /ROW2
- SW52 pad 1: /ROW1 -> /COL10
- SW52 pad 2: unconnected-(SW52-A-Pad2) -> Net-(SW52-A)
- SW52 pad 3: /COL10 -> /ROW1
- SW53 pad 1: /ROW0 -> /COL10
- SW53 pad 2: unconnected-(SW53-A-Pad2) -> Net-(SW53-A)
- SW53 pad 3: /COL10 -> /ROW0
- SW54 pad 1: /ROW4 -> /COL11
- SW54 pad 2: unconnected-(SW54-A-Pad2) -> Net-(SW54-A)
- SW54 pad 3: /COL11 -> /ROW4
- SW55 pad 1: /ROW3 -> /COL11
- SW55 pad 2: unconnected-(SW55-A-Pad2) -> Net-(SW55-A)
- SW55 pad 3: /COL11 -> /ROW3
- SW56 pad 1: /ROW2 -> /COL11
- SW56 pad 2: unconnected-(SW56-A-Pad2) -> Net-(SW56-A)
- SW56 pad 3: /COL11 -> /ROW2
- SW57 pad 1: /ROW1 -> /COL11
- SW57 pad 2: unconnected-(SW57-A-Pad2) -> Net-(SW57-A)
- SW57 pad 3: /COL11 -> /ROW1
- SW58 pad 1: /ROW0 -> /COL11
- SW58 pad 2: unconnected-(SW58-A-Pad2) -> Net-(SW58-A)
- SW58 pad 3: /COL11 -> /ROW0
- SW59 pad 1: /ROW4 -> /COL12
- SW59 pad 2: unconnected-(SW59-A-Pad2) -> Net-(SW59-A)
- SW59 pad 3: /COL12 -> /ROW4
- SW6 pad 1: /ROW3 -> /COL1
- SW6 pad 2: unconnected-(SW6-A-Pad2) -> Net-(SW6-A)
- SW6 pad 3: /COL1 -> /ROW3
- SW60 pad 1: /ROW3 -> /COL12
- SW60 pad 2: unconnected-(SW60-A-Pad2) -> Net-(SW60-A)
- SW60 pad 3: /COL12 -> /ROW3
- SW61 pad 1: /ROW2 -> /COL12
- SW61 pad 2: unconnected-(SW61-A-Pad2) -> Net-(SW61-A)
- SW61 pad 3: /COL12 -> /ROW2
- SW62 pad 1: /ROW1 -> /COL12
- SW62 pad 2: unconnected-(SW62-A-Pad2) -> Net-(SW62-A)
- SW62 pad 3: /COL12 -> /ROW1
- SW63 pad 1: /ROW0 -> /COL12
- SW63 pad 2: unconnected-(SW63-A-Pad2) -> Net-(SW63-A)
- SW63 pad 3: /COL12 -> /ROW0
- SW7 pad 1: /ROW2 -> /COL1
- SW7 pad 2: unconnected-(SW7-A-Pad2) -> Net-(SW7-A)
- SW7 pad 3: /COL1 -> /ROW2
- SW8 pad 1: /ROW1 -> /COL1
- SW8 pad 2: unconnected-(SW8-A-Pad2) -> Net-(SW8-A)
- SW8 pad 3: /COL1 -> /ROW1
- SW9 pad 1: /ROW0 -> /COL1
- SW9 pad 2: unconnected-(SW9-A-Pad2) -> Net-(SW9-A)
- SW9 pad 3: /COL1 -> /ROW0
Routing:
- net /COL12: track 218.6 -> 192.4 mm
- net /ROW1: track 314.7 -> 293.9 mm, vias 0 -> 14
- net /COL6: track 95.2 -> 76.2 mm
- net /COL0: track 184.4 -> 203.1 mm
- net /ROW2: track 311.9 -> 293.5 mm, vias 0 -> 13
- net /COL4: track 141.1 -> 157.5 mm
- net /COL11: track 192.1 -> 176.3 mm
- net /ROW0: track 312.2 -> 296.9 mm, vias 0 -> 13
- net /COL10: track 173.7 -> 159.0 mm
- net /COL7: track 100.0 -> 85.7 mm
- net /COL8: track 140.4 -> 126.2 mm
- net /COL9: track 155.3 -> 141.7 mm
- net Net-(SW62-A): track 0.00 -> 11.9 mm
- net Net-(SW61-A): track 0.00 -> 11.9 mm
- net Net-(SW8-A): track 0.00 -> 11.9 mm
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- removed copper zone on B.Cu, net GND
Other:
- board size 266.7 x 95.2 mm -> 256 x 90.6 mm

Commit message: Slight mods to kfs.
Parts:
- moved RST0 8.50 mm to (135.0, 34.0)
- moved U0 3.94 mm to (135.0, 39.6)
Routing:
- net /ROW4: track 296.4 -> 303.6 mm
- net /COL5: track 80.1 -> 86.5 mm
- net /ROW1: track 293.9 -> 298.0 mm
- net /ROW0: track 296.9 -> 301.0 mm
- net /ROW3: track 291.9 -> 295.9 mm
- net Net-(U0-RST): track 9.70 -> 5.75 mm
- net /ROW2: track 293.5 -> 297.4 mm
- net /COL4: track 157.5 -> 153.9 mm
- net /COL3: track 139.4 -> 136.6 mm
- net /COL12: track 192.4 -> 189.9 mm
- net /COL1: track 168.5 -> 166.3 mm
- net /COL2: track 151.2 -> 149.0 mm
- net /COL7: track 85.7 -> 83.5 mm
- net /COL8: track 126.2 -> 124.6 mm
- net /COL11: track 176.3 -> 174.7 mm
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Other:
- board size 256 x 90.6 mm -> 256 x 94.5 mm

Commit message: Moved some mounting holes on the kfs.
Parts:
- moved H0 23.2 mm to (148.0, 24.0)
- moved H4 23.2 mm to (122.0, 24.0)
- moved H3 17.0 mm to (216.0, 59.5)
- moved H7 14.1 mm to (22.0, 24.0)
- moved H9 14.1 mm to (266.0, 24.0)
- moved H10 4.53 mm to (266.0, 106.5)
- moved H8 4.53 mm to (22.0, 106.5)
Changed lines of the file:
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@@
   )
   (footprint "MountingHole:MountingHole_3.5mm" (layer "F.Cu")
-    (at 162 42.5)
+    (at 148 24)
     (descr "Mounting Hole 3.5mm, no annular")
     (tags "mounting hole 3.5mm no annular")
@@
   )
   (footprint "MountingHole:MountingHole_3.5mm" (layer "F.Cu")
-    (at 265.5 102)
+    (at 266 106.5)
     (descr "Mounting Hole 3.5mm, no annular")
     (tags "mounting hole 3.5mm no annular")
@@
   )
   (footprint "MountingHole:MountingHole_3.5mm" (layer "F.Cu")
-    (at 22.5 102)
+    (at 22 106.5)
     (descr "Mounting Hole 3.5mm, no annular")
     (tags "mounting hole 3.5mm no annular")
@@
   )
   (footprint "MountingHole:MountingHole_3.5mm" (layer "F.Cu")
-    (at 36 25.5)
+    (at 22 24)
     (descr "Mounting Hole 3.5mm, no annular")
     (tags "mounting hole 3.5mm no annular")
@@
   )
   (footprint "MountingHole:MountingHole_3.5mm" (layer "F.Cu")
-    (at 108 42.5)
+    (at 122 24)
     (descr "Mounting Hole 3.5mm, no annular")
     (tags "mounting hole 3.5mm no annular")
@@
   )
   (footprint "MountingHole:MountingHole_3.5mm" (layer "F.Cu")
-    (at 216 76.5)
+    (at 216 59.5)
     (descr "Mounting Hole 3.5mm, no annular")
     (tags "mounting hole 3.5mm no annular")
@@
   )
   (footprint "MountingHole:MountingHole_3.5mm" (layer "F.Cu")
-    (at 252 25.5)
+    (at 266 24)
     (descr "Mounting Hole 3.5mm, no annular")
     (tags "mounting hole 3.5mm no annular")
@@
   (segment (start 236.5 24.825) (end 153.545 24.825) (width 0.25) (layer "B.Cu") (net 85))
   (segment (start 257.725 28.05) (end 257.725 87.05) (width 0.25) (layer "B.Cu") (net 86))
-  (segment (start 245.65165 28.05) (end 241.97665 24.375) (width 0.25) (layer "B.Cu") (net 86))
-  (segment (start 257.725 87.05) (end 248.725 96.05) (width 0.25) (layer "B.Cu") (net 86))
   (segment (start 257.725 28.05) (end 245.65165 28.05) (width 0.25) (layer "B.Cu") (net 86))
-  (segment (start 146.375 24.375) (end 142.62 28.13) (width 0.25) (layer "B.Cu") (net 86))
-  (segment (start 241.97665 24.375) (end 146.375 24.375) (width 0.25) (layer "B.Cu") (net 86))
+  (segment (start 257.725 87.05) (end 248.725 96.05) (width 0.25) (layer "B.Cu") (net 86))
+  (segment (start 151.625 24.375) (end 147.87 28.13) (width 0.25) (layer "B.Cu") (net 86))
+  (segment (start 241.97665 24.375) (end 151.625 24.375) (width 0.25) (layer "B.Cu") (net 86))
+  (segment (start 147.87 28.13) (end 142.62 28.13) (width 0.25) (layer "B.Cu") (net 86))
+  (segment (start 245.65165 28.05) (end 241.97665 24.375) (width 0.25) (layer "B.Cu") (net 86))
   (zone (net 3) (net_name "GND") (layer "F.Cu") (hatch edge 0.5)
     (connect_pads (clearance 0.508))

Commit message: Switched to staggered kfs layout.
Parts:
- moved H3 200.3 mm to (16.5, 41.5)
- moved H8 196.2 mm to (216.0, 77.0)
- moved H5 184.1 mm to (289.5, 124.5)
- moved H10 150.7 mm to (130.0, 41.5)
- moved H2 137.7 mm to (289.5, 41.5)
- moved H4 114.1 mm to (176.0, 124.5)
- moved H9 109.4 mm to (158.0, 41.5)
- moved H0 106.8 mm to (112.0, 124.5)
- moved H6 85.5 mm to (16.5, 124.5)
- moved H7 72.9 mm to (72.0, 77.0)
- moved SW43 31.9 mm to (202.5, 119.0)
- moved SW48 31.9 mm to (225.0, 119.0)
- moved SW53 31.9 mm to (243.0, 119.0)
- moved SW58 31.9 mm to (261.0, 119.0)
- moved SW63 31.9 mm to (279.0, 119.0)
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Routing:
- net /COL5: track 86.5 -> 111.2 mm
- net /ROW0: track 301.0 -> 321.5 mm, vias 13 -> 12
- net /COL4: track 153.9 -> 171.3 mm
- net /ROW1: track 298.0 -> 314.5 mm, vias 14 -> 13
- net /COL0: track 201.4 -> 186.0 mm
- net /COL6: track 77.6 -> 86.8 mm
- net /COL7: track 83.5 -> 89.7 mm
- net /ROW4: track 303.6 -> 297.6 mm
- net /COL12: track 189.9 -> 194.6 mm
- net /COL9: track 140.1 -> 144.4 mm
- net /COL8: track 124.6 -> 128.9 mm
- net /COL11: track 174.7 -> 179.0 mm
- net /COL10: track 157.4 -> 161.7 mm
- net /COL2: track 149.0 -> 151.3 mm
- net /COL1: track 166.3 -> 168.6 mm
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Other:
- board size 256 x 94.5 mm -> 283 x 93 mm

Commit message: Moved the bottom row of kfs farther inward.
Parts:
- added H1: MountingHole, MountingHole:MountingHole_3.5mm, F.Cu at (153.0, 93.5)
- U0: value Arduino Pro Micro -> ARDUINO_PRO_MICRO
- moved SW14 9.00 mm to (72.0, 119.0)
- moved SW19 9.00 mm to (94.5, 119.0)
- moved SW4 9.00 mm to (36.0, 119.0)
- moved SW43 9.00 mm to (193.5, 119.0)
- moved SW48 9.00 mm to (216.0, 119.0)
- moved SW53 9.00 mm to (234.0, 119.0)
- moved SW58 9.00 mm to (252.0, 119.0)
- moved SW63 9.00 mm to (270.0, 119.0)
- moved SW9 9.00 mm to (54.0, 119.0)
Routing:
- net /ROW0: track 321.5 -> 303.5 mm
- net /COL0: track 186.0 -> 194.5 mm
- net /COL3: track 137.8 -> 144.7 mm
- net /COL1: track 168.6 -> 174.8 mm
- net /COL2: track 151.3 -> 157.5 mm
- net /COL8: track 128.9 -> 133.3 mm
- net /COL11: track 179.0 -> 182.8 mm
- net /COL12: track 194.6 -> 198.3 mm
- net /COL10: track 161.7 -> 165.5 mm
- net /COL9: track 144.4 -> 148.1 mm
- net /COL4: track 171.3 -> 168.8 mm

Commit message: Updated reset button and mounting holes on kfs.
Parts:
- removed H1, H7, H8: MountingHole, MountingHole:MountingHole_3.5mm
- RST0: footprint footprints:reset_button -> footprints:reset_button_1
- turned RST0 to 180 degrees
Connections:
- RST0 pad 1: Net-(U0-RST) -> GND
- RST0 pad 2: GND -> Net-(U0-RST)
Routing:
- net Net-(U0-RST): track 5.13 -> 11.3 mm
- net /ROW1: track 314.5 -> 315.0 mm
- added copper zone on B.Cu, net GND
- removed copper zone on F.Cu, net GND

Commit message: Changed reset button again. Removed some standoffs.
Parts:
- added H1: MountingHole, MountingHole:MountingHole_3.5mm, F.Cu at (155.0, 91.5)
- RST0: value RESET_SWITCH -> RESET
- moved RST0 26.1 mm to (121.5, 37.8)
Connections:
- RST0 pad 1: GND -> Net-(RST0-A)
- RST0 pad 2: Net-(U0-RST) -> GND
- U0 pad 22: Net-(U0-RST) -> Net-(RST0-A)
Routing:
- net Net-(RST0-A): track 0.00 -> 21.8 mm
- net Net-(U0-RST): track 11.3 -> 0.00 mm
Changed lines of the file:
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@@
   )
   (net 0 "")
-  (net 1 "Net-(U0-RST)")
+  (net 1 "Net-(RST0-A)")
   (net 2 "/ROW3")
   (net 3 "GND")
@@
       (net 8 "/ROW1") (pinfunction "K") (pintype "passive"))
   )
+  (footprint "MountingHole:MountingHole_3.5mm" (layer "F.Cu")
+    (at 155 91.5)
+    (descr "Mounting Hole 3.5mm, no annular")
+    (tags "mounting hole 3.5mm no annular")
+    (property "Sheetfile" "kfs_pcb.kicad_sch")
+    (property "Sheetname" "")
+    (property "ki_description" "Mounting Hole without connection")
+    (property "ki_keywords" "mounting hole")
+    (attr exclude_from_pos_files)
+    (fp_text reference "H1" (at 0 -4.5) (layer "F.SilkS") hide
+        (effects (font (size 1 1) (thickness 0.15)))
+    )
+    (fp_text value "MountingHole" (at 0 4.5) (layer "F.Fab")
+        (effects (font (size 1 1) (thickness 0.15)))
+    )
+    (fp_text user "${REFERENCE}" (at 0 0) (layer "F.Fab")
+        (effects (font (size 1 1) (thickness 0.15)))
+    )
+    (fp_circle (center 0 0) (end 3.5 0)
+      (stroke (width 0.15) (type solid)) (fill none) (layer "Cmts.User"))
+    (fp_circle (center 0 0) (end 3.75 0)
+      (stroke (width 0.05) (type solid)) (fill none) (layer "F.CrtYd"))
+    (pad "" np_thru_hole circle (at 0 0) (size 3.5 3.5) (drill 3.5) (layers "*.Cu" "*.Mask"))
+  )
   (footprint "footprints:kailh_choc_with_diode" (layer "F.Cu")
     (at 126 119)
@@
       (net 4 "VCC") (pinfunction "VCC") (pintype "power_in"))
     (pad "22" thru_hole circle (at -8.89 7.62 270) (size 1.7526 1.7526) (drill 1.0922) (layers "*.Cu" "*.SilkS" "*.Mask")
-      (net 1 "Net-(U0-RST)") (pinfunction "RST") (pintype "input"))
+      (net 1 "Net-(RST0-A)") (pinfunction "RST") (pintype "input"))
     (pad "23" thru_hole circle (at -11.43 7.62 270) (size 1.7526 1.7526) (drill 1.0922) (layers "*.Cu" "*.SilkS" "*.Mask")
       (net 3 "GND") (pinfunction "GND") (pintype "power_in"))
@@
   )
   (footprint "footprints:reset_button_1" (layer "B.Cu")
-    (at 144 51 180)
+    (at 121.5 37.75 180)
     (property "Sheetfile" "kfs_pcb.kicad_sch")
     (property "Sheetname" "")
+    (property "ki_description" "Single Pole Single Throw (SPST) switch")
+    (property "ki_keywords" "switch lever")
     (attr through_hole)
     (fp_text reference "RST0" (at 0 2.5) (layer "B.SilkS") hide
         (effects (font (size 1 1) (thickness 0.1)) (justify mirror))
     )
-    (fp_text value "RESET_SWITCH" (at 0 -2 unlocked) (layer "B.Fab") hide
+    (fp_text value "RESET" (at 0 -2 unlocked) (layer "B.Fab") hide
         (effects (font (size 1 1) (thickness 0.15)) (justify mirror))
     )
-    (fp_rect (start -2.05 1.4) (end 2.05 -1.4)
+    (fp_rect (start -1.5 1.25) (end 1.5 -1.25)
+      (stroke (width 0.1) (type default)) (fill none) (layer "Dwgs.User"))
+    (fp_rect (start -0.85 1.95) (end 0.85 1.25)
       (stroke (width 0.1) (type default)) (fill none) (layer "Dwgs.User"))
-    (pad "1" smd rect (at 2.55 0.8 180) (size 1.8 1) (layers "B.Cu" "B.Paste" "B.Mask")
-      (net 3 "GND") (pintype "passive"))
-    (pad "2" smd rect (at 2.55 -0.8 180) (size 1.8 1) (layers "B.Cu" "B.Paste" "B.Mask")
-      (net 1 "Net-(U0-RST)") (pintype "passive"))
-    (pad "3" smd rect (at -2.55 -0.8 180) (size 1.8 1) (layers "B.Cu" "B.Paste" "B.Mask")
-      (net 1 "Net-(U0-RST)") (pintype "passive"))
-    (pad "4" smd rect (at -2.55 0.8 180) (size 1.8 1) (layers "B.Cu" "B.Paste" "B.Mask")
-      (net 3 "GND") (pintype "passive"))
-    (pad "5" smd rect (at 0 2 180) (size 1.7 1.55) (layers "B.Cu" "B.Paste" "B.Mask")
-      (net 3 "GND") (pintype "passive"))
+    (pad "" np_thru_hole circle (at 0 0 180) (size 0.75 0.75) (drill 0.75) (layers "F&B.Cu" "*.Mask")
+      (thermal_bridge_angle 90))
+    (pad "1" smd rect (at 2.2 0 180) (size 1.8 1.7) (layers "B.Cu" "B.Paste" "B.Mask")
+      (net 1 "Net-(RST0-A)") (pinfunction "A") (pintype "passive"))
+    (pad "2" smd rect (at -2.2 0 180) (size 1.8 1.7) (layers "B.Cu" "B.Paste" "B.Mask")
+      (net 3 "GND") (pinfunction "B") (pintype "passive"))
   )
   (gr_arc (start 16.5 129.5) (mid 12.964466 128.035534) (end 11.5 124.5)
@@
   (gr_line (start 289.5 129.5) (end 16.5 129.5)
     (stroke (width 0.1) (type default)) (layer "Edge.Cuts"))
-  (segment (start 146.55 51.8) (end 139.01 51.8) (width 0.25) (layer "B.Cu") (net 1))
-  (segment (start 139.01 51.8) (end 136.38 49.17) (width 0.25) (layer "B.Cu") (net 1))
+  (segment (start 120.05 38.5) (end 119.3 37.75) (width 0.25) (layer "B.Cu") (net 1))
+  (segment (start 121.266396 38.5) (end 120.05 38.5) (width 0.25) (layer "B.Cu") (net 1))
+  (segment (start 136.38 49.17) (end 131.936396 49.17) (width 0.25) (layer "B.Cu") (net 1))
+  (segment (start 131.936396 49.17) (end 121.266396 38.5) (width 0.25) (layer "B.Cu") (net 1))
   (segment (start 101.725 72.08) (end 114.225 72.08) (width 0.25) (layer "F.Cu") (net 2))
   (segment (start 200.725 72.08) (end 218.725 72.08) (width 0.25) (layer "F.Cu") (net 2))
@@
     (polygon
       (pts
-        (xy 135 41.06)
-        (xy 153 41.06)
-        (xy 153 75.06)
-        (xy 135 75.06)
+        (xy 115 36.06)
+        (xy 153 36.06)
+        (xy 153 73.56)
+        (xy 115 73.56)
       )
     )
