File: kfs/kfs_pcb/kfs_pcb.kicad_pcb (KiCad board)
At the start: 2 copper layers, 283 x 93 mm, 75 parts, among them SW0 SWITCH, SW1 SWITCH, SW10 SWITCH, SW11 SWITCH, SW12 SWITCH, SW13 SWITCH, SW14 SWITCH, SW15 SWITCH, SW16 SWITCH, SW17 SWITCH, SW18 SWITCH, SW19 SWITCH, SW2 SWITCH, SW20 SWITCH, SW21 SWITCH, SW22 SWITCH, SW23 SWITCH, SW24 SWITCH, SW25 SWITCH, SW26 SWITCH, SW27 SWITCH, SW28 SWITCH, SW29 SWITCH, SW3 SWITCH, SW30 SWITCH, SW31 SWITCH, SW32 SWITCH, SW33 SWITCH, SW34 SWITCH, SW35 SWITCH, SW36 SWITCH, SW37 SWITCH, SW38 SWITCH, SW39 SWITCH, SW4 SWITCH, SW40 SWITCH, SW41 SWITCH, SW42 SWITCH, SW43 SWITCH, SW44 SWITCH, SW45 SWITCH, SW46 SWITCH, SW47 SWITCH, SW48 SWITCH, SW49 SWITCH, SW5 SWITCH, SW50 SWITCH, SW51 SWITCH, SW52 SWITCH, SW53 SWITCH, SW54 SWITCH, SW55 SWITCH, SW56 SWITCH, SW57 SWITCH, SW58 SWITCH, SW59 SWITCH, SW6 SWITCH, SW60 SWITCH, SW61 SWITCH, SW62 SWITCH, SW63 SWITCH, SW7 SWITCH, SW8 SWITCH, SW9 SWITCH, U0 ARDUINO_PRO_MICRO

Commit message: Switched kfs to use nice!nano.
Parts:
- added H11: MountingHole, MountingHole:MountingHole_3.5mm, F.Cu at (290.6, 78.2)
- added H12: B+, Connector_Pin:Pin_D0.9mm_L10.0mm_W2.4mm_FlatFork, B.Cu at (167.6, 44.2)
- added H13: B-, Connector_Pin:Pin_D0.9mm_L10.0mm_W2.4mm_FlatFork, B.Cu at (167.6, 49.3)
- added H7: MountingHole, MountingHole:MountingHole_3.5mm, F.Cu at (131.6, 84.8)
- added H8: MountingHole, MountingHole:MountingHole_3.5mm, F.Cu at (17.6, 78.2)
- added PWR0: POWER, footprints:AYZ0102AGRLC, B.Cu at (167.6, 34.2)
- U0: value ARDUINO_PRO_MICRO -> NICE!; footprint footprints:ARDUINO_PRO_MICRO -> footprints:nice!nano; moved to B.Cu
- moved U0 25.3 mm to (145.1, 32.8)
- moved H1 7.66 mm to (158.6, 84.8)
- moved H0 6.84 mm to (113.1, 117.8)
- moved H4 6.84 mm to (177.1, 117.8)
- moved H5 6.84 mm to (290.6, 117.8)
- moved H6 6.84 mm to (17.6, 117.8)
- moved SW0 6.84 mm to (37.1, 44.2)
- moved SW1 6.84 mm to (32.6, 61.2)
- moved SW10 6.84 mm to (73.1, 44.2)
- moved SW11 6.84 mm to (68.6, 61.2)
- moved SW12 6.84 mm to (64.1, 78.2)
- moved SW13 6.84 mm to (59.6, 95.2)
- moved SW14 6.84 mm to (73.1, 112.2)
- moved SW15 6.84 mm to (91.1, 44.2)
- moved SW16 6.84 mm to (86.6, 61.2)
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Connections:
- U0 pad 1: /ROW4 -> /COL12
- U0 pad 10: /COL6 -> /ROW4
- U0 pad 2: /COL12 -> /COL11
- U0 pad 21: VCC -> unconnected-(U0-VCC-Pad21)
- U0 pad 24: unconnected-(U0-RAW-Pad24) -> /RAW
- U0 pad 5: /COL11 -> /COL10
- U0 pad 6: /COL10 -> /COL9
- U0 pad 7: /COL9 -> /COL8
- U0 pad 8: /COL8 -> /COL7
- U0 pad 9: /COL7 -> /COL6
Routing:
- net /RAW: track 0.00 -> 29.8 mm
- net /ROW4: track 297.6 -> 270.8 mm
- net Net-(PWR0-B): track 0.00 -> 7.00 mm
- net /ROW3: track 293.9 -> 300.7 mm, vias 13 -> 14
- net /ROW0: track 303.5 -> 299.0 mm, vias 12 -> 13
- net /COL4: track 168.8 -> 172.1 mm
- net /ROW1: track 315.0 -> 312.1 mm, vias 13 -> 14
- net /COL11: track 182.8 -> 180.6 mm, vias 0 -> 1
- net /COL6: track 86.8 -> 88.8 mm
- net /ROW2: track 299.5 -> 301.2 mm, vias 13 -> 14
- net Net-(RST0-A): track 21.8 -> 20.2 mm
- net /COL7: track 89.7 -> 88.4 mm, vias 0 -> 1
- net /COL12: track 198.3 -> 197.2 mm, vias 0 -> 1
- net /COL8: track 133.3 -> 132.2 mm, vias 0 -> 1
- net /COL10: track 165.5 -> 164.5 mm, vias 0 -> 1
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Other:
- board size 283 x 93 mm -> 283 x 90 mm

Commit message: Changed the reset and power switches for kfs and jlk.
Parts:
- PWR0: footprint footprints:AYZ0102AGRLC -> footprints:power_switch
- RST0: footprint footprints:reset_button_1 -> footprints:reset_button_2
- moved RST0 4.36 mm to (125.9, 31.1), turned to 0 degrees
- moved PWR0 3.16 mm to (167.9, 31.1)
- moved SW13 1.67 mm to (59.9, 93.6)
- moved SW4 1.67 mm to (37.4, 110.6)
- moved SW7 1.67 mm to (46.4, 76.6)
- moved SW8 1.67 mm to (41.9, 93.6)
- moved SW9 1.67 mm to (55.4, 110.6)
- moved H6 1.67 mm to (17.9, 116.1)
- moved H8 1.67 mm to (17.9, 76.6)
- moved SW2 1.67 mm to (28.4, 76.6)
- moved SW3 1.67 mm to (23.9, 93.6)
- moved H0 1.67 mm to (113.4, 116.1)
- moved H1 1.67 mm to (158.9, 83.1)
- moved H11 1.67 mm to (290.9, 76.6)
- moved H13 1.67 mm to (167.9, 47.6)
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Connections:
- RST0 pad 1: Net-(RST0-A) -> GND
- RST0 pad 2: GND -> Net-(RST0-B)
- U0 pad 22: Net-(RST0-A) -> Net-(RST0-B)
Routing:
- net Net-(RST0-A): track 20.2 -> 0.00 mm
- net Net-(RST0-B): track 0.00 -> 13.0 mm, vias 0 -> 1
- net Net-(PWR0-B): track 7.00 -> 8.26 mm

Commit message: Moved some kfs mounting holes.
Parts:
- moved H1 6.50 mm to (158.9, 76.6)
- moved H7 6.50 mm to (131.9, 76.6)
Changed lines of the file:
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@@
   )
   (footprint "MountingHole:MountingHole_3.5mm" (layer "F.Cu")
-    (at 158.875 83.1)
+    (at 158.875 76.6)
     (descr "Mounting Hole 3.5mm, no annular")
     (tags "mounting hole 3.5mm no annular")
@@
   )
   (footprint "MountingHole:MountingHole_3.5mm" (layer "F.Cu")
-    (at 131.875 83.1)
+    (at 131.875 76.6)
     (descr "Mounting Hole 3.5mm, no annular")
     (tags "mounting hole 3.5mm no annular")

Commit message: Moved mcu to underside of pcb, added battery jack.
Parts:
- removed H12: B+, Connector_Pin:Pin_D0.9mm_L10.0mm_W2.4mm_FlatFork
- removed H13: B-, Connector_Pin:Pin_D0.9mm_L10.0mm_W2.4mm_FlatFork
- added J0: Conn_01x02_Socket, footprints:jst_ph, F.Cu at (157.1, 54.5)
- U0: moved to F.Cu
- moved RST0 3.61 mm to (122.3, 31.4)
- moved H11 1.62 mm to (290.3, 75.1)
- moved H2 1.62 mm to (290.3, 34.6)
- moved H5 1.62 mm to (290.3, 114.6)
- moved SW55 1.62 mm to (257.3, 58.1)
- moved SW56 1.62 mm to (261.8, 75.1)
- moved SW57 1.62 mm to (266.3, 92.1)
- moved SW59 1.62 mm to (270.8, 41.1)
- moved SW60 1.62 mm to (275.3, 58.1)
- moved SW61 1.62 mm to (279.8, 75.1)
- moved SW62 1.62 mm to (284.3, 92.1)
- moved SW63 1.62 mm to (270.8, 109.1)
- moved H3 1.62 mm to (17.3, 34.6)
- moved H6 1.62 mm to (17.3, 114.6)
- moved H8 1.62 mm to (17.3, 75.1)
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Connections:
- PWR0 pad 0: GND -> (no net)
- U0 pad 1: /COL12 -> /COL0
- U0 pad 11: /ROW3 -> /ROW1
- U0 pad 12: /ROW2 -> /ROW0
- U0 pad 13: /ROW0 -> /ROW2
- U0 pad 14: /ROW1 -> /ROW3
- U0 pad 15: /COL5 -> /COL7
- U0 pad 16: /COL4 -> /COL8
- U0 pad 17: /COL3 -> /COL9
- U0 pad 18: /COL2 -> /COL10
- U0 pad 19: /COL1 -> /COL11
- U0 pad 2: /COL11 -> /COL1
- U0 pad 20: /COL0 -> /COL12
- U0 pad 5: /COL10 -> /COL2
- U0 pad 6: /COL9 -> /COL3
- U0 pad 7: /COL8 -> /COL4
- U0 pad 8: /COL7 -> /COL6
- U0 pad 9: /COL6 -> /COL5
Routing:
- net Net-(J0-Pin_1): track 8.26 -> 26.3 mm
- net Net-(RST0-B): track 13.0 -> 30.8 mm
- net /RAW: track 30.1 -> 15.8 mm
- net /COL6: track 88.8 -> 102.0 mm
- net /COL12: track 197.2 -> 202.7 mm
- net /COL7: track 88.4 -> 93.3 mm
- net /COL11: track 180.6 -> 185.3 mm
- net /COL8: track 132.2 -> 135.8 mm
- net /COL10: track 164.5 -> 168.0 mm
- net /COL9: track 147.2 -> 150.7 mm
- net /ROW4: track 270.8 -> 274.1 mm
- net /COL0: track 194.2 -> 191.4 mm, vias 0 -> 1
- net /COL1: track 174.5 -> 172.3 mm, vias 0 -> 1
- net /COL5: track 111.7 -> 113.2 mm
- net /COL4: track 172.1 -> 171.3 mm, vias 0 -> 1
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