File: kfs/kfs_pcb/kfs_pcb.kicad_pcb (KiCad board)
At the start: 2 copper layers, 283 x 90 mm, 80 parts, among them J0 Conn_01x02_Socket, SW0 SWITCH, SW1 SWITCH, SW10 SWITCH, SW11 SWITCH, SW12 SWITCH, SW13 SWITCH, SW14 SWITCH, SW15 SWITCH, SW16 SWITCH, SW17 SWITCH, SW18 SWITCH, SW19 SWITCH, SW2 SWITCH, SW20 SWITCH, SW21 SWITCH, SW22 SWITCH, SW23 SWITCH, SW24 SWITCH, SW25 SWITCH, SW26 SWITCH, SW27 SWITCH, SW28 SWITCH, SW29 SWITCH, SW3 SWITCH, SW30 SWITCH, SW31 SWITCH, SW32 SWITCH, SW33 SWITCH, SW34 SWITCH, SW35 SWITCH, SW36 SWITCH, SW37 SWITCH, SW38 SWITCH, SW39 SWITCH, SW4 SWITCH, SW40 SWITCH, SW41 SWITCH, SW42 SWITCH, SW43 SWITCH, SW44 SWITCH, SW45 SWITCH, SW46 SWITCH, SW47 SWITCH, SW48 SWITCH, SW49 SWITCH, SW5 SWITCH, SW50 SWITCH, SW51 SWITCH, SW52 SWITCH, SW53 SWITCH, SW54 SWITCH, SW55 SWITCH, SW56 SWITCH, SW57 SWITCH, SW58 SWITCH, SW59 SWITCH, SW6 SWITCH, SW60 SWITCH, SW61 SWITCH, SW62 SWITCH, SW63 SWITCH, SW7 SWITCH, SW8 SWITCH, SW9 SWITCH, U0 NICE!

Commit message: Small changes.
Parts:
- J0: moved to B.Cu
- moved J0 0.15 mm to (157.2, 54.4), turned to 0 degrees
Connections:
- J0 pad 1: Net-(J0-Pin_1) -> GND
- J0 pad 2: GND -> Net-(J0-Pin_2)
- PWR0 pad 2: Net-(J0-Pin_1) -> Net-(J0-Pin_2)
Routing:
- net Net-(J0-Pin_1): track 26.3 -> 0.00 mm
- net Net-(J0-Pin_2): track 0.00 -> 26.1 mm
Changed lines of the file:
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@@
   (net 84 "/COL11")
   (net 85 "/COL12")
-  (net 86 "Net-(J0-Pin_1)")
+  (net 86 "Net-(J0-Pin_2)")
   (net 87 "unconnected-(PWR0-C-Pad3)")
   (net 88 "Net-(RST0-B)")
@@
       (net 7 "/ROW1") (pinfunction "K") (pintype "passive"))
   )
-  (footprint "footprints:jst_ph" (layer "F.Cu")
-    (at 157.1 54.5 180)
-    (property "Sheetfile" "kfs_pcb.kicad_sch")
-    (property "Sheetname" "")
-    (property "ki_description" "Generic connector, single row, 01x02, script generated")
-    (property "ki_keywords" "connector")
-    (attr through_hole)
-    (fp_text reference "J0" (at 0 -0.5 180 unlocked) (layer "F.SilkS")
-        (effects (font (size 1 1) (thickness 0.1)))
-    )
-    (fp_text value "Conn_01x02_Socket" (at 0 1 180 unlocked) (layer "F.Fab")
-        (effects (font (size 1 1) (thickness 0.15)))
-    )
-    (fp_text user "${REFERENCE}" (at 0 2.5 180 unlocked) (layer "F.Fab")
-        (effects (font (size 1 1) (thickness 0.15)))
-    )
-    (fp_rect (start -2.95 -8.25) (end 2.95 1.35)
-      (stroke (width 0.1) (type default)) (fill none) (layer "F.SilkS"))
-    (fp_rect (start -2.95 -1.35) (end 2.95 8.25)
-      (stroke (width 0.1) (type default)) (fill none) (layer "F.SilkS"))
-    (pad "1" thru_hole circle (at 1 0 180) (size 1.4 1.4) (drill 0.7) (layers "*.Cu" "*.Mask")
-      (net 86 "Net-(J0-Pin_1)") (pinfunction "Pin_1") (pintype "passive"))
-    (pad "2" thru_hole circle (at -1 0 180) (size 1.4 1.4) (drill 0.7) (layers "*.Cu" "*.Mask")
-      (net 2 "GND") (pinfunction "Pin_2") (pintype "passive"))
-  )
   (footprint "footprints:kailh_choc_with_diode" (layer "F.Cu")
     (at 117.775 75.1)
@@
     (pad "" np_thru_hole circle (at 0 0) (size 3.5 3.5) (drill 3.5) (layers "*.Cu" "*.Mask"))
   )
+  (footprint "footprints:jst_ph" (layer "B.Cu")
+    (at 157.165 54.37)
+    (property "Sheetfile" "kfs_pcb.kicad_sch")
+    (property "Sheetname" "")
+    (property "ki_description" "Generic connector, single row, 01x02, script generated")
+    (property "ki_keywords" "connector")
+    (attr through_hole)
+    (fp_text reference "J0" (at 0 0.5 180 unlocked) (layer "B.SilkS") hide
+        (effects (font (size 1 1) (thickness 0.1)) (justify mirror))
+    )
+    (fp_text value "Conn_01x02_Socket" (at 0 -1 180 unlocked) (layer "B.Fab")
+        (effects (font (size 1 1) (thickness 0.15)) (justify mirror))
+    )
+    (fp_text user "${REFERENCE}" (at 0 -2.5 180 unlocked) (layer "B.Fab")
+        (effects (font (size 1 1) (thickness 0.15)) (justify mirror))
+    )
+    (fp_line (start -2.95 6.25) (end 2.95 6.25)
+      (stroke (width 0.1) (type default)) (layer "B.SilkS"))
+    (fp_rect (start -2.95 8.25) (end 2.95 -1.35)
+      (stroke (width 0.1) (type default)) (fill none) (layer "B.SilkS"))
+    (pad "1" thru_hole circle (at 1 0) (size 1.4 1.4) (drill 0.7) (layers "*.Cu" "*.Mask")
+      (net 2 "GND") (pinfunction "Pin_1") (pintype "passive"))
+    (pad "2" thru_hole circle (at -1 0) (size 1.4 1.4) (drill 0.7) (layers "*.Cu" "*.Mask")
+      (net 86 "Net-(J0-Pin_2)") (pinfunction "Pin_2") (pintype "passive"))
+  )
   (footprint "footprints:reset_button_2" (layer "B.Cu")
     (at 122.275 31.35)
@@
       (net 81 "/RAW") (pinfunction "A") (pintype "passive"))
     (pad "2" smd rect (at 0.75 3.55) (size 0.7 1.5) (layers "B.Cu" "B.Paste" "B.Mask")
-      (net 86 "Net-(J0-Pin_1)") (pinfunction "B") (pintype "passive"))
+      (net 86 "Net-(J0-Pin_2)") (pinfunction "B") (pintype "passive"))
     (pad "3" smd rect (at 2.25 3.55) (size 0.7 1.5) (layers "B.Cu" "B.Paste" "B.Mask")
       (net 87 "unconnected-(PWR0-C-Pad3)") (pinfunction "C") (pintype "passive"))
@@
   (segment (start 267.5 103.15) (end 267.5 99.65) (width 0.25) (layer "B.Cu") (net 85))
   (segment (start 276.5 69.15) (end 276.5 81.65) (width 0.25) (layer "B.Cu") (net 85))
-  (segment (start 156.1 49.4) (end 156.1 54.5) (width 0.7) (layer "B.Cu") (net 86))
-  (segment (start 168.025 33.15) (end 168.025 37.475) (width 0.7) (layer "B.Cu") (net 86))
-  (segment (start 168.025 37.475) (end 156.1 49.4) (width 0.7) (layer "B.Cu") (net 86))
+  (segment (start 168.025 33.15) (end 168.025 37.0025) (width 0.7) (layer "B.Cu") (net 86))
+  (segment (start 168.025 37.0025) (end 156.165 48.8625) (width 0.7) (layer "B.Cu") (net 86))
+  (segment (start 156.165 48.8625) (end 156.165 54.37) (width 0.7) (layer "B.Cu") (net 86))
   (segment (start 127 30.5) (end 144.405 30.5) (width 0.25) (layer "F.Cu") (net 88))
   (segment (start 144.405 30.5) (end 152.395 38.49) (width 0.25) (layer "F.Cu") (net 88))
