File: jlk/jlk_pcb/jlk_pcb.kicad_pcb (KiCad board)
At the start: 2 copper layers, 254.5 x 111 mm, 38 parts, among them SW12 SWITCH_PUSH, SW13 SWITCH_PUSH, SW14 SWITCH_PUSH, SW17 SWITCH_PUSH, SW18 SWITCH_PUSH, SW19 SWITCH_PUSH, SW22 SWITCH_PUSH, SW23 SWITCH_PUSH, SW24 SWITCH_PUSH, SW25 SWITCH_PUSH, SW27 SWITCH_PUSH, SW28 SWITCH_PUSH, SW29 SWITCH_PUSH, SW30 SWITCH_PUSH, SW34 SWITCH_PUSH, SW35 SWITCH_PUSH, SW36 SWITCH_PUSH, SW37 SWITCH_PUSH, SW39 SWITCH_PUSH, SW40 SWITCH_PUSH, SW41 SWITCH_PUSH, SW42 SWITCH_PUSH, SW44 SWITCH_PUSH, SW45 SWITCH_PUSH, SW46 SWITCH_PUSH, SW49 SWITCH_PUSH, SW50 SWITCH_PUSH, SW51 SWITCH_PUSH, SW54 SWITCH_PUSH, SW55 SWITCH_PUSH, SW56 SWITCH_PUSH, SW7 SWITCH_PUSH, SW8 SWITCH_PUSH, SW9 SWITCH_PUSH, U1 ARDUINO_PRO_MICRO

Commit message: Final? design of jlk before fillet and creating plates.
Parts:
- removed REF** (x2): MountingHole_3.5mm, MountingHole:MountingHole_3.5mm
- added H0: MountingHole_Pad, MountingHole:MountingHole_2.2mm_M2_ISO7380_Pad, F.Cu at (240.2, 83.5)
- added H1: MountingHole_Pad, MountingHole:MountingHole_2.2mm_M2_ISO7380_Pad, F.Cu at (171.1, 115.7)
- added H10: MountingHole_Pad, MountingHole:MountingHole_2.2mm_M2_ISO7380_Pad, F.Cu at (121.8, 55.9)
- added H11: MountingHole_Pad, MountingHole:MountingHole_2.2mm_M2_ISO7380_Pad, F.Cu at (114.9, 115.7)
- added H12: MountingHole, MountingHole:MountingHole_3.5mm, F.Cu at (156.4, 48.9)
- added H13: MountingHole, MountingHole:MountingHole_3.5mm, F.Cu at (156.4, 115.7)
- added H14: MountingHole, MountingHole:MountingHole_3.5mm, F.Cu at (129.3, 48.9)
- added H15: MountingHole, MountingHole:MountingHole_3.5mm, F.Cu at (129.3, 115.7)
- added H2: MountingHole_Pad, MountingHole:MountingHole_2.2mm_M2_ISO7380_Pad, F.Cu at (49.5, 32.0)
- added H3: MountingHole_Pad, MountingHole:MountingHole_2.2mm_M2_ISO7380_Pad, F.Cu at (164.2, 55.9)
- added H4: MountingHole_Pad, MountingHole:MountingHole_2.2mm_M2_ISO7380_Pad, F.Cu at (205.7, 99.6)
- added H5: MountingHole_Pad, MountingHole:MountingHole_2.2mm_M2_ISO7380_Pad, F.Cu at (45.8, 83.5)
- added H6: MountingHole_Pad, MountingHole:MountingHole_2.2mm_M2_ISO7380_Pad, F.Cu at (195.0, 31.7)
- added H7: MountingHole_Pad, MountingHole:MountingHole_2.2mm_M2_ISO7380_Pad, F.Cu at (91.0, 31.7)
- added H8: MountingHole_Pad, MountingHole:MountingHole_2.2mm_M2_ISO7380_Pad, F.Cu at (80.4, 99.6)
- added H9: MountingHole_Pad, MountingHole:MountingHole_2.2mm_M2_ISO7380_Pad, F.Cu at (237.1, 31.7)
- RST0: renamed from RST1; footprint footprints:reset_button -> footprints:kailh_choc
- U0: renamed from U1; value ARDUINO_PRO_MICRO -> Arduino Pro Micro
- moved U0 28.7 mm to (142.9, 66.5)
- moved RST0 23.4 mm to (142.9, 91.2)
- moved SW33 16.6 mm to (257.2, 74.9)
- moved SW32 16.6 mm to (249.1, 57.6)
- moved SW31 16.6 mm to (241.1, 40.3)
- moved SW2 16.1 mm to (28.8, 74.9)
- moved SW0 16.1 mm to (44.9, 40.3)
- moved SW1 16.1 mm to (36.9, 57.6)
- moved SW17 16.0 mm to (168.3, 64.5)
- moved SW22 16.0 mm to (193.6, 73.7)
- moved SW21 16.0 mm to (185.5, 56.4)
- moved SW20 16.0 mm to (175.2, 124.3)
- moved SW23 16.0 mm to (201.6, 91.0)
- moved SW19 16.0 mm to (184.4, 99.0)
- moved SW18 16.0 mm to (176.3, 81.8)
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- renumbered SW7 to SW0, SW8 to SW1, SW23 to SW10, SW24 to SW11, SW25 to SW12, SW27 to SW13, SW28 to SW14, SW29 to SW15, SW30 to SW16, SW34 to SW17, SW35 to SW18, SW36 to SW19, SW9 to SW2, SW37 to SW20, SW39 to SW21, SW40 to SW22, SW41 to SW23, SW42 to SW24, SW44 to SW25, SW45 to SW26, SW46 to SW27, SW49 to SW28, SW50 to SW29, SW12 to SW3, SW51 to SW30, SW54 to SW31, SW55 to SW32, SW56 to SW33, SW13 to SW4, SW14 to SW5, SW17 to SW6, SW18 to SW7, SW19 to SW8, SW22 to SW9
Connections:
- U0 pad 10: /COL6 -> unconnected-(U0-E6-Pad10)
- U0 pad 15: /COL5 -> unconnected-(U0-B3-Pad15)
- U0 pad 16: /COL4 -> /COL5
- U0 pad 17: /COL3 -> /COL4
- U0 pad 18: /COL2 -> /COL3
- U0 pad 19: /COL1 -> /COL2
- U0 pad 20: unconnected-(U1-F4-Pad20) -> /COL1
- U0 pad 5: unconnected-(U1-SDA-Pad5) -> /COL10
- U0 pad 6: /COL10 -> /COL9
- U0 pad 7: /COL9 -> /COL8
- U0 pad 8: /COL8 -> /COL7
- U0 pad 9: /COL7 -> /COL6
Routing:
- net /ROW3: track 281.7 -> 259.6 mm
- net /ROW0: track 127.2 -> 148.3 mm
- net /COL2: track 130.6 -> 114.6 mm
- net /COL9: track 136.9 -> 123.9 mm
- net /COL10: track 160.3 -> 147.6 mm
- net /COL7: track 125.4 -> 113.3 mm
- net /COL3: track 104.8 -> 93.7 mm
- net /COL1: track 149.4 -> 139.0 mm
- net /COL5: track 96.5 -> 86.4 mm
- net /COL6: track 101.4 -> 91.6 mm
- net /COL8: track 112.4 -> 103.9 mm
- net /ROW2: track 269.4 -> 260.9 mm
- net /COL4: track 114.4 -> 107.2 mm
- net /ROW1: track 275.2 -> 282.1 mm
- net Net-(U0-RST): track 29.5 -> 30.9 mm
- added copper zone on B.Cu, net GND
Other:
- board size 254.5 x 111 mm -> 253.7 x 109.3 mm

Commit message: Fillet lines, add tplate, bplate for jlk.
Other:
- board size 253.7 x 109.3 mm -> 252.8 x 108.8 mm
- board text removed: "L"
Changed lines of the file:
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@@
       (net 3 "GND") (pinfunction "1") (pintype "input"))
   )
-  (gr_line (start 123.51681 119.729961) (end 115.465937 136.99513)
+  (gr_line (start 122.43986 122.039489) (end 116.099864 135.635668)
     (stroke (width 0.1) (type default)) (layer "Edge.Cuts"))
-  (gr_line (start 170.555333 27.680088) (end 245.696979 27.680082)
+  (gr_line (start 173.103614 27.680088) (end 244.741374 27.680082)
     (stroke (width 0.1) (type default)) (layer "Edge.Cuts"))
-  (gr_line (start 123.516808 44.945246) (end 162.504456 44.945254)
+  (gr_line (start 126.065089 44.945247) (end 159.956174 44.945254)
     (stroke (width 0.1) (type default)) (layer "Edge.Cuts"))
-  (gr_line (start 123.516808 44.945246) (end 115.465932 27.680078)
+  (gr_arc (start 126.065089 44.945247) (mid 123.915891 44.318812) (end 122.439859 42.635719)
     (stroke (width 0.1) (type default)) (layer "Edge.Cuts"))
-  (gr_line (start 80.935609 120.893374) (end 16.171644 79.475577)
+  (gr_line (start 122.439859 42.635719) (end 116.542882 29.989606)
     (stroke (width 0.1) (type default)) (layer "Edge.Cuts"))
-  (gr_line (start 40.324276 27.680087) (end 115.465932 27.680078)
+  (gr_arc (start 17.27792 80.183062) (mid 16.64563 79.33787) (end 16.726608 78.285452)
     (stroke (width 0.1) (type default)) (layer "Edge.Cuts"))
-  (gr_line (start 245.696979 27.680082) (end 269.849615 79.475571)
+  (gr_arc (start 169.478383 29.989615) (mid 170.954419 28.306532) (end 173.103614 27.680088)
     (stroke (width 0.1) (type default)) (layer "Edge.Cuts"))
-  (gr_line (start 16.171644 79.475577) (end 40.324276 27.680087)
+  (gr_arc (start 269.29465 78.285446) (mid 269.375628 79.337863) (end 268.743339 80.183056)
     (stroke (width 0.1) (type default)) (layer "Edge.Cuts"))
-  (gr_line (start 170.555333 136.995121) (end 162.504452 119.729955)
+  (gr_line (start 80.851679 120.839699) (end 17.27792 80.183062)
     (stroke (width 0.1) (type default)) (layer "Edge.Cuts"))
-  (gr_line (start 269.849615 79.475571) (end 205.085652 120.893372)
+  (gr_arc (start 159.956171 119.729955) (mid 162.105388 120.356374) (end 163.581402 122.039482)
     (stroke (width 0.1) (type default)) (layer "Edge.Cuts"))
-  (gr_line (start 123.51681 119.729961) (end 162.504452 119.729955)
+  (gr_line (start 41.279881 27.680087) (end 112.917651 27.680078)
     (stroke (width 0.1) (type default)) (layer "Edge.Cuts"))
-  (gr_line (start 170.555333 27.680088) (end 162.504456 44.945254)
+  (gr_arc (start 163.581406 42.635727) (mid 162.105378 44.318829) (end 159.956174 44.945254)
     (stroke (width 0.1) (type default)) (layer "Edge.Cuts"))
-  (gr_line (start 115.465937 136.99513) (end 80.935609 120.893374)
+  (gr_line (start 246.100835 28.546155) (end 269.29465 78.285446)
     (stroke (width 0.1) (type default)) (layer "Edge.Cuts"))
-  (gr_line (start 205.085662 120.893368) (end 170.555333 136.995121)
+  (gr_arc (start 81.025901 120.935478) (mid 80.9372 120.89048) (end 80.851679 120.839699)
+    (stroke (width 0.1) (type default)) (layer "Edge.Cuts"))
+  (gr_line (start 16.726608 78.285452) (end 39.92042 28.54616)
+    (stroke (width 0.1) (type default)) (layer "Edge.Cuts"))
+  (gr_line (start 169.921406 135.635659) (end 163.581402 122.039482)
+    (stroke (width 0.1) (type default)) (layer "Edge.Cuts"))
+  (gr_arc (start 122.43986 122.039489) (mid 123.915892 120.356396) (end 126.065091 119.729961)
+    (stroke (width 0.1) (type default)) (layer "Edge.Cuts"))
+  (gr_line (start 268.743339 80.183056) (end 205.085652 120.893372)
+    (stroke (width 0.1) (type default)) (layer "Edge.Cuts"))
+  (gr_line (start 126.065091 119.729961) (end 159.956171 119.729955)
+    (stroke (width 0.1) (type default)) (layer "Edge.Cuts"))
+  (gr_arc (start 244.741374 27.680082) (mid 245.547323 27.914995) (end 246.100835 28.546155)
+    (stroke (width 0.1) (type default)) (layer "Edge.Cuts"))
+  (gr_arc (start 116.099864 135.635668) (mid 115.253433 136.41128) (end 114.106475 136.361202)
+    (stroke (width 0.1) (type default)) (layer "Edge.Cuts"))
+  (gr_arc (start 112.917651 27.680078) (mid 115.066833 28.30653) (end 116.542882 29.989606)
+    (stroke (width 0.1) (type default)) (layer "Edge.Cuts"))
+  (gr_arc (start 171.914794 136.361194) (mid 170.767836 136.411271) (end 169.921406 135.635659)
+    (stroke (width 0.1) (type default)) (layer "Edge.Cuts"))
+  (gr_arc (start 39.92042 28.54616) (mid 40.473932 27.914998) (end 41.279881 27.680087)
+    (stroke (width 0.1) (type default)) (layer "Edge.Cuts"))
+  (gr_line (start 169.478383 29.989615) (end 163.581406 42.635727)
+    (stroke (width 0.1) (type default)) (layer "Edge.Cuts"))
+  (gr_line (start 114.106475 136.361202) (end 81.025901 120.935478)
+    (stroke (width 0.1) (type default)) (layer "Edge.Cuts"))
+  (gr_line (start 205.085662 120.893368) (end 171.914794 136.361194)
     (stroke (width 0.1) (type default)) (layer "Edge.Cuts"))
   (gr_text "\n" (at 142.875005 117.352533) (layer "B.SilkS")
@@
     )
   )
-  (gr_text "L" (at 142.375003 115.249984) (layer "F.SilkS")
-    (effects (font (face "Avenir Book") (size 10 10) (thickness 0.15)) (justify left bottom))
-    (render_cache "L" 0
-      (polygon
-        (pts
-          (xy 144.739273 112.612091)          (xy 149.379887 112.612091)          (xy 149.379887 113.549984)          (xy 143.725665 113.549984)
-          (xy 143.725665 103.545796)          (xy 144.739273 103.545796)
-        )
-      )
-    )
-  )
-  (gr_text "L" (at 143.375006 115.249984) (layer "F.SilkS")
-    (effects (font (face "Avenir Book") (size 10 10) (thickness 0.15)) (justify left bottom mirror))
-    (render_cache "L" 0
-      (polygon
-        (pts
-          (xy 141.010735 112.612091)          (xy 136.370121 112.612091)          (xy 136.370121 113.549984)          (xy 142.024343 113.549984)
-          (xy 142.024343 103.545796)          (xy 141.010735 103.545796)
-        )
-      )
-    )
-  )

Commit message: Switched to SMD diode, col2row.
Parts:
- removed H12, H13, H14, H15: MountingHole, MountingHole:MountingHole_3.5mm
- H0, H1, H10, H11, H2, H3, H4, H5, H6, H7, H8, H9: value MountingHole_Pad -> MountingHole; footprint MountingHole:MountingHole_2.2mm_M2_ISO7380_Pad -> MountingHole:MountingHole_3.5mm
- moved SW17 23.4 mm to (187.3, 78.0)
- moved SW0 23.4 mm to (64.0, 53.9)
- moved SW28 23.4 mm to (239.1, 53.9)
- moved RST0 23.4 mm to (161.9, 104.8)
- moved SW7 23.4 mm to (97.9, 71.2)
- moved SW27 23.4 mm to (234.2, 88.4)
- moved SW2 23.4 mm to (47.9, 88.4)
- moved SW16 23.4 mm to (129.9, 137.9)
- moved SW19 23.4 mm to (203.4, 112.6)
- moved U0 23.4 mm to (161.9, 80.0)
- moved SW26 23.4 mm to (226.2, 71.1)
- moved SW10 23.4 mm to (111.5, 87.2)
- moved H3 23.4 mm to (183.3, 69.4)
- moved H5 23.4 mm to (64.9, 97.0)
- moved SW9 23.4 mm to (119.5, 70.0)
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Connections:
- SW0 pad 1: /ROW3 -> /COL1
- SW0 pad 3: /COL1 -> /ROW3
- SW1 pad 1: /ROW2 -> /COL1
- SW1 pad 3: /COL1 -> /ROW2
- SW10 pad 1: /ROW2 -> /COL4
- SW10 pad 3: /COL4 -> /ROW2
- SW11 pad 1: /ROW1 -> /COL4
- SW11 pad 3: /COL4 -> /ROW1
- SW12 pad 1: /ROW0 -> /COL4
- SW12 pad 3: /COL4 -> /ROW0
- SW13 pad 1: /ROW3 -> /COL5
- SW13 pad 3: /COL5 -> /ROW3
- SW14 pad 1: /ROW2 -> /COL5
- SW14 pad 3: /COL5 -> /ROW2
- SW15 pad 1: /ROW1 -> /COL5
- SW15 pad 3: /COL5 -> /ROW1
- SW16 pad 1: /ROW0 -> /COL5
- SW16 pad 3: /COL5 -> /ROW0
- SW17 pad 1: /ROW3 -> /COL6
- SW17 pad 3: /COL6 -> /ROW3
- SW18 pad 1: /ROW2 -> /COL6
- SW18 pad 3: /COL6 -> /ROW2
- SW19 pad 1: /ROW1 -> /COL6
- SW19 pad 3: /COL6 -> /ROW1
- SW2 pad 1: /ROW1 -> /COL1
- SW2 pad 3: /COL1 -> /ROW1
- SW20 pad 1: /ROW0 -> /COL6
- SW20 pad 3: /COL6 -> /ROW0
- SW21 pad 1: /ROW3 -> /COL7
- SW21 pad 3: /COL7 -> /ROW3
- SW22 pad 1: /ROW2 -> /COL7
- SW22 pad 3: /COL7 -> /ROW2
- SW23 pad 1: /ROW1 -> /COL7
- SW23 pad 3: /COL7 -> /ROW1
- SW24 pad 1: /ROW0 -> /COL7
- SW24 pad 3: /COL7 -> /ROW0
- SW25 pad 1: /ROW3 -> /COL8
- SW25 pad 3: /COL8 -> /ROW3
- SW26 pad 1: /ROW2 -> /COL8
- SW26 pad 3: /COL8 -> /ROW2
- SW27 pad 1: /ROW1 -> /COL8
- SW27 pad 3: /COL8 -> /ROW1
- SW28 pad 1: /ROW3 -> /COL9
- SW28 pad 3: /COL9 -> /ROW3
- SW29 pad 1: /ROW2 -> /COL9
- SW29 pad 3: /COL9 -> /ROW2
- SW3 pad 1: /ROW3 -> /COL2
- SW3 pad 3: /COL2 -> /ROW3
- SW30 pad 1: /ROW1 -> /COL9
- SW30 pad 3: /COL9 -> /ROW1
- SW31 pad 1: /ROW3 -> /COL10
- SW31 pad 3: /COL10 -> /ROW3
- SW32 pad 1: /ROW2 -> /COL10
- SW32 pad 3: /COL10 -> /ROW2
- SW33 pad 1: /ROW1 -> /COL10
- SW33 pad 3: /COL10 -> /ROW1
- SW4 pad 1: /ROW2 -> /COL2
- SW4 pad 3: /COL2 -> /ROW2
- SW5 pad 1: /ROW1 -> /COL2
- SW5 pad 3: /COL2 -> /ROW1
- SW6 pad 1: /ROW3 -> /COL3
- SW6 pad 3: /COL3 -> /ROW3
- SW7 pad 1: /ROW2 -> /COL3
- SW7 pad 3: /COL3 -> /ROW2
- SW8 pad 1: /ROW1 -> /COL3
- SW8 pad 3: /COL3 -> /ROW1
- SW9 pad 1: /ROW3 -> /COL4
- SW9 pad 3: /COL4 -> /ROW3
Routing:
- net /COL2: track 114.6 -> 131.4 mm
- net /ROW1: track 282.1 -> 298.4 mm, vias 0 -> 10
- net /COL7: track 113.3 -> 99.5 mm
- net /COL3: track 93.7 -> 107.4 mm
- net /ROW0: track 148.3 -> 161.2 mm, vias 0 -> 4
- net /COL4: track 107.2 -> 119.2 mm
- net /COL1: track 139.0 -> 151.0 mm
- net /COL6: track 91.6 -> 80.6 mm
- net /COL5: track 86.4 -> 97.1 mm
- net /ROW3: track 259.6 -> 249.2 mm, vias 0 -> 10
- net /COL8: track 103.9 -> 94.4 mm
- net /ROW2: track 260.9 -> 267.8 mm, vias 0 -> 10
- net /COL10: track 147.6 -> 143.6 mm
- net Net-(SW7-A): track 8.98 -> 12.2 mm
- net Net-(SW2-A): track 8.98 -> 12.2 mm
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- removed copper zone on F.Cu, net GND
Other:
- board size 252.8 x 108.8 mm -> 253.4 x 109.2 mm

Commit message: Changed the reset button on the jlk.
Parts:
- removed RST0: RESET_SWITCH, footprints:kailh_choc
- added U1: RESET_BUTTON, footprints:reset_button_1, B.Cu at (154.0, 54.7)
- U0: value Arduino Pro Micro -> ARDUINO_PRO_MICRO
- moved H5 23.1 mm to (49.3, 79.9)
- moved H6 21.2 mm to (198.5, 30.8)
- moved H9 21.2 mm to (240.6, 30.8)
- moved H1 19.6 mm to (181.5, 111.6)
- moved H3 19.6 mm to (174.6, 51.8)
- moved H10 18.9 mm to (133.8, 51.8)
- moved H11 18.9 mm to (126.9, 111.6)
- moved SW15 17.6 mm to (112.8, 96.8)
- moved U0 17.6 mm to (154.0, 64.3)
- moved SW8 17.6 mm to (82.0, 72.6)
- moved SW22 17.6 mm to (204.8, 71.5)
- moved SW27 17.6 mm to (226.3, 72.6)
- moved SW12 17.6 mm to (104.8, 114.0)
- moved SW25 17.6 mm to (210.2, 38.1)
- moved SW24 17.6 mm to (203.6, 114.0)
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Routing:
- net Net-(U0-RST): track 30.9 -> 10.2 mm
- net /COL10: track 143.6 -> 139.1 mm
- net /COL9: track 124.0 -> 119.5 mm
- net /COL8: track 94.4 -> 92.5 mm
- net /COL1: track 151.0 -> 149.3 mm
- net /COL2: track 131.4 -> 130.1 mm
- net /ROW1: track 298.4 -> 299.5 mm
- net /COL6: track 80.6 -> 81.4 mm
- net /COL3: track 107.4 -> 108.1 mm

Commit message: Changed reset button again. Removed some standoffs.
Parts:
- removed H4, H6, H7, H8: MountingHole, MountingHole:MountingHole_3.5mm
- removed U1: RESET_BUTTON, footprints:reset_button_1
- added RST0: RESET, footprints:reset_button_1, F.Cu at (132.6, 64.3)
- moved H10 25.4 mm to (116.0, 70.0)
- moved H11 25.4 mm to (109.2, 129.8)
- moved H0 22.0 mm to (250.8, 100.3)
- moved SW4 22.0 mm to (60.8, 75.8)
- moved SW32 22.0 mm to (252.0, 75.8)
- moved SW22 22.0 mm to (196.5, 91.9)
- moved SW24 22.0 mm to (195.3, 134.4)
- moved SW14 22.0 mm to (112.6, 99.9)
- moved SW28 22.0 mm to (223.0, 58.5)
- moved SW3 22.0 mm to (68.9, 58.5)
- moved SW31 22.0 mm to (244.0, 58.5)
- moved SW10 22.0 mm to (95.3, 91.9)
- moved SW17 22.0 mm to (171.2, 82.6)
- moved SW0 22.0 mm to (47.8, 58.5)
- moved SW29 22.0 mm to (231.0, 75.8)
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Routing:
- net Net-(RST0-B): track 10.2 -> 14.6 mm
- net /COL2: track 130.1 -> 126.9 mm
- net /COL3: track 108.1 -> 105.7 mm
- net /COL4: track 119.2 -> 116.9 mm
- net /COL8: track 92.5 -> 90.2 mm
- net /COL9: track 119.5 -> 118.4 mm
- net /COL1: track 149.3 -> 150.0 mm
- added copper zone on F.Cu, net GND
- removed copper zone on B.Cu, net GND

Commit message: Changed jlk for mounting promicro under the pcb.
Parts:
- U0: value ARDUINO_PRO_MICRO -> Arduino Pro Micro
- moved RST0 32.0 mm to (164.3, 60.2)
- moved U0 26.2 mm to (151.0, 59.0)
- moved SW27 6.64 mm to (223.3, 88.9)
- moved SW31 6.64 mm to (249.2, 54.4)
- moved SW25 6.64 mm to (207.2, 54.4)
- moved SW19 6.64 mm to (192.5, 113.1)
- moved SW26 6.64 mm to (215.2, 71.7)
- moved SW32 6.64 mm to (257.3, 71.7)
- moved SW33 6.64 mm to (265.3, 88.9)
- moved SW13 6.64 mm to (125.9, 78.5)
- moved SW14 6.64 mm to (117.8, 95.8)
- moved SW15 6.64 mm to (109.8, 113.1)
- moved SW3 6.64 mm to (74.1, 54.4)
- moved SW4 6.64 mm to (66.0, 71.7)
- moved H2 6.64 mm to (64.7, 47.1)
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Connections:
- RST0 pad 1: GND -> Net-(RST0-A)
- RST0 pad 2: Net-(RST0-B) -> GND
- U0 pad 11: /ROW3 -> /ROW1
- U0 pad 12: /ROW2 -> /ROW0
- U0 pad 13: /ROW0 -> /ROW2
- U0 pad 14: /ROW1 -> /ROW3
- U0 pad 16: /COL5 -> /COL6
- U0 pad 17: /COL4 -> /COL7
- U0 pad 18: /COL3 -> /COL8
- U0 pad 19: /COL2 -> /COL9
- U0 pad 20: /COL1 -> /COL10
- U0 pad 22: Net-(RST0-B) -> Net-(RST0-A)
- U0 pad 5: /COL10 -> /COL1
- U0 pad 6: /COL9 -> /COL2
- U0 pad 7: /COL8 -> /COL3
- U0 pad 8: /COL7 -> /COL4
- U0 pad 9: /COL6 -> /COL5
Routing:
- net Net-(RST0-A): track 0.00 -> 14.7 mm
- net Net-(RST0-B): track 14.6 -> 0.00 mm
- net /ROW3: track 249.2 -> 259.9 mm
- net /ROW1: track 299.5 -> 306.3 mm, vias 10 -> 11
- net /ROW0: track 161.2 -> 162.8 mm, vias 4 -> 5
- net /ROW2: track 267.8 -> 268.6 mm, vias 10 -> 11
Other:
- outline, holes or cut-outs redrawn

Commit message: Switched jlk to use nice!nano.
Parts:
- added B+0: B+, Connector_Pin:Pin_D0.9mm_L10.0mm_W2.4mm_FlatFork, B.Cu at (148.5, 94.0)
- added B-0: B-, Connector_Pin:Pin_D0.9mm_L10.0mm_W2.4mm_FlatFork, B.Cu at (153.5, 94.0)
- added PWR0: POWER, footprints:AYZ0102AGRLC, F.Cu at (137.7, 58.2)
- U0: value Arduino Pro Micro -> NICE!; footprint footprints:ARDUINO_PRO_MICRO -> footprints:nice!nano; moved to B.Cu
- moved H3 2.25 mm to (181.0, 63.6)
- moved H0 2.25 mm to (256.0, 93.9)
- moved H1 2.25 mm to (187.9, 123.5)
- moved H11 2.25 mm to (114.4, 123.5)
- moved H2 2.25 mm to (64.7, 44.9)
- moved H5 2.25 mm to (46.3, 93.9)
- moved H9 2.25 mm to (237.5, 44.9)
- moved RST0 2.25 mm to (164.3, 58.0)
- moved SW0 2.25 mm to (53.1, 52.1)
- moved SW1 2.25 mm to (45.0, 69.4)
- moved SW10 2.25 mm to (100.6, 85.5)
- moved SW11 2.25 mm to (92.5, 102.8)
- moved SW12 2.25 mm to (101.7, 128.1)
- moved SW13 2.25 mm to (125.9, 76.3)
- moved SW14 2.25 mm to (117.8, 93.6)
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Connections:
- net Net-(RST0-A) renamed /RST
- U0 pad 11: /ROW1 -> /ROW3
- U0 pad 12: /ROW0 -> /ROW2
- U0 pad 13: /ROW2 -> /ROW0
- U0 pad 14: /ROW3 -> /ROW1
- U0 pad 16: /COL6 -> /COL5
- U0 pad 17: /COL7 -> /COL4
- U0 pad 18: /COL8 -> /COL3
- U0 pad 19: /COL9 -> /COL2
- U0 pad 20: /COL10 -> /COL1
- U0 pad 21: VCC -> unconnected-(U0-VCC-Pad21)
- U0 pad 24: unconnected-(U0-RAW-Pad24) -> /RAW
- U0 pad 5: /COL1 -> /COL10
- U0 pad 6: /COL2 -> /COL9
- U0 pad 7: /COL3 -> /COL8
- U0 pad 8: /COL4 -> /COL7
- U0 pad 9: /COL5 -> /COL6
Routing:
- net Net-(PWR0-B): track 0.00 -> 39.6 mm
- net /ROW3: track 259.9 -> 246.0 mm
- net /RST: track 14.7 -> 28.0 mm, vias 0 -> 1
- net /ROW2: track 268.6 -> 272.3 mm, vias 11 -> 10
- net /ROW0: track 162.8 -> 166.5 mm
- net /ROW1: track 306.3 -> 309.9 mm
- net /RAW: track 0.00 -> 3.47 mm
- net /COL5: track 97.1 -> 94.1 mm
- net /COL1: track 150.0 -> 147.3 mm
- net /COL7: track 99.5 -> 97.9 mm
- net /COL6: track 81.4 -> 79.8 mm
- net /COL2: track 126.9 -> 125.3 mm
- net /COL10: track 138.7 -> 137.2 mm
- net /COL8: track 90.2 -> 88.7 mm
- net /COL4: track 116.9 -> 115.4 mm
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- added copper zone on B.Cu, net GND
Other:
- outline, holes or cut-outs redrawn

Commit message: Changed the reset and power switches for kfs and jlk.
Parts:
- PWR0: footprint footprints:AYZ0102AGRLC -> footprints:power_switch
- RST0: footprint footprints:reset_button_1 -> footprints:reset_button_2
- moved PWR0 2.73 mm to (137.0, 55.6)
- moved RST0 2.49 mm to (163.6, 55.6), turned to 180 degrees
- moved B+0 1.33 mm to (147.8, 92.8)
- moved H1 1.33 mm to (187.2, 122.3)
- moved H11 1.33 mm to (113.7, 122.3)
- moved SW17 1.33 mm to (175.7, 75.1)
- moved SW18 1.33 mm to (183.8, 92.4)
- moved SW19 1.33 mm to (191.8, 109.7)
- moved SW26 1.33 mm to (214.5, 68.3)
- moved SW32 1.33 mm to (256.6, 68.3)
- moved SW33 1.33 mm to (264.6, 85.5)
- moved SW4 1.33 mm to (65.3, 68.3)
- moved SW25 1.33 mm to (206.5, 51.0)
- moved SW28 1.33 mm to (227.5, 51.0)
- moved SW3 1.33 mm to (73.4, 51.0)
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Connections:
- RST0 pad 1: /RST -> GND
- RST0 pad 2: GND -> /RST
Routing:
- net /RST: track 28.0 -> 21.6 mm
- net GND: vias 0 -> 4
Other:
- board text added: "B+"
- board text added: "B-"
