File: jlk/jlk_pcb/jlk_pcb.kicad_pcb (KiCad board)
At the start: 2 copper layers, 253.4 x 109.2 mm, 47 parts, among them SW0 SWITCH_PUSH, SW1 SWITCH_PUSH, SW10 SWITCH_PUSH, SW11 SWITCH_PUSH, SW12 SWITCH_PUSH, SW13 SWITCH_PUSH, SW14 SWITCH_PUSH, SW15 SWITCH_PUSH, SW16 SWITCH_PUSH, SW17 SWITCH_PUSH, SW18 SWITCH_PUSH, SW19 SWITCH_PUSH, SW2 SWITCH_PUSH, SW20 SWITCH_PUSH, SW21 SWITCH_PUSH, SW22 SWITCH_PUSH, SW23 SWITCH_PUSH, SW24 SWITCH_PUSH, SW25 SWITCH_PUSH, SW26 SWITCH_PUSH, SW27 SWITCH_PUSH, SW28 SWITCH_PUSH, SW29 SWITCH_PUSH, SW3 SWITCH_PUSH, SW30 SWITCH_PUSH, SW31 SWITCH_PUSH, SW32 SWITCH_PUSH, SW33 SWITCH_PUSH, SW4 SWITCH_PUSH, SW5 SWITCH_PUSH, SW6 SWITCH_PUSH, SW7 SWITCH_PUSH, SW8 SWITCH_PUSH, SW9 SWITCH_PUSH, U0 NICE!

Commit message: Slight update to jlk.
Connections:
- PWR0 pad 0: (no net) -> GND
Routing:
- net /COL1: track 147.3 -> 147.8 mm
- net GND: vias 4 -> 2
Changed lines of the file:
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@@
     (pad "" np_thru_hole circle (at 1.5 -1.8 180) (size 0.9 0.9) (drill 0.9) (layers "F&B.Cu" "*.Mask"))
     (pad "0" smd rect (at -3.65 -2.9 180) (size 1 0.8) (layers "F.Cu" "F.Paste" "F.Mask"))
-    (pad "0" smd rect (at -3.65 -0.7 180) (size 1 0.8) (layers "F.Cu" "F.Paste" "F.Mask"))
+    (pad "0" smd rect (at -3.65 -0.7 180) (size 1 0.8) (layers "F.Cu" "F.Paste" "F.Mask")
+      (net 2 "GND"))
     (pad "0" smd rect (at 3.65 -2.9 180) (size 1 0.8) (layers "F.Cu" "F.Paste" "F.Mask"))
     (pad "0" smd rect (at 3.65 -0.7 180) (size 1 0.8) (layers "F.Cu" "F.Paste" "F.Mask"))
@@
   (segment (start 156.740616 83.6087) (end 157.941916 84.81) (width 0.25) (layer "B.Cu") (net 1))
   (segment (start 48.622733 54.846755) (end 47.549282 57.148774) (width 0.25) (layer "B.Cu") (net 1))
-  (via (at 135 56) (size 0.6) (drill 0.4) (layers "F.Cu" "B.Cu") (free) (net 2))
-  (via (at 133.5 60.5) (size 0.6) (drill 0.4) (layers "F.Cu" "B.Cu") (free) (net 2))
-  (via (at 142 57) (size 0.6) (drill 0.4) (layers "F.Cu" "B.Cu") (free) (net 2))
+  (via (at 142.5 56.5) (size 0.6) (drill 0.4) (layers "F.Cu" "B.Cu") (free) (net 2))
   (via (at 161 60) (size 0.6) (drill 0.4) (layers "F.Cu" "B.Cu") (free) (net 2))
   (segment (start 142.611916 59.5) (end 142.701916 59.41) (width 0.7) (layer "F.Cu") (net 3))
@@
   (segment (start 81.063173 49.473054) (end 78.879507 54.155947) (width 0.25) (layer "B.Cu") (net 7))
   (segment (start 47.030587 45.696586) (end 30.92883 80.226913) (width 0.25) (layer "B.Cu") (net 8))
-  (segment (start 142.701916 69.57) (end 141.07 69.57) (width 0.25) (layer "B.Cu") (net 8))
-  (segment (start 112.85 41.35) (end 51.377174 41.35) (width 0.25) (layer "B.Cu") (net 8))
-  (segment (start 51.377174 41.35) (end 47.030591 45.696583) (width 0.25) (layer "B.Cu") (net 8))
+  (segment (start 52.087174 40.64) (end 47.030591 45.696583) (width 0.25) (layer "B.Cu") (net 8))
+  (segment (start 113.771916 40.64) (end 52.087174 40.64) (width 0.25) (layer "B.Cu") (net 8))
+  (segment (start 142.701916 69.57) (end 113.771916 40.64) (width 0.25) (layer "B.Cu") (net 8))
   (segment (start 30.92883 80.226913) (end 30.928826 80.226916) (width 0.25) (layer "B.Cu") (net 8))
-  (segment (start 141.07 69.57) (end 112.85 41.35) (width 0.25) (layer "B.Cu") (net 8))
   (segment (start 95.584804 89.364691) (end 112.849966 97.415569) (width 0.25) (layer "F.Cu") (net 9))
   (segment (start 157.941916 98.915853) (end 184.847721 98.915853) (width 0.25) (layer "F.Cu") (net 9))

Commit message: Moved mcu to underside of pcb, added battery jack.
Parts:
- removed B+0: B+, Connector_Pin:Pin_D0.9mm_L10.0mm_W2.4mm_FlatFork
- removed B-0: B-, Connector_Pin:Pin_D0.9mm_L10.0mm_W2.4mm_FlatFork
- added J0: Conn_01x02_Socket, footprints:jst_ph, B.Cu at (163.0, 80.5)
- U0: moved to F.Cu
- moved RST0 26.7 mm to (137.0, 57.4), turned to 0 degrees
- moved PWR0 26.6 mm to (163.6, 55.6)
Connections:
- PWR0 pad 0: GND -> (no net)
- PWR0 pad 1: /RAW -> unconnected-(PWR0-A-Pad1)
- PWR0 pad 3: unconnected-(PWR0-C-Pad3) -> /RAW
- RST0 pad 1: GND -> /RST
- RST0 pad 2: /RST -> GND
- U0 pad 11: /ROW3 -> /ROW1
- U0 pad 12: /ROW2 -> /ROW0
- U0 pad 13: /ROW0 -> /ROW2
- U0 pad 14: /ROW1 -> /ROW3
- U0 pad 16: /COL5 -> /COL6
- U0 pad 17: /COL4 -> /COL7
- U0 pad 18: /COL3 -> /COL8
- U0 pad 19: /COL2 -> /COL9
- U0 pad 20: /COL1 -> /COL10
- U0 pad 5: /COL10 -> /COL1
- U0 pad 6: /COL9 -> /COL2
- U0 pad 7: /COL8 -> /COL3
- U0 pad 8: /COL7 -> /COL4
- U0 pad 9: /COL6 -> /COL5
Routing:
- net Net-(J0-Pin_1): track 39.9 -> 21.7 mm
- net /ROW3: vias 10 -> 11
- net GND: vias 2 -> 0
- net /ROW2: vias 10 -> 11
- removed copper zone on B.Cu, net GND
Other:
- board text removed: "B+"
- board text removed: "B-"
