File: jlk/jlk_pcb/jlk_pcb.kicad_pcb (KiCad board)
At the start: 2 copper layers, 253.4 x 109.2 mm, 46 parts, among them J0 Conn_01x02_Socket, SW0 SWITCH_PUSH, SW1 SWITCH_PUSH, SW10 SWITCH_PUSH, SW11 SWITCH_PUSH, SW12 SWITCH_PUSH, SW13 SWITCH_PUSH, SW14 SWITCH_PUSH, SW15 SWITCH_PUSH, SW16 SWITCH_PUSH, SW17 SWITCH_PUSH, SW18 SWITCH_PUSH, SW19 SWITCH_PUSH, SW2 SWITCH_PUSH, SW20 SWITCH_PUSH, SW21 SWITCH_PUSH, SW22 SWITCH_PUSH, SW23 SWITCH_PUSH, SW24 SWITCH_PUSH, SW25 SWITCH_PUSH, SW26 SWITCH_PUSH, SW27 SWITCH_PUSH, SW28 SWITCH_PUSH, SW29 SWITCH_PUSH, SW3 SWITCH_PUSH, SW30 SWITCH_PUSH, SW31 SWITCH_PUSH, SW32 SWITCH_PUSH, SW33 SWITCH_PUSH, SW4 SWITCH_PUSH, SW5 SWITCH_PUSH, SW6 SWITCH_PUSH, SW7 SWITCH_PUSH, SW8 SWITCH_PUSH, SW9 SWITCH_PUSH, U0 NICE!

Commit message: Small changes.
Parts:
- moved J0 0.32 mm to (162.7, 80.4), turned to 0 degrees
Connections:
- J0 pad 1: Net-(J0-Pin_1) -> GND
- J0 pad 2: GND -> Net-(J0-Pin_2)
- PWR0 pad 2: Net-(J0-Pin_1) -> Net-(J0-Pin_2)
Routing:
- net Net-(J0-Pin_1): track 21.7 -> 0.00 mm
- net Net-(J0-Pin_2): track 0.00 -> 21.7 mm
Changed lines of the file:
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@@
   (net 54 "unconnected-(U0-TX-Pad1)")
   (net 55 "/RST")
-  (net 56 "Net-(J0-Pin_1)")
+  (net 56 "Net-(J0-Pin_2)")
   (net 57 "unconnected-(PWR0-A-Pad1)")
   (net 58 "unconnected-(U0-VCC-Pad21)")
@@
       (net 57 "unconnected-(PWR0-A-Pad1)") (pinfunction "A") (pintype "passive"))
     (pad "2" smd rect (at 0.75 -3.55 180) (size 0.7 1.5) (layers "F.Cu" "F.Paste" "F.Mask")
-      (net 56 "Net-(J0-Pin_1)") (pinfunction "B") (pintype "passive"))
+      (net 56 "Net-(J0-Pin_2)") (pinfunction "B") (pintype "passive"))
     (pad "3" smd rect (at 2.25 -3.55 180) (size 0.7 1.5) (layers "F.Cu" "F.Paste" "F.Mask")
       (net 3 "/RAW") (pinfunction "C") (pintype "passive"))
@@
   )
   (footprint "footprints:jst_ph" (layer "B.Cu")
-    (at 163 80.5 180)
+    (at 162.711916 80.37)
     (property "Sheetfile" "jlk_pcb.kicad_sch")
     (property "Sheetname" "")
@@
     (property "ki_keywords" "connector")
     (attr through_hole)
-    (fp_text reference "J0" (at 0 0.5 unlocked) (layer "B.SilkS")
+    (fp_text reference "J0" (at 0 0.5 -180 unlocked) (layer "B.SilkS") hide
         (effects (font (size 1 1) (thickness 0.1)) (justify mirror))
     )
-    (fp_text value "Conn_01x02_Socket" (at 0 -1 unlocked) (layer "B.Fab")
+    (fp_text value "Conn_01x02_Socket" (at 0 -1 -180 unlocked) (layer "B.Fab")
         (effects (font (size 1 1) (thickness 0.15)) (justify mirror))
     )
-    (fp_text user "${REFERENCE}" (at 0 -2.5 unlocked) (layer "B.Fab")
+    (fp_text user "${REFERENCE}" (at 0 -2.5 -180 unlocked) (layer "B.Fab")
         (effects (font (size 1 1) (thickness 0.15)) (justify mirror))
     )
-    (fp_rect (start -2.95 1.35) (end 2.95 -8.25)
-      (stroke (width 0.1) (type default)) (fill none) (layer "B.SilkS"))
+    (fp_line (start -2.95 6.25) (end 2.95 6.25)
+      (stroke (width 0.1) (type default)) (layer "B.SilkS"))
     (fp_rect (start -2.95 8.25) (end 2.95 -1.35)
       (stroke (width 0.1) (type default)) (fill none) (layer "B.SilkS"))
-    (pad "1" thru_hole circle (at 1 0 180) (size 1.4 1.4) (drill 0.7) (layers "*.Cu" "*.Mask")
-      (net 56 "Net-(J0-Pin_1)") (pinfunction "Pin_1") (pintype "passive"))
-    (pad "2" thru_hole circle (at -1 0 180) (size 1.4 1.4) (drill 0.7) (layers "*.Cu" "*.Mask")
-      (net 2 "GND") (pinfunction "Pin_2") (pintype "passive"))
+    (pad "1" thru_hole circle (at 1 0) (size 1.4 1.4) (drill 0.7) (layers "*.Cu" "*.Mask")
+      (net 2 "GND") (pinfunction "Pin_1") (pintype "passive"))
+    (pad "2" thru_hole circle (at -1 0) (size 1.4 1.4) (drill 0.7) (layers "*.Cu" "*.Mask")
+      (net 56 "Net-(J0-Pin_2)") (pinfunction "Pin_2") (pintype "passive"))
   )
   (gr_line (start 129.886767 132.694246) (end 123.124162 147.196726)
@@
   (segment (start 149.951916 56.5) (end 157.941916 64.49) (width 0.25) (layer "B.Cu") (net 55))
   (segment (start 142.5 56.5) (end 149.951916 56.5) (width 0.25) (layer "B.Cu") (net 55))
-  (segment (start 162.875 73.875) (end 162 74.75) (width 0.7) (layer "F.Cu") (net 56))
-  (segment (start 162 74.75) (end 162 80.5) (width 0.7) (layer "F.Cu") (net 56))
+  (segment (start 162.875 73.875) (end 161.711916 75.038084) (width 0.7) (layer "F.Cu") (net 56))
+  (segment (start 161.711916 75.038084) (end 161.711916 80.37) (width 0.7) (layer "F.Cu") (net 56))
   (segment (start 162.875 59.15) (end 162.875 73.875) (width 0.7) (layer "F.Cu") (net 56))
   (zone (net 2) (net_name "GND") (layer "F.Cu") (hatch edge 0.5)
