File: jlk/jlk_pcb/jlk_pcb.kicad_sch (KiCad schematic)
At the start: 47 parts, among them SW0 SWITCH_PUSH, SW1 SWITCH_PUSH, SW10 SWITCH_PUSH, SW11 SWITCH_PUSH, SW12 SWITCH_PUSH, SW13 SWITCH_PUSH, SW14 SWITCH_PUSH, SW15 SWITCH_PUSH, SW16 SWITCH_PUSH, SW17 SWITCH_PUSH, SW18 SWITCH_PUSH, SW19 SWITCH_PUSH, SW2 SWITCH_PUSH, SW20 SWITCH_PUSH, SW21 SWITCH_PUSH, SW22 SWITCH_PUSH, SW23 SWITCH_PUSH, SW24 SWITCH_PUSH, SW25 SWITCH_PUSH, SW26 SWITCH_PUSH, SW27 SWITCH_PUSH, SW28 SWITCH_PUSH, SW29 SWITCH_PUSH, SW3 SWITCH_PUSH, SW30 SWITCH_PUSH, SW31 SWITCH_PUSH, SW32 SWITCH_PUSH, SW33 SWITCH_PUSH, SW4 SWITCH_PUSH, SW5 SWITCH_PUSH, SW6 SWITCH_PUSH, SW7 SWITCH_PUSH, SW8 SWITCH_PUSH, SW9 SWITCH_PUSH, U0 NICE!

Commit message: Moved mcu to underside of pcb, added battery jack.
Parts:
- removed B+0: B+, Connector_Pin:Pin_D0.9mm_L10.0mm_W2.4mm_FlatFork, symbol Mechanical:MountingHole_Pad
- removed B-0: B-, Connector_Pin:Pin_D0.9mm_L10.0mm_W2.4mm_FlatFork, symbol Mechanical:MountingHole_Pad
- added J0: Conn_01x02_Socket, footprints:jst_ph, symbol Connector:Conn_01x02_Socket
Connections:
- net COL1: now also U0.5 (SDA); no longer U0.20 (F4)
- net COL10: now also U0.20 (F4); no longer U0.5 (SDA)
- net COL2: now also U0.6 (SCL); no longer U0.19 (F5)
- net COL3: now also U0.7 (D4); no longer U0.18 (F6)
- net COL4: now also U0.8 (C6); no longer U0.17 (F7)
- net COL5: now also U0.9 (D7); no longer U0.16 (B1)
- net COL6: now also U0.16 (B1); no longer U0.9 (D7)
- net COL7: now also U0.17 (F7); no longer U0.8 (C6)
- net COL8: now also U0.18 (F6); no longer U0.7 (D4)
- net COL9: now also U0.19 (F5); no longer U0.6 (SCL)
- net GND: now also RST0.2 (B), J0.2 (Pin_2); no longer RST0.1 (A)
- net RAW: now also PWR0.3 (C); no longer PWR0.1 (A)
- net ROW0: now also U0.12 (B5); no longer U0.13 (B6)
- net ROW1: now also U0.11 (B4); no longer U0.14 (B2)
- net ROW2: now also U0.13 (B6); no longer U0.12 (B5)
- net ROW3: now also U0.14 (B2); no longer U0.11 (B4)
- net RST: now also RST0.1 (A); no longer RST0.2 (B)
- net at PWR0.2 (B): now also J0.1 (Pin_1)
Changed lines of the file:
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@@
     (stroke (width 0) (type default))
   )
-  (label "COL5" (at 142.24 165.1 0) (fields_autoplaced)
+  (label "COL5" (at 106.68 165.1 180) (fields_autoplaced)
+    (effects (font (size 1.524 1.524)) (justify right bottom))
+  )
+  (label "COL2" (at 77.47 116.84 270) (fields_autoplaced)
+    (effects (font (size 1.524 1.524)) (justify right bottom))
+  )
+  (label "COL1" (at 106.68 154.94 180) (fields_autoplaced)
+    (effects (font (size 1.524 1.524)) (justify right bottom))
+  )
+  (label "GND" (at 106.68 149.86 180) (fields_autoplaced)
+    (effects (font (size 1.524 1.524)) (justify right bottom))
+  )
+  (label "COL8" (at 142.24 160.02 0) (fields_autoplaced)
     (effects (font (size 1.524 1.524)) (justify left bottom))
   )
-  (label "COL2" (at 77.47 116.84 270) (fields_autoplaced)
-    (effects (font (size 1.524 1.524)) (justify right bottom))
-  )
-  (label "COL1" (at 142.24 154.94 0) (fields_autoplaced)
+  (label "COL10" (at 294.64 116.84 270) (fields_autoplaced)
+    (effects (font (size 1.524 1.524)) (justify right bottom))
+  )
+  (label "ROW2" (at 21.59 71.12 180) (fields_autoplaced)
+    (effects (font (size 1.524 1.524)) (justify right bottom))
+  )
+  (label "COL6" (at 142.24 165.1 0) (fields_autoplaced)
     (effects (font (size 1.524 1.524)) (justify left bottom))
   )
-  (label "GND" (at 106.68 149.86 180) (fields_autoplaced)
-    (effects (font (size 1.524 1.524)) (justify right bottom))
-  )
-  (label "COL8" (at 106.68 160.02 180) (fields_autoplaced)
-    (effects (font (size 1.524 1.524)) (justify right bottom))
-  )
-  (label "COL10" (at 294.64 116.84 270) (fields_autoplaced)
-    (effects (font (size 1.524 1.524)) (justify right bottom))
-  )
-  (label "ROW2" (at 21.59 71.12 180) (fields_autoplaced)
-    (effects (font (size 1.524 1.524)) (justify right bottom))
-  )
-  (label "COL6" (at 106.68 165.1 180) (fields_autoplaced)
-    (effects (font (size 1.524 1.524)) (justify right bottom))
-  )
   (label "COL8" (at 246.38 116.84 270) (fields_autoplaced)
     (effects (font (size 1.524 1.524)) (justify right bottom))
   )
-  (label "COL3" (at 142.24 160.02 0) (fields_autoplaced)
-    (effects (font (size 1.524 1.524)) (justify left bottom))
-  )
-  (label "ROW0" (at 142.24 172.72 0) (fields_autoplaced)
-    (effects (font (size 1.524 1.524)) (justify left bottom))
+  (label "COL3" (at 106.68 160.02 180) (fields_autoplaced)
+    (effects (font (size 1.524 1.524)) (justify right bottom))
+  )
+  (label "ROW0" (at 106.68 172.72 180) (fields_autoplaced)
+    (effects (font (size 1.524 1.524)) (justify right bottom))
   )
   (label "RST" (at 271.78 175.26 180) (fields_autoplaced)
@@
     (effects (font (size 1.524 1.524)) (justify right bottom))
   )
-  (label "RAW" (at 265.43 152.4 180) (fields_autoplaced)
+  (label "RAW" (at 265.43 157.48 180) (fields_autoplaced)
     (effects (font (size 1.27 1.27)) (justify right bottom))
   )
-  (label "COL7" (at 106.68 162.56 180) (fields_autoplaced)
-    (effects (font (size 1.524 1.524)) (justify right bottom))
+  (label "COL7" (at 142.24 162.56 0) (fields_autoplaced)
+    (effects (font (size 1.524 1.524)) (justify left bottom))
   )
   (label "GND" (at 281.94 175.26 0) (fields_autoplaced)
@@
     (effects (font (size 1.524 1.524)) (justify right bottom))
   )
-  (label "COL4" (at 142.24 162.56 0) (fields_autoplaced)
+  (label "COL4" (at 106.68 162.56 180) (fields_autoplaced)
+    (effects (font (size 1.524 1.524)) (justify right bottom))
+  )
+  (label "COL10" (at 142.24 154.94 0) (fields_autoplaced)
     (effects (font (size 1.524 1.524)) (justify left bottom))
-  )
-  (label "COL10" (at 106.68 154.94 180) (fields_autoplaced)
-    (effects (font (size 1.524 1.524)) (justify right bottom))
   )
   (label "RST" (at 142.24 149.86 0) (fields_autoplaced)
     (effects (font (size 1.524 1.524)) (justify left bottom))
   )
-  (label "ROW1" (at 142.24 170.18 0) (fields_autoplaced)
+  (label "ROW1" (at 106.68 170.18 180) (fields_autoplaced)
+    (effects (font (size 1.524 1.524)) (justify right bottom))
+  )
+  (label "ROW3" (at 142.24 170.18 0) (fields_autoplaced)
     (effects (font (size 1.524 1.524)) (justify left bottom))
   )
-  (label "ROW3" (at 106.68 170.18 180) (fields_autoplaced)
-    (effects (font (size 1.524 1.524)) (justify right bottom))
-  )
-  (label "COL9" (at 106.68 157.48 180) (fields_autoplaced)
-    (effects (font (size 1.524 1.524)) (justify right bottom))
+  (label "COL9" (at 142.24 157.48 0) (fields_autoplaced)
+    (effects (font (size 1.524 1.524)) (justify left bottom))
   )
   (label "ROW3" (at 21.59 53.34 180) (fields_autoplaced)
@@
     (effects (font (size 1.524 1.524)) (justify right bottom))
   )
-  (label "COL2" (at 142.24 157.48 0) (fields_autoplaced)
+  (label "COL2" (at 106.68 157.48 180) (fields_autoplaced)
+    (effects (font (size 1.524 1.524)) (justify right bottom))
+  )
+  (label "ROW2" (at 142.24 172.72 0) (fields_autoplaced)
     (effects (font (size 1.524 1.524)) (justify left bottom))
-  )
-  (label "ROW2" (at 106.68 172.72 180) (fields_autoplaced)
-    (effects (font (size 1.524 1.524)) (justify right bottom))
   )
   (label "ROW1" (at 21.59 88.9 180) (fields_autoplaced)
@@
     )
   )
-  (symbol (lib_id "Mechanical:MountingHole_Pad") (at 275.59 152.4 0) (unit 1)
+  (symbol (lib_id "Connector:Conn_01x02_Socket") (at 280.67 154.94 0) (unit 1)
     (in_bom yes) (on_board yes) (dnp no) (fields_autoplaced)
-    (property "Reference" "B+0" (at 278.13 149.86 0)
-      (effects (font (size 1.27 1.27)) (justify left))
-    )
-    (property "Value" "B+" (at 278.13 152.4 0)
-      (effects (font (size 1.27 1.27)) (justify left))
-    )
-    (property "Footprint" "Connector_Pin:Pin_D0.9mm_L10.0mm_W2.4mm_FlatFork" (at 275.59 152.4 0)
-      (effects (font (size 1.27 1.27)) hide)
-    )
-    (property "Datasheet" "~" (at 275.59 152.4 0)
-      (effects (font (size 1.27 1.27)) hide)
-    )
-    (pin "1")
-    (instances
-      (project "jlk_pcb"
-        (path "/97127b28-60f4-45ff-835e-dccfbc833331"
-          (reference "B+0") (unit 1)
+    (property "Reference" "J0" (at 281.94 154.94 0)
+      (effects (font (size 1.27 1.27)) (justify left))
+    )
+    (property "Value" "Conn_01x02_Socket" (at 281.94 157.48 0)
+      (effects (font (size 1.27 1.27)) (justify left))
+    )
+    (property "Footprint" "footprints:jst_ph" (at 280.67 154.94 0)
+      (effects (font (size 1.27 1.27)) hide)
+    )
+    (property "Datasheet" "~" (at 280.67 154.94 0)
+      (effects (font (size 1.27 1.27)) hide)
+    )
+    (pin "1")
+    (pin "2")
+    (instances
+      (project "jlk_pcb"
+        (path "/97127b28-60f4-45ff-835e-dccfbc833331"
+          (reference "J0") (unit 1)
         )
       )
@@
     )
   )
-  (symbol (lib_id "power:GND") (at 283.21 154.94 0) (unit 1)
+  (symbol (lib_id "power:GND") (at 275.59 157.48 0) (unit 1)
     (in_bom yes) (on_board yes) (dnp no) (fields_autoplaced)
-    (property "Reference" "#PWR00" (at 283.21 161.29 0)
-      (effects (font (size 1.27 1.27)) hide)
-    )
-    (property "Value" "GND" (at 283.21 160.02 0)
-      (effects (font (size 1.27 1.27)))
-    )
-    (property "Footprint" "" (at 283.21 154.94 0)
-      (effects (font (size 1.27 1.27)) hide)
-    )
-    (property "Datasheet" "" (at 283.21 154.94 0)
+    (property "Reference" "#PWR00" (at 275.59 163.83 0)
+      (effects (font (size 1.27 1.27)) hide)
+    )
+    (property "Value" "GND" (at 275.59 162.56 0)
+      (effects (font (size 1.27 1.27)))
+    )
+    (property "Footprint" "" (at 275.59 157.48 0)
+      (effects (font (size 1.27 1.27)) hide)
+    )
+    (property "Datasheet" "" (at 275.59 157.48 0)
       (effects (font (size 1.27 1.27)) hide)
     )
@@
     )
   )
-  (symbol (lib_id "Switch:SW_SPST") (at 276.86 175.26 0) (mirror y) (unit 1)
+  (symbol (lib_id "Switch:SW_SPST") (at 276.86 175.26 0) (unit 1)
     (in_bom yes) (on_board yes) (dnp no)
     (property "Reference" "RST0" (at 276.86 168.91 0)
@@
         )
       )
-    )
-  )
-  (symbol (lib_id "Mechanical:MountingHole_Pad") (at 283.21 152.4 0) (unit 1)
-    (in_bom yes) (on_board yes) (dnp no) (fields_autoplaced)
-    (property "Reference" "B-0" (at 285.75 149.86 0)
-      (effects (font (size 1.27 1.27)) (justify left))
-    )
-    (property "Value" "B-" (at 285.75 152.4 0)
-      (effects (font (size 1.27 1.27)) (justify left))
-    )
-    (property "Footprint" "Connector_Pin:Pin_D0.9mm_L10.0mm_W2.4mm_FlatFork" (at 283.21 152.4 0)
-      (effects (font (size 1.27 1.27)) hide)
-    )
-    (property "Datasheet" "~" (at 283.21 152.4 0)
-      (effects (font (size 1.27 1.27)) hide)
-    )
-    (pin "1")
-    (instances
-      (project "jlk_pcb"
-        (path "/97127b28-60f4-45ff-835e-dccfbc833331"
-          (reference "B-0") (unit 1)
-        )
-      )

Commit message: Small changes.
Connections:
- net GND: now also J0.1 (Pin_1); no longer J0.2 (Pin_2)
- net at PWR0.2 (B): now also J0.2 (Pin_2); no longer J0.1 (Pin_1)
Changed lines of the file:
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@@
     )
   )
-  (symbol (lib_id "Connector:Conn_01x02_Socket") (at 280.67 154.94 0) (unit 1)
-    (in_bom yes) (on_board yes) (dnp no) (fields_autoplaced)
-    (property "Reference" "J0" (at 281.94 154.94 0)
+  (symbol (lib_id "Connector:Conn_01x02_Socket") (at 280.67 157.48 0) (mirror x) (unit 1)
+    (in_bom yes) (on_board yes) (dnp no)
+    (property "Reference" "J0" (at 281.94 157.48 0)
       (effects (font (size 1.27 1.27)) (justify left))
     )
-    (property "Value" "Conn_01x02_Socket" (at 281.94 157.48 0)
+    (property "Value" "Conn_01x02_Socket" (at 281.94 154.94 0)
       (effects (font (size 1.27 1.27)) (justify left))
     )
-    (property "Footprint" "footprints:jst_ph" (at 280.67 154.94 0)
+    (property "Footprint" "footprints:jst_ph" (at 280.67 157.48 0)
       (effects (font (size 1.27 1.27)) hide)
     )
-    (property "Datasheet" "~" (at 280.67 154.94 0)
+    (property "Datasheet" "~" (at 280.67 157.48 0)
       (effects (font (size 1.27 1.27)) hide)
     )
