File: jlk/jlk_bplate/jlk_bplate.kicad_pcb (KiCad board)
At the start: 2 copper layers, 252.8 x 108.8 mm, 16 parts

Commit message: Switched to SMD diode, col2row.
Parts:
- removed H12, H13, H14, H15: MountingHole, MountingHole:MountingHole_2.2mm_M2_ISO7380_Pad
- H0, H1, H10, H11, H2, H3, H4, H5, H6, H7, H8, H9: value MountingHole_Pad -> MountingHole
- moved H3 23.4 mm to (183.3, 69.4)
- moved H5 23.4 mm to (64.9, 97.0)
- moved H10 23.4 mm to (140.8, 69.4)
- moved H1 23.4 mm to (190.2, 129.2)
- moved H2 23.4 mm to (68.5, 45.5)
- moved H4 23.4 mm to (224.7, 113.1)
- moved H7 23.4 mm to (110.0, 45.2)
- moved H6 23.4 mm to (214.1, 45.2)
- moved H11 23.4 mm to (133.9, 129.2)
- moved H8 23.4 mm to (99.4, 113.1)
- moved H0 23.4 mm to (259.2, 97.0)
- moved H9 23.4 mm to (256.1, 45.2)
Other:
- board size 252.8 x 108.8 mm -> 253.4 x 109.2 mm

Commit message: Changed the reset button on the jlk.
Parts:
- added U1: RESET_BUTTON, MountingHole:MountingHole_8.4mm_M8, B.Cu at (154.0, 54.7)
- moved H5 23.1 mm to (49.3, 79.9)
- moved H6 21.2 mm to (198.5, 30.8)
- moved H9 21.2 mm to (240.6, 30.8)
- moved H1 19.6 mm to (181.5, 111.6)
- moved H3 19.6 mm to (174.6, 51.8)
- moved H10 18.9 mm to (133.8, 51.8)
- moved H11 18.9 mm to (126.9, 111.6)
- moved H4 17.6 mm to (210.9, 102.4)
- moved H0 17.1 mm to (259.0, 79.9)
- moved H2 14.7 mm to (67.8, 30.8)
- moved H7 14.4 mm to (109.8, 30.8)
- moved H8 10.9 mm to (97.5, 102.4)

Commit message: Changed jlk for mounting promicro under the pcb.
Parts:
- removed H4, H6, H7, H8: MountingHole, MountingHole:MountingHole_2.2mm_M2_ISO7380_Pad
- removed U1: RESET_BUTTON, MountingHole:MountingHole_8.4mm_M8
- moved H10 16.5 mm to (122.7, 64.0)
- moved H11 16.5 mm to (115.8, 123.9)
- moved H0 14.5 mm to (257.4, 94.3)
- moved H2 14.5 mm to (66.1, 45.3)
- moved H5 14.5 mm to (47.7, 94.3)
- moved H9 14.5 mm to (238.9, 45.3)
- moved H1 14.5 mm to (189.3, 123.9)
- moved H3 14.5 mm to (182.4, 64.0)
Other:
- outline, holes or cut-outs redrawn

Commit message: Switched jlk to use nice!nano.
Parts:
- moved H2 0.18 mm to (66.1, 45.1)
- moved H10 0.18 mm to (122.6, 63.9)
- moved H9 0.18 mm to (238.8, 45.1)
- moved H3 0.18 mm to (182.3, 63.9)
- moved H1 0.18 mm to (189.2, 123.7)
- moved H11 0.18 mm to (115.7, 123.7)
- moved H5 0.18 mm to (47.6, 94.2)
- moved H0 0.18 mm to (257.3, 94.2)
Other:
- outline, holes or cut-outs redrawn

Commit message: Moved mcu to underside of pcb, added battery jack.
Parts:
- moved H1 6.95 mm to (182.9, 120.7)
- moved H11 6.95 mm to (109.4, 120.7)
- moved H5 6.95 mm to (41.3, 91.2)
- moved H10 6.95 mm to (116.3, 60.9)
- moved H2 6.95 mm to (59.8, 42.1)
- moved H3 6.95 mm to (176.1, 60.9)
- moved H9 6.95 mm to (232.6, 42.1)
- moved H0 6.95 mm to (251.0, 91.2)
Other:
- outline, holes or cut-outs redrawn

Commit message: Added filled polygons on top and bottom plates.
Routing:
- added copper zone on B.Cu, net (none)
- added copper zone on F.Cu, net (none)
Changed lines of the file:
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@@
+    )
+  )
+  (zone (net 0) (net_name "") (layers "F&B.Cu") (hatch edge 0.5)
+    (connect_pads (clearance 0.508))
+    (min_thickness 0.25) (filled_areas_thickness no)
+    (fill yes (thermal_gap 0.5) (thermal_bridge_width 0.5) (island_removal_mode 1) (island_area_min 10))
+    (polygon
+      (pts
+        (xy 18.5 35.5)
+        (xy 274 35.5)
+        (xy 274 147)
+        (xy 270 151)
+        (xy 18.5 151)
+      )
     )
   )
