File: kfs/kfs_bplate/kfs_bplate.kicad_pcb (KiCad board)
At the start: 2 copper layers, 283 x 90 mm, 12 parts

Commit message: Moved mcu to underside of pcb, added battery jack.
Parts:
- moved H10 5.68 mm to (129.5, 32.3)
- moved H2 5.68 mm to (289.0, 32.3)
- moved H9 5.68 mm to (157.5, 32.3)
- moved H3 5.68 mm to (16.0, 32.3)
- moved H1 5.68 mm to (157.0, 72.8)
- moved H11 5.68 mm to (289.0, 72.8)
- moved H4 5.68 mm to (175.5, 112.3)
- moved H5 5.68 mm to (289.0, 112.3)
- moved H7 5.68 mm to (130.0, 72.8)
- moved H0 5.68 mm to (111.5, 112.3)
- moved H6 5.68 mm to (16.0, 112.3)
- moved H8 5.68 mm to (16.0, 72.8)
Other:
- outline, holes or cut-outs redrawn
Changed lines of the file:
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@@
   (net 0 "")
   (footprint "MountingHole:MountingHole_2.2mm_M2_ISO7380_Pad" (layer "F.Cu")
-    (at 17.62 78.25)
+    (at 16.01 72.805)
     (descr "Mounting Hole 2.2mm, M2, ISO7380")
     (tags "mounting hole 2.2mm m2 iso7380")
@@
   )
   (footprint "MountingHole:MountingHole_2.2mm_M2_ISO7380_Pad" (layer "F.Cu")
-    (at 113.12 117.75)
+    (at 111.51 112.305)
     (descr "Mounting Hole 2.2mm, M2, ISO7380")
     (tags "mounting hole 2.2mm m2 iso7380")
@@
   )
   (footprint "MountingHole:MountingHole_2.2mm_M2_ISO7380_Pad" (layer "F.Cu")
-    (at 290.62 78.25)
+    (at 289.01 72.805)
     (descr "Mounting Hole 2.2mm, M2, ISO7380")
     (tags "mounting hole 2.2mm m2 iso7380")
@@
   )
   (footprint "MountingHole:MountingHole_2.2mm_M2_ISO7380_Pad" (layer "F.Cu")
-    (at 131.12 37.75)
+    (at 129.51 32.305)
     (descr "Mounting Hole 2.2mm, M2, ISO7380")
     (tags "mounting hole 2.2mm m2 iso7380")
@@
   )
   (footprint "MountingHole:MountingHole_2.2mm_M2_ISO7380_Pad" (layer "F.Cu")
-    (at 290.62 37.75)
+    (at 289.01 32.305)
     (descr "Mounting Hole 2.2mm, M2, ISO7380")
     (tags "mounting hole 2.2mm m2 iso7380")
@@
   )
   (footprint "MountingHole:MountingHole_2.2mm_M2_ISO7380_Pad" (layer "F.Cu")
-    (at 17.62 117.75)
+    (at 16.01 112.305)
     (descr "Mounting Hole 2.2mm, M2, ISO7380")
     (tags "mounting hole 2.2mm m2 iso7380")
@@
   )
   (footprint "MountingHole:MountingHole_2.2mm_M2_ISO7380_Pad" (layer "F.Cu")
-    (at 158.62 78.25)
+    (at 157.01 72.805)
     (descr "Mounting Hole 2.2mm, M2, ISO7380")
     (tags "mounting hole 2.2mm m2 iso7380")
@@
   )
   (footprint "MountingHole:MountingHole_2.2mm_M2_ISO7380_Pad" (layer "F.Cu")
-    (at 177.12 117.75)
+    (at 175.51 112.305)
     (descr "Mounting Hole 2.2mm, M2, ISO7380")
     (tags "mounting hole 2.2mm m2 iso7380")
@@
   )
   (footprint "MountingHole:MountingHole_2.2mm_M2_ISO7380_Pad" (layer "F.Cu")
-    (at 131.62 78.25)
+    (at 130.01 72.805)
     (descr "Mounting Hole 2.2mm, M2, ISO7380")
     (tags "mounting hole 2.2mm m2 iso7380")
@@
   )
   (footprint "MountingHole:MountingHole_2.2mm_M2_ISO7380_Pad" (layer "F.Cu")
-    (at 290.62 117.75)
+    (at 289.01 112.305)
     (descr "Mounting Hole 2.2mm, M2, ISO7380")
     (tags "mounting hole 2.2mm m2 iso7380")
@@
   )
   (footprint "MountingHole:MountingHole_2.2mm_M2_ISO7380_Pad" (layer "F.Cu")
-    (at 17.62 37.75)
+    (at 16.01 32.305)
     (descr "Mounting Hole 2.2mm, M2, ISO7380")
     (tags "mounting hole 2.2mm m2 iso7380")
@@
   )
   (footprint "MountingHole:MountingHole_2.2mm_M2_ISO7380_Pad" (layer "F.Cu")
-    (at 159.12 37.75)
+    (at 157.51 32.305)
     (descr "Mounting Hole 2.2mm, M2, ISO7380")
     (tags "mounting hole 2.2mm m2 iso7380")
@@
     (pad "1" thru_hole circle (at 0 0) (size 3.5 3.5) (drill 2.2) (layers "*.Cu" "*.Mask"))
   )
-  (gr_arc (start 290.62 32.75) (mid 294.155534 34.214466) (end 295.62 37.75)
-    (stroke (width 0.1) (type default)) (layer "Edge.Cuts"))
-  (gr_arc (start 17.62 122.75) (mid 14.084466 121.285534) (end 12.62 117.75)
-    (stroke (width 0.1) (type default)) (layer "Edge.Cuts"))
-  (gr_arc (start 12.62 37.75) (mid 14.084466 34.214466) (end 17.62 32.75)
-    (stroke (width 0.1) (type default)) (layer "Edge.Cuts"))
-  (gr_line (start 17.62 32.75) (end 290.62 32.75)
-    (stroke (width 0.1) (type default)) (layer "Edge.Cuts"))
-  (gr_line (start 12.62 117.75) (end 12.62 37.75)
-    (stroke (width 0.1) (type default)) (layer "Edge.Cuts"))
-  (gr_line (start 295.62 37.75) (end 295.62 117.75)
-    (stroke (width 0.1) (type default)) (layer "Edge.Cuts"))
-  (gr_arc (start 295.62 117.75) (mid 294.155534 121.285534) (end 290.62 122.75)
-    (stroke (width 0.1) (type default)) (layer "Edge.Cuts"))
-  (gr_line (start 290.62 122.75) (end 17.62 122.75)
+  (gr_arc (start 289.01 27.305) (mid 292.545534 28.769466) (end 294.01 32.305)
+    (stroke (width 0.1) (type default)) (layer "Edge.Cuts"))
+  (gr_arc (start 153.035 60.46) (mid 152.888553 60.813553) (end 152.535 60.96)
+    (stroke (width 0.1) (type default)) (layer "Edge.Cuts"))
+  (gr_arc (start 16.01 117.305) (mid 12.474466 115.840534) (end 11.01 112.305)
+    (stroke (width 0.1) (type default)) (layer "Edge.Cuts"))
+  (gr_arc (start 133.485 27.305) (mid 133.838553 27.451447) (end 133.985 27.805)
+    (stroke (width 0.1) (type default)) (layer "Edge.Cuts"))
+  (gr_arc (start 11.01 32.305) (mid 12.474466 28.769466) (end 16.01 27.305)
+    (stroke (width 0.1) (type default)) (layer "Edge.Cuts"))
+  (gr_line (start 16.01 27.305) (end 133.485 27.305)
+    (stroke (width 0.1) (type default)) (layer "Edge.Cuts"))
+  (gr_arc (start 153.035 27.805) (mid 153.181447 27.451447) (end 153.535 27.305)
+    (stroke (width 0.1) (type default)) (layer "Edge.Cuts"))
+  (gr_line (start 134.485 60.96) (end 152.535 60.96)
+    (stroke (width 0.1) (type default)) (layer "Edge.Cuts"))
+  (gr_line (start 11.01 112.305) (end 11.01 32.305)
+    (stroke (width 0.1) (type default)) (layer "Edge.Cuts"))
+  (gr_line (start 294.01 32.305) (end 294.01 112.305)
+    (stroke (width 0.1) (type default)) (layer "Edge.Cuts"))
+  (gr_arc (start 294.01 112.305) (mid 292.545534 115.840534) (end 289.01 117.305)
+    (stroke (width 0.1) (type default)) (layer "Edge.Cuts"))
+  (gr_line (start 133.985 27.805) (end 133.985 60.46)
+    (stroke (width 0.1) (type default)) (layer "Edge.Cuts"))
+  (gr_arc (start 134.485 60.96) (mid 134.131447 60.813553) (end 133.985 60.46)
+    (stroke (width 0.1) (type default)) (layer "Edge.Cuts"))
+  (gr_line (start 289.01 117.305) (end 16.01 117.305)
+    (stroke (width 0.1) (type default)) (layer "Edge.Cuts"))
+  (gr_line (start 153.035 60.46) (end 153.035 27.805)
+    (stroke (width 0.1) (type default)) (layer "Edge.Cuts"))
+  (gr_line (start 153.535 27.305) (end 289.01 27.305)
     (stroke (width 0.1) (type default)) (layer "Edge.Cuts"))
 )

Commit message: Added filled polygons on top and bottom plates.
Routing:
- added copper zone on B.Cu, net (none)
- added copper zone on F.Cu, net (none)
Changed lines of the file:
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@@
   (gr_line (start 153.535 27.305) (end 289.01 27.305)
     (stroke (width 0.1) (type default)) (layer "Edge.Cuts"))
+  (zone (net 0) (net_name "") (layers "F&B.Cu") (hatch edge 0.5)
+    (connect_pads (clearance 0.508))
+    (min_thickness 0.25) (filled_areas_thickness no)
+    (fill yes (thermal_gap 0.5) (thermal_bridge_width 0.5) (island_removal_mode 1) (island_area_min 10))
+    (polygon
+      (pts
+        (xy 9 25)
+        (xy 295.5 25)
+        (xy 296 25.5)
+        (xy 296 118.5)
+        (xy 9 118.5)
+      )
+    )
+  )
 )
