File: kfs/kfs_tplate/kfs_tplate.kicad_pcb (KiCad board)
At the start: 2 copper layers, 283 x 95.5 mm, 76 parts, among them SW0 SWITCH, SW1 SWITCH, SW10 SWITCH, SW11 SWITCH, SW12 SWITCH, SW13 SWITCH, SW14 SWITCH, SW15 SWITCH, SW16 SWITCH, SW17 SWITCH, SW18 SWITCH, SW19 SWITCH, SW2 SWITCH, SW20 SWITCH, SW21 SWITCH, SW22 SWITCH, SW23 SWITCH, SW24 SWITCH, SW25 SWITCH, SW26 SWITCH, SW27 SWITCH, SW28 SWITCH, SW29 SWITCH, SW3 SWITCH, SW30 SWITCH, SW31 SWITCH, SW32 SWITCH, SW33 SWITCH, SW34 SWITCH, SW35 SWITCH, SW36 SWITCH, SW37 SWITCH, SW38 SWITCH, SW39 SWITCH, SW4 SWITCH, SW40 SWITCH, SW41 SWITCH, SW42 SWITCH, SW43 SWITCH, SW44 SWITCH, SW45 SWITCH, SW46 SWITCH, SW47 SWITCH, SW48 SWITCH, SW49 SWITCH, SW5 SWITCH, SW50 SWITCH, SW51 SWITCH, SW52 SWITCH, SW53 SWITCH, SW54 SWITCH, SW55 SWITCH, SW56 SWITCH, SW57 SWITCH, SW58 SWITCH, SW59 SWITCH, SW6 SWITCH, SW60 SWITCH, SW61 SWITCH, SW62 SWITCH, SW63 SWITCH, SW7 SWITCH, SW8 SWITCH, SW9 SWITCH

Commit message: Moved mcu to underside of pcb, added battery jack.
Parts:
- added U1: ${VALUE}, footprints:nice!nano_holes, F.Cu at (154.9, 26.7)
- moved H3 4.74 mm to (27.4, 31.7)
- moved H6 4.74 mm to (27.4, 111.7)
- moved H8 4.74 mm to (27.4, 72.2)
- moved H0 4.74 mm to (122.9, 111.7)
- moved H1 4.74 mm to (168.4, 72.2)
- moved H10 4.74 mm to (140.9, 31.7)
- moved H11 4.74 mm to (300.4, 72.2)
- moved H2 4.74 mm to (300.4, 31.7)
- moved H4 4.74 mm to (186.9, 111.7)
- moved H5 4.74 mm to (300.4, 111.7)
- moved H7 4.74 mm to (141.4, 72.2)
- moved H9 4.74 mm to (168.9, 31.7)
- moved SW0 4.74 mm to (46.9, 38.2)
- moved SW1 4.74 mm to (42.4, 55.2)
- moved SW10 4.74 mm to (82.9, 38.2)
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Other:
- outline, holes or cut-outs redrawn

Commit message: Small changes.
Parts:
- removed U1: ${VALUE}, footprints:nice!nano_holes
Other:
- board size 283 x 95.5 mm -> 283 x 90 mm
- board text removed: "CHRISTINE IS CUTE!"
Changed lines of the file:
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@@
       (stroke (width 0.05) (type default)) (layer "Edge.Cuts"))
-  )
-  (footprint "footprints:nice!nano_holes" (layer "F.Cu")
-    (at 154.94 26.67 -90)
-    (attr through_hole)
-    (fp_text reference "U1" (at 17.78 -1.625 90) (layer "F.SilkS") hide
-        (effects (font (size 1.27 1.524) (thickness 0.2032)))
-    )
-    (fp_text value "${VALUE}" (at 17.78 0 90) (layer "F.SilkS") hide
-        (effects (font (size 1.27 1.524) (thickness 0.254) bold))
-    )
-    (fp_rect (start 0 -8.89) (end 33.02 8.89)
-      (stroke (width 0.1) (type default)) (fill none) (layer "Dwgs.User"))
-    (pad "" np_thru_hole circle (at 3.81 -7.62 270) (size 0.85 0.85) (drill 0.85) (layers "*.Cu" "*.Mask"))
-    (pad "" np_thru_hole circle (at 3.81 7.62 270) (size 0.85 0.85) (drill 0.85) (layers "*.Cu" "*.Mask"))
-    (pad "" np_thru_hole circle (at 6.35 -7.62 270) (size 0.85 0.85) (drill 0.85) (layers "*.Cu" "*.Mask"))
-    (pad "" np_thru_hole circle (at 6.35 7.62 270) (size 0.85 0.85) (drill 0.85) (layers "*.Cu" "*.Mask"))
-    (pad "" np_thru_hole circle (at 8.89 -7.62 270) (size 0.85 0.85) (drill 0.85) (layers "*.Cu" "*.Mask"))
-    (pad "" np_thru_hole circle (at 8.89 7.62 270) (size 0.85 0.85) (drill 0.85) (layers "*.Cu" "*.Mask"))
-    (pad "" np_thru_hole circle (at 11.43 -7.62 270) (size 0.85 0.85) (drill 0.85) (layers "*.Cu" "*.Mask"))
-    (pad "" np_thru_hole circle (at 11.43 7.62 270) (size 0.85 0.85) (drill 0.85) (layers "*.Cu" "*.Mask"))
-    (pad "" np_thru_hole circle (at 13.97 -7.62 270) (size 0.85 0.85) (drill 0.85) (layers "*.Cu" "*.Mask"))
-    (pad "" np_thru_hole circle (at 13.97 7.62 270) (size 0.85 0.85) (drill 0.85) (layers "*.Cu" "*.Mask"))
-    (pad "" np_thru_hole circle (at 16.51 -7.62 270) (size 0.85 0.85) (drill 0.85) (layers "*.Cu" "*.Mask"))
-    (pad "" np_thru_hole circle (at 16.51 7.62 270) (size 0.85 0.85) (drill 0.85) (layers "*.Cu" "*.Mask"))
-    (pad "" np_thru_hole circle (at 19.05 -7.62 270) (size 0.85 0.85) (drill 0.85) (layers "*.Cu" "*.Mask"))
-    (pad "" np_thru_hole circle (at 19.05 7.62 270) (size 0.85 0.85) (drill 0.85) (layers "*.Cu" "*.Mask"))
-    (pad "" np_thru_hole circle (at 21.59 -7.62 270) (size 0.85 0.85) (drill 0.85) (layers "*.Cu" "*.Mask"))
-    (pad "" np_thru_hole circle (at 21.59 7.62 270) (size 0.85 0.85) (drill 0.85) (layers "*.Cu" "*.Mask"))
-    (pad "" np_thru_hole circle (at 24.13 -7.62 270) (size 0.85 0.85) (drill 0.85) (layers "*.Cu" "*.Mask"))
-    (pad "" np_thru_hole circle (at 24.13 7.62 270) (size 0.85 0.85) (drill 0.85) (layers "*.Cu" "*.Mask"))
-    (pad "" np_thru_hole circle (at 26.67 -7.62 270) (size 0.85 0.85) (drill 0.85) (layers "*.Cu" "*.Mask"))
-    (pad "" np_thru_hole circle (at 26.67 7.62 270) (size 0.85 0.85) (drill 0.85) (layers "*.Cu" "*.Mask"))
-    (pad "" np_thru_hole circle (at 29.21 -7.62 270) (size 0.85 0.85) (drill 0.85) (layers "*.Cu" "*.Mask"))
-    (pad "" np_thru_hole circle (at 29.21 7.62 270) (size 0.85 0.85) (drill 0.85) (layers "*.Cu" "*.Mask"))
-    (pad "" np_thru_hole circle (at 31.75 -7.62 270) (size 0.85 0.85) (drill 0.85) (layers "*.Cu" "*.Mask"))
-    (pad "" np_thru_hole circle (at 31.75 7.62 270) (size 0.85 0.85) (drill 0.85) (layers "*.Cu" "*.Mask"))
   )
   (footprint "footprints:kailh_choc_plate" (layer "F.Cu")
@@
     (pad "1" thru_hole circle (at 0 0) (size 3.5 3.5) (drill 2.2) (layers "*.Cu" "*.Mask"))
   )
-  (gr_line (start 193.44 21.17) (end 278.44 21.17)
-    (stroke (width 0.1) (type default)) (layer "Edge.Cuts"))
+  (gr_line (start 127.94 35.17) (end 181.94 35.17)
+    (stroke (width 0.6) (type default)) (layer "F.SilkS"))
+  (gr_line (start 127.94 43.17) (end 181.94 43.17)
+    (stroke (width 0.6) (type default)) (layer "F.SilkS"))
   (gr_arc (start 300.44 26.67) (mid 303.975534 28.134466) (end 305.44 31.67)
     (stroke (width 0.1) (type default)) (layer "Edge.Cuts"))
   (gr_arc (start 27.44 116.67) (mid 23.904466 115.205534) (end 22.44 111.67)
     (stroke (width 0.1) (type default)) (layer "Edge.Cuts"))
-  (gr_line (start 190.94 24.17) (end 190.94 23.67)
-    (stroke (width 0.1) (type default)) (layer "Edge.Cuts"))
   (gr_arc (start 22.44 31.67) (mid 23.904466 28.134466) (end 27.44 26.67)
     (stroke (width 0.1) (type default)) (layer "Edge.Cuts"))
-  (gr_line (start 27.44 26.67) (end 188.44 26.67)
+  (gr_line (start 27.44 26.67) (end 300.44 26.67)
     (stroke (width 0.1) (type default)) (layer "Edge.Cuts"))
   (gr_line (start 22.44 111.67) (end 22.44 31.67)
@@
   (gr_line (start 305.44 31.67) (end 305.44 111.67)
     (stroke (width 0.1) (type default)) (layer "Edge.Cuts"))
-  (gr_arc (start 278.44 21.17) (mid 280.207767 21.902233) (end 280.94 23.67)
-    (stroke (width 0.1) (type default)) (layer "Edge.Cuts"))
-  (gr_arc (start 190.94 23.67) (mid 191.672233 21.902233) (end 193.44 21.17)
-    (stroke (width 0.1) (type default)) (layer "Edge.Cuts"))
   (gr_arc (start 305.44 111.67) (mid 303.975534 115.205534) (end 300.44 116.67)
-    (stroke (width 0.1) (type default)) (layer "Edge.Cuts"))
-  (gr_line (start 280.94 24.17) (end 280.94 23.67)
-    (stroke (width 0.1) (type default)) (layer "Edge.Cuts"))
-  (gr_arc (start 190.94 24.17) (mid 190.207767 25.937767) (end 188.44 26.67)
-    (stroke (width 0.1) (type default)) (layer "Edge.Cuts"))
-  (gr_line (start 283.44 26.67) (end 300.44 26.67)
-    (stroke (width 0.1) (type default)) (layer "Edge.Cuts"))
-  (gr_arc (start 283.44 26.67) (mid 281.672233 25.937767) (end 280.94 24.17)
     (stroke (width 0.1) (type default)) (layer "Edge.Cuts"))
   (gr_line (start 300.44 116.67) (end 27.44 116.67)
     (stroke (width 0.1) (type default)) (layer "Edge.Cuts"))
-  (gr_text "CHRISTINE\nIS CUTE!" (at 154.94 43.18 270) (layer "B.Cu")
-    (effects (font (size 3 3) (thickness 0.5) bold) (justify mirror))
-  )
-  (gr_text "KEYS FOR SUCCESS" (at 235.94 25.67) (layer "F.SilkS")
-    (effects (font (size 5.5 5.5) (thickness 1) bold))
+  (gr_text "KEYS FOR SUCCESS" (at 154.94 39.17) (layer "F.SilkS")
+    (effects (font (size 3.4 3.4) (thickness 0.6) bold))
   )
 )

Commit message: Added filled polygons on top and bottom plates.
Routing:
- added copper zone on B.Cu, net (none)
- added copper zone on F.Cu, net (none)
Changed lines of the file:
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@@
     (effects (font (size 3.4 3.4) (thickness 0.6) bold))
   )
+  (zone (net 0) (net_name "") (layers "F&B.Cu") (hatch edge 0.5)
+    (connect_pads (clearance 0.508))
+    (min_thickness 0.25) (filled_areas_thickness no)
+    (fill yes (thermal_gap 0.5) (thermal_bridge_width 0.5) (island_removal_mode 1) (island_area_min 10))
+    (polygon
+      (pts
+        (xy 306.5 26)
+        (xy 306.5 117.5)
+        (xy 22 117.5)
+        (xy 21.5 117)
+        (xy 21.5 26)
+      )
+    )
+  )
 )
