File: jlks/jlks_pcb/jlks_pcb.kicad_sch (KiCad schematic)
At the start: 27 parts, among them J0 Conn_01x02_Socket, SW0 SW_Push, SW1 SW_Push, SW10 SW_Push, SW11 SW_Push, SW12 SW_Push, SW13 SW_Push, SW14 SW_Push, SW15 SW_Push, SW16 SW_Push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

Commit message: Changed out the power switch and reset button on jlks.
Parts:
- removed PWR1: POWER, footprints:power_switch, symbol Switch:SW_SPDT
- removed RST1: RESET, footprints:reset_button_2, symbol Switch:SW_SPST
- PWR0: footprint footprints:power_switch -> footprints:power_switch_1
- RST0: footprint footprints:reset_button_2 -> footprints:reset_button
Connections:
- net KEY0: now also U0.1 (TX); no longer U0.19 (F5)
- net KEY1: now also U0.7 (D4); no longer U0.14 (B2)
- net KEY10: now also U0.10 (E6); no longer U0.16 (B1)
- net KEY11: now also U0.16 (B1); no longer U0.8 (C6)
- net KEY12: now also U0.6 (SCL); no longer U0.5 (SDA)
- net KEY13: now also U0.11 (B4); no longer U0.15 (B3)
- net KEY14: now also U0.15 (B3); no longer U0.9 (D7)
- net KEY15: now also U0.14 (B2); no longer U0.11 (B4)
- net KEY16: now also U0.13 (B6); no longer U0.12 (B5)
- net KEY2: now also U0.12 (B5); no longer U0.10 (E6)
- net KEY3: now also U0.2 (RX); no longer U0.1 (TX)
- net KEY4: now also U0.8 (C6); no longer U0.18 (F6)
- net KEY5: now also U0.18 (F6); no longer U0.13 (B6)
- net KEY6: now also U0.20 (F4); no longer U0.2 (RX)
- net KEY7: now also U0.9 (D7); no longer U0.17 (F7)
- net KEY8: now also U0.17 (F7); no longer U0.7 (D4)
- net KEY9: now also U0.5 (SDA); no longer U0.20 (F4)
