File: jlks/jlks_pcb/jlks_pcb.kicad_pcb (KiCad board)
At the start: 2 copper layers, 114.3 x 99.4 mm, 25 parts, among them J0 Conn_01x02_Socket, SW0 SW_Push, SW1 SW_Push, SW10 SW_Push, SW11 SW_Push, SW12 SW_Push, SW13 SW_Push, SW14 SW_Push, SW15 SW_Push, SW16 SW_Push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

Commit message: Moved the battery pins and power switch on the jlks.
Parts:
- moved PWR0 61.0 mm to (123.8, 133.3), turned to 180 degrees
- moved J0 15.5 mm to (97.0, 110.0)
Routing:
- net /RAW: track 43.8 -> 130.3 mm
- net /B+: track 111.0 -> 32.8 mm
- net GND: vias 18 -> 17
Changed lines of the file:
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@@
   )
   (footprint "Connector_PinHeader_2.54mm:PinHeader_1x02_P2.54mm_Vertical" (layer "F.Cu")
-    (at 112.5 109.96)
+    (at 97 109.96)
     (descr "Through hole straight pin header, 1x02, 2.54mm pitch, single row")
     (tags "Through hole pin header THT 1x02 2.54mm single row")
@@
   )
   (footprint "footprints:power_switch_1" (layer "B.Cu")
-    (at 171.45 95.25 -90)
+    (at 123.825 133.35 180)
     (property "Sheetfile" "jlks_pcb.kicad_sch")
     (property "Sheetname" "")
@@
     (property "ki_keywords" "switch single-pole double-throw spdt ON-ON")
     (attr smd)
-    (fp_text reference "PWR0" (at 0 8.8 90 unlocked) (layer "B.SilkS") hide
+    (fp_text reference "PWR0" (at 0 8.8 unlocked) (layer "B.SilkS") hide
         (effects (font (size 1 1) (thickness 0.1)) (justify mirror))
     )
-    (fp_text value "POWER" (at 0 7.3 90 unlocked) (layer "B.Fab")
+    (fp_text value "POWER" (at 0 7.3 unlocked) (layer "B.Fab")
         (effects (font (size 1 1) (thickness 0.15)) (justify mirror))
     )
-    (fp_text user "${REFERENCE}" (at 0 5.8 90 unlocked) (layer "B.Fab")
+    (fp_text user "${REFERENCE}" (at 0 5.8 unlocked) (layer "B.Fab")
         (effects (font (size 1 1) (thickness 0.15)) (justify mirror))
     )
@@
     (fp_rect (start -5 5.3) (end 5 0)
       (stroke (width 0.1) (type default)) (fill none) (layer "B.Fab"))
-    (pad "1" thru_hole circle (at 2.54 6.5 270) (size 1.5 1.5) (drill 0.8) (layers "*.Cu" "*.Mask")
+    (pad "1" thru_hole circle (at 2.54 6.5 180) (size 1.5 1.5) (drill 0.8) (layers "*.Cu" "*.Mask")
       (net 23 "unconnected-(PWR0-A-Pad1)") (pinfunction "A") (pintype "passive"))
-    (pad "2" thru_hole circle (at 0 6.5 270) (size 1.5 1.5) (drill 0.8) (layers "*.Cu" "*.Mask")
+    (pad "2" thru_hole circle (at 0 6.5 180) (size 1.5 1.5) (drill 0.8) (layers "*.Cu" "*.Mask")
       (net 22 "/B+") (pinfunction "B") (pintype "passive"))
-    (pad "3" thru_hole circle (at -2.54 6.5 270) (size 1.5 1.5) (drill 0.8) (layers "*.Cu" "*.Mask")
+    (pad "3" thru_hole circle (at -2.54 6.5 180) (size 1.5 1.5) (drill 0.8) (layers "*.Cu" "*.Mask")
       (net 2 "/RAW") (pinfunction "C") (pintype "passive"))
   )
@@
   (via (at 134.72 61.849) (size 0.6) (drill 0.4) (layers "F.Cu" "B.Cu") (free) (net 1))
   (via (at 77.57 99.949) (size 0.6) (drill 0.4) (layers "F.Cu" "B.Cu") (free) (net 1))
-  (via (at 161.925 64.776839) (size 0.6) (drill 0.4) (layers "F.Cu" "B.Cu") (free) (net 1))
   (via (at 96.62 62.611) (size 0.6) (drill 0.4) (layers "F.Cu" "B.Cu") (free) (net 1))
   (via (at 96.62 100.711) (size 0.6) (drill 0.4) (layers "F.Cu" "B.Cu") (free) (net 1))
@@
   (via (at 134.72 99.949) (size 0.6) (drill 0.4) (layers "F.Cu" "B.Cu") (free) (net 1))
   (via (at 58.52 108.839) (size 0.6) (drill 0.4) (layers "F.Cu" "B.Cu") (free) (net 1))
-  (segment (start 171.025 86.635) (end 171.025 53.556839) (width 0.7) (layer "B.Cu") (net 2))
-  (segment (start 171.025 53.556839) (end 169.545 52.076839) (width 0.7) (layer "B.Cu") (net 2))
-  (segment (start 164.95 92.71) (end 171.025 86.635) (width 0.7) (layer "B.Cu") (net 2))
+  (segment (start 126.365 126.85) (end 135.515 136) (width 0.7) (layer "B.Cu") (net 2))
+  (segment (start 166.5 136) (end 171 131.5) (width 0.7) (layer "B.Cu") (net 2))
+  (segment (start 135.515 136) (end 166.5 136) (width 0.7) (layer "B.Cu") (net 2))
+  (segment (start 171 53.531839) (end 169.545 52.076839) (width 0.7) (layer "B.Cu") (net 2))
+  (segment (start 171 131.5) (end 171 53.531839) (width 0.7) (layer "B.Cu") (net 2))
   (segment (start 75.057 71.721161) (end 73.76 73.018161) (width 0.25) (layer "F.Cu") (net 3))
   (segment (start 75.057 70.478161) (end 75.057 71.721161) (width 0.25) (layer "F.Cu") (net 3))
@@
   (segment (start 169.545 57.156839) (end 170.7463 58.358139) (width 0.25) (layer "F.Cu") (net 20))
   (segment (start 170.7463 58.358139) (end 170.7463 80.7537) (width 0.25) (layer "F.Cu") (net 20))
-  (segment (start 171.05 101.35) (end 164.95 95.25) (width 0.7) (layer "B.Cu") (net 22))
-  (segment (start 167.425 137.1) (end 137.1 137.1) (width 0.7) (layer "B.Cu") (net 22))
-  (segment (start 167.425 137.1) (end 171.05 133.475) (width 0.7) (layer "B.Cu") (net 22))
-  (segment (start 137.1 137.1) (end 112.5 112.5) (width 0.7) (layer "B.Cu") (net 22))
-  (segment (start 171.05 133.475) (end 171.05 101.35) (width 0.7) (layer "B.Cu") (net 22))
+  (segment (start 97 112.5) (end 109.475 112.5) (width 0.7) (layer "B.Cu") (net 22))
+  (segment (start 109.475 112.5) (end 123.825 126.85) (width 0.7) (layer "B.Cu") (net 22))
   (zone (net 1) (net_name "GND") (layers "F&B.Cu") (hatch edge 0.5)
     (connect_pads (clearance 0.508))

Commit message: Moved some of the mounting holes around.
Parts:
- moved H1 7.79 mm to (74.2, 64.0)
- moved H0 2.00 mm to (142.9, 55.1)
- moved H2 2.00 mm to (78.2, 116.3)
Routing:
- net /KEY6: track 68.2 -> 65.5 mm
- net /KEY11: track 55.7 -> 54.3 mm
- net /KEY3: track 69.2 -> 70.0 mm
Changed lines of the file:
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@@
   (net 24 "unconnected-(U0-F5-Pad19)")
   (footprint "MountingHole:MountingHole_3.5mm" (layer "F.Cu")
-    (at 78.2 114.3)
+    (at 78.2 116.3)
     (descr "Mounting Hole 3.5mm, no annular")
     (tags "mounting hole 3.5mm no annular")
@@
   )
   (footprint "MountingHole:MountingHole_3.5mm" (layer "F.Cu")
-    (at 142.875 57.15)
+    (at 142.875 55.15)
     (descr "Mounting Hole 3.5mm, no annular")
     (tags "mounting hole 3.5mm no annular")
@@
   )
   (footprint "MountingHole:MountingHole_3.5mm" (layer "F.Cu")
-    (at 66.675 66.033161)
+    (at 74.2 64.033161)
     (descr "Mounting Hole 3.5mm, no annular")
     (tags "mounting hole 3.5mm no annular")
@@
   (segment (start 75.057 70.478161) (end 75.057 71.721161) (width 0.25) (layer "F.Cu") (net 3))
   (via (at 75.057 70.478161) (size 0.6) (drill 0.4) (layers "F.Cu" "B.Cu") (net 3))
-  (segment (start 75.057 62.943) (end 75.057 70.478161) (width 0.25) (layer "B.Cu") (net 3))
+  (segment (start 75.057 70.478161) (end 76.945 68.590161) (width 0.25) (layer "B.Cu") (net 3))
+  (segment (start 76.945 61.055) (end 85.923161 52.076839) (width 0.25) (layer "B.Cu") (net 3))
+  (segment (start 76.945 68.590161) (end 76.945 61.055) (width 0.25) (layer "B.Cu") (net 3))
   (segment (start 154.305 52.076839) (end 85.923161 52.076839) (width 0.25) (layer "B.Cu") (net 3))
-  (segment (start 85.923161 52.076839) (end 75.057 62.943) (width 0.25) (layer "B.Cu") (net 3))
   (segment (start 72.517 70.478161) (end 75.057 70.478161) (width 0.25) (layer "B.Cu") (net 3))
   (segment (start 75.057 89.528161) (end 75.057 90.771161) (width 0.25) (layer "F.Cu") (net 4))
@@
   (via (at 94.107 61.595) (size 0.6) (drill 0.4) (layers "F.Cu" "B.Cu") (net 6))
   (segment (start 91.567 61.595) (end 94.107 61.595) (width 0.25) (layer "B.Cu") (net 6))
-  (segment (start 153.688161 54) (end 101.702 54) (width 0.25) (layer "B.Cu") (net 6))
-  (segment (start 154.305 54.616839) (end 153.688161 54) (width 0.25) (layer "B.Cu") (net 6))
-  (segment (start 101.702 54) (end 94.107 61.595) (width 0.25) (layer "B.Cu") (net 6))
+  (segment (start 154.305 54.616839) (end 152.713161 53.025) (width 0.25) (layer "B.Cu") (net 6))
+  (segment (start 152.713161 53.025) (end 102.677 53.025) (width 0.25) (layer "B.Cu") (net 6))
+  (segment (start 102.677 53.025) (end 94.107 61.595) (width 0.25) (layer "B.Cu") (net 6))
   (segment (start 94.107 81.888) (end 92.81 83.185) (width 0.25) (layer "F.Cu") (net 7))
   (segment (start 94.107 80.645) (end 94.107 81.888) (width 0.25) (layer "F.Cu") (net 7))
@@
   (segment (start 110.617 62.871839) (end 113.157 62.871839) (width 0.25) (layer "F.Cu") (net 9))
   (via (at 113.157 62.871839) (size 0.6) (drill 0.4) (layers "F.Cu" "B.Cu") (net 9))
-  (segment (start 121.003839 55.025) (end 113.157 62.871839) (width 0.25) (layer "B.Cu") (net 9))
-  (segment (start 144.548343 55.818139) (end 143.755204 55.025) (width 0.25) (layer "B.Cu") (net 9))
-  (segment (start 169.545 62.236839) (end 163.1263 55.818139) (width 0.25) (layer "B.Cu") (net 9))
+  (segment (start 165.6663 58.358139) (end 117.6707 58.358139) (width 0.25) (layer "B.Cu") (net 9))
   (segment (start 113.157 61.628839) (end 111.86 60.331839) (width 0.25) (layer "B.Cu") (net 9))
-  (segment (start 163.1263 55.818139) (end 144.548343 55.818139) (width 0.25) (layer "B.Cu") (net 9))
   (segment (start 113.157 62.871839) (end 113.157 61.628839) (width 0.25) (layer "B.Cu") (net 9))
-  (segment (start 143.755204 55.025) (end 121.003839 55.025) (width 0.25) (layer "B.Cu") (net 9))
+  (segment (start 169.545 62.236839) (end 165.6663 58.358139) (width 0.25) (layer "B.Cu") (net 9))
+  (segment (start 117.6707 58.358139) (end 113.157 62.871839) (width 0.25) (layer "B.Cu") (net 9))
   (segment (start 110.617 81.921839) (end 113.157 81.921839) (width 0.25) (layer "F.Cu") (net 10))
   (via (at 113.157 81.921839) (size 0.6) (drill 0.4) (layers "F.Cu" "B.Cu") (net 10))
@@
   (segment (start 132.207 100.938) (end 130.91 102.235) (width 0.25) (layer "F.Cu") (net 14))
   (via (at 132.207 99.695) (size 0.6) (drill 0.4) (layers "F.Cu" "B.Cu") (net 14))
-  (segment (start 146.925672 97.5) (end 134.402 97.5) (width 0.25) (layer "B.Cu") (net 14))
-  (segment (start 161 80.941839) (end 161 83.425672) (width 0.25) (layer "B.Cu") (net 14))
-  (segment (start 161 83.425672) (end 146.925672 97.5) (width 0.25) (layer "B.Cu") (net 14))
   (segment (start 169.545 72.396839) (end 161 80.941839) (width 0.25) (layer "B.Cu") (net 14))
+  (segment (start 143 97.5) (end 134.402 97.5) (width 0.25) (layer "B.Cu") (net 14))
   (segment (start 134.402 97.5) (end 132.207 99.695) (width 0.25) (layer "B.Cu") (net 14))
+  (segment (start 161 80.941839) (end 159.558161 80.941839) (width 0.25) (layer "B.Cu") (net 14))
   (segment (start 129.667 99.695) (end 132.207 99.695) (width 0.25) (layer "B.Cu") (net 14))
+  (segment (start 159.558161 80.941839) (end 143 97.5) (width 0.25) (layer "B.Cu") (net 14))
   (segment (start 151.257 62.838) (end 149.96 64.135) (width 0.25) (layer "F.Cu") (net 15))
   (segment (start 151.257 61.595) (end 151.257 62.838) (width 0.25) (layer "F.Cu") (net 15))
