File: jlkfs/jlkfs_pcb/jlkfs_pcb.kicad_sch (KiCad schematic)
At the start: 38 parts, among them J0 Conn_01x02_Socket, SW0 SWITCH, SW1 SWITCH, SW10 SWITCH, SW11 SWITCH, SW12 SWITCH, SW13 SWITCH, SW14 SWITCH, SW15 SWITCH, SW16 SWITCH, SW17 SWITCH, SW18 SWITCH, SW19 SWITCH, SW2 SWITCH, SW20 SWITCH, SW21 SWITCH, SW22 SWITCH, SW23 SWITCH, SW24 SWITCH, SW25 SWITCH, SW26 SWITCH, SW27 SWITCH, SW28 SWITCH, SW29 SWITCH, SW3 SWITCH, SW4 SWITCH, SW5 SWITCH, SW6 SWITCH, SW7 SWITCH, SW8 SWITCH, SW9 SWITCH, U0 NICE!

Commit message: Routed jlkfs.
Connections:
- net KEY0 is gone; now on net COL0: U0.1 (TX)
- net KEY1 is gone; now on net COL4: U0.7 (D4)
- net KEY12 is gone; now on net COL3: U0.6 (SCL)
- net KEY13 is gone; now on net ROW3: U0.11 (B4)
- net KEY14 is gone; now on net ROW4: U0.15 (B3)
- net KEY15 is gone; now on net ROW1: U0.14 (B2)
- net KEY16 is gone; now on net COL6: U0.13 (B6)
- net KEY2 is gone; now on net ROW2: U0.12 (B5)
- net KEY3 is gone; now on net COL1: U0.2 (RX)
- net KEY4 is gone; now on net COL5: U0.8 (C6)
- net KEY7 is gone; now on net ROW0: U0.9 (D7)
- net KEY9 is gone; now on net COL2: U0.5 (SDA)
- net COL5: now reaches SW3.1, SW4.1, SW5.1, SW6.1
- net ROW2: now reaches SW1.3 (K), SW13.3 (K), SW18.3 (K), SW23.3 (K), SW27.3 (K), SW5.3 (K), SW9.3 (K)
- net COL0: now reaches SW26.1, SW27.1, SW28.1, SW29.1
- net COL2: now reaches SW16.1, SW17.1, SW18.1, SW19.1, SW20.1
- net ROW3: now reaches SW10.3 (K), SW14.3 (K), SW19.3 (K), SW2.3 (K), SW24.3 (K), SW28.3 (K), SW6.3 (K)
- net COL4: now reaches SW10.1, SW7.1, SW8.1, SW9.1
- net COL1: now reaches SW21.1, SW22.1, SW23.1, SW24.1, SW25.1
- net ROW1: now reaches SW0.3 (K), SW12.3 (K), SW17.3 (K), SW22.3 (K), SW26.3 (K), SW4.3 (K), SW8.3 (K)
- net ROW4: now reaches SW15.3 (K), SW20.3 (K), SW25.3 (K), SW29.3 (K)
- net COL3: now reaches SW11.1, SW12.1, SW13.1, SW14.1, SW15.1
- net ROW0: now reaches SW11.3 (K), SW16.3 (K), SW21.3 (K), SW3.3 (K), SW7.3 (K)
- net COL6: now reaches SW0.1, SW1.1, SW2.1
- net KEY10: no longer names the net of U0.10 (E6)
- net KEY11: no longer names the net of U0.16 (B1)
- net KEY5: no longer names the net of U0.18 (F6)
- net KEY6: no longer names the net of U0.20 (F4)
- net KEY8: no longer names the net of U0.17 (F7)
Changed lines of the file:
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@@
   (junction (at 78.74 91.44) (diameter 0) (color 0 0 0 0)
   )
+  (junction (at 162.56 119.38) (diameter 0) (color 0 0 0 0)
+  )
   (junction (at 149.86 99.06) (diameter 0) (color 0 0 0 0)
   )
@@
   (junction (at 93.98 71.12) (diameter 0) (color 0 0 0 0)
   )
+  (junction (at 190.5 119.38) (diameter 0) (color 0 0 0 0)
+  )
   (junction (at 66.04 85.09) (diameter 0) (color 0 0 0 0)
   )
@@
   (junction (at 78.74 77.47) (diameter 0) (color 0 0 0 0)
   )
+  (junction (at 22.86 105.41) (diameter 0) (color 0 0 0 0)
+  )
   (junction (at 162.56 105.41) (diameter 0) (color 0 0 0 0)
   )
@@
   (junction (at 177.8 99.06) (diameter 0) (color 0 0 0 0)
   )
+  (junction (at 78.74 105.41) (diameter 0) (color 0 0 0 0)
+  )
   (junction (at 149.86 113.03) (diameter 0) (color 0 0 0 0)
   )
@@
   (junction (at 162.56 77.47) (diameter 0) (color 0 0 0 0)
   )
+  (junction (at 134.62 119.38) (diameter 0) (color 0 0 0 0)
+  )
   (junction (at 149.86 85.09) (diameter 0) (color 0 0 0 0)
   )
+  (junction (at 106.68 119.38) (diameter 0) (color 0 0 0 0)
+  )
   (junction (at 177.8 127) (diameter 0) (color 0 0 0 0)
   )
@@
   (junction (at 134.62 105.41) (diameter 0) (color 0 0 0 0)
   )
+  (junction (at 50.8 105.41) (diameter 0) (color 0 0 0 0)
+  )
   (junction (at 149.86 127) (diameter 0) (color 0 0 0 0)
   )
@@
     (stroke (width 0) (type default))
   )
+  (wire (pts (xy 50.8 105.41) (xy 50.8 129.54))
+    (stroke (width 0) (type default))
+  )
   (wire (pts (xy 93.98 71.12) (xy 121.92 71.12))
     (stroke (width 0) (type default))
@@
     (stroke (width 0) (type default))
   )
+  (wire (pts (xy 162.56 119.38) (xy 162.56 130.81))
+    (stroke (width 0) (type default))
+  )
   (wire (pts (xy 205.74 85.09) (xy 218.44 85.09))
     (stroke (width 0) (type default))
   )
+  (wire (pts (xy 190.5 119.38) (xy 190.5 132.08))
+    (stroke (width 0) (type default))
+  )
   (wire (pts (xy 149.86 85.09) (xy 177.8 85.09))
     (stroke (width 0) (type default))
@@
     (stroke (width 0) (type default))
   )
+  (wire (pts (xy 106.68 119.38) (xy 106.68 130.81))
+    (stroke (width 0) (type default))
+  )
+  (wire (pts (xy 78.74 105.41) (xy 78.74 130.81))
+    (stroke (width 0) (type default))
+  )
   (wire (pts (xy 177.8 113.03) (xy 205.74 113.03))
     (stroke (width 0) (type default))
@@
     (stroke (width 0) (type default))
   )
+  (wire (pts (xy 134.62 119.38) (xy 134.62 130.81))
+    (stroke (width 0) (type default))
+  )
   (wire (pts (xy 78.74 77.47) (xy 78.74 91.44))
     (stroke (width 0) (type default))
@@
     (stroke (width 0) (type default))
   )
-  (wire (pts (xy 177.8 71.12) (xy 217.17 71.12))
+  (wire (pts (xy 177.8 71.12) (xy 218.44 71.12))
     (stroke (width 0) (type default))
   )
@@
     (stroke (width 0) (type default))
   )
+  (wire (pts (xy 22.86 105.41) (xy 22.86 129.54))
+    (stroke (width 0) (type default))
+  )
   (wire (pts (xy 177.8 127) (xy 205.74 127))
     (stroke (width 0) (type default))
@@
   (wire (pts (xy 78.74 63.5) (xy 78.74 77.47))
     (stroke (width 0) (type default))
-  )
-  (label "KEY10" (at 101.6 213.36 180) (fields_autoplaced)
-    (effects (font (size 1.27 1.27)) (justify right bottom))
   )
   (label "GND" (at 101.6 195.58 180) (fields_autoplaced)
     (effects (font (size 1.524 1.524)) (justify right bottom))
   )
-  (label "KEY8" (at 137.16 208.28 0) (fields_autoplaced)
-    (effects (font (size 1.27 1.27)) (justify left bottom))
+  (label "COL1" (at 101.6 193.04 180) (fields_autoplaced)
+    (effects (font (size 1.27 1.27)) (justify right bottom))
+  )
+  (label "COL3" (at 101.6 203.2 180) (fields_autoplaced)
+    (effects (font (size 1.27 1.27)) (justify right bottom))
   )
   (label "RST" (at 167.64 224.79 180) (fields_autoplaced)
+    (effects (font (size 1.27 1.27)) (justify right bottom))
+  )
+  (label "ROW3" (at 101.6 215.9 180) (fields_autoplaced)
     (effects (font (size 1.27 1.27)) (justify right bottom))
   )
@@
     (effects (font (size 1.524 1.524)) (justify right bottom))
   )
-  (label "KEY1" (at 101.6 205.74 180) (fields_autoplaced)
+  (label "ROW4" (at 218.44 127 0) (fields_autoplaced)
+    (effects (font (size 1.27 1.27)) (justify left bottom))
+  )
+  (label "COL2" (at 134.62 130.81 0) (fields_autoplaced)
+    (effects (font (size 1.27 1.27)) (justify left bottom))
+  )
+  (label "COL5" (at 101.6 208.28 180) (fields_autoplaced)
+    (effects (font (size 1.27 1.27)) (justify right bottom))
+  )
+  (label "ROW0" (at 101.6 210.82 180) (fields_autoplaced)
     (effects (font (size 1.27 1.27)) (justify right bottom))
   )
@@
     (effects (font (size 1.27 1.27)) (justify right bottom))
   )
-  (label "KEY6" (at 137.16 200.66 0) (fields_autoplaced)
-    (effects (font (size 1.27 1.27)) (justify left bottom))
-  )
   (label "GND" (at 177.8 224.79 0) (fields_autoplaced)
     (effects (font (size 1.27 1.27)) (justify left bottom))
   )
-  (label "KEY0" (at 101.6 190.5 180) (fields_autoplaced)
-    (effects (font (size 1.27 1.27)) (justify right bottom))
+  (label "ROW1" (at 137.16 215.9 0) (fields_autoplaced)
+    (effects (font (size 1.27 1.27)) (justify left bottom))
   )
   (label "RST" (at 137.16 195.58 0) (fields_autoplaced)
     (effects (font (size 1.524 1.524)) (justify left bottom))
   )
-  (label "KEY15" (at 137.16 215.9 0) (fields_autoplaced)
-    (effects (font (size 1.27 1.27)) (justify left bottom))
-  )
-  (label "KEY7" (at 101.6 210.82 180) (fields_autoplaced)
-    (effects (font (size 1.27 1.27)) (justify right bottom))
+  (label "ROW1" (at 218.44 85.09 0) (fields_autoplaced)
+    (effects (font (size 1.27 1.27)) (justify left bottom))
   )
   (label "B+" (at 176.53 195.58 0) (fields_autoplaced)
     (effects (font (size 1.27 1.27)) (justify left bottom))
   )
-  (label "KEY14" (at 137.16 213.36 0) (fields_autoplaced)
-    (effects (font (size 1.27 1.27)) (justify left bottom))
-  )
-  (label "KEY11" (at 137.16 210.82 0) (fields_autoplaced)
-    (effects (font (size 1.27 1.27)) (justify left bottom))
-  )
-  (label "KEY4" (at 101.6 208.28 180) (fields_autoplaced)
-    (effects (font (size 1.27 1.27)) (justify right bottom))
-  )
-  (label "KEY3" (at 101.6 193.04 180) (fields_autoplaced)
-    (effects (font (size 1.27 1.27)) (justify right bottom))
+  (label "COL4" (at 101.6 205.74 180) (fields_autoplaced)
+    (effects (font (size 1.27 1.27)) (justify right bottom))
+  )
+  (label "COL0" (at 101.6 190.5 180) (fields_autoplaced)
+    (effects (font (size 1.27 1.27)) (justify right bottom))
+  )
+  (label "ROW4" (at 137.16 213.36 0) (fields_autoplaced)
+    (effects (font (size 1.27 1.27)) (justify left bottom))
+  )
+  (label "ROW2" (at 218.44 99.06 0) (fields_autoplaced)
+    (effects (font (size 1.27 1.27)) (justify left bottom))
+  )
+  (label "COL2" (at 101.6 200.66 180) (fields_autoplaced)
+    (effects (font (size 1.27 1.27)) (justify right bottom))
+  )
+  (label "COL1" (at 162.56 130.81 0) (fields_autoplaced)
+    (effects (font (size 1.27 1.27)) (justify left bottom))
+  )
+  (label "ROW2" (at 101.6 218.44 180) (fields_autoplaced)
+    (effects (font (size 1.27 1.27)) (justify right bottom))
+  )
+  (label "ROW0" (at 218.44 71.12 0) (fields_autoplaced)
+    (effects (font (size 1.27 1.27)) (justify left bottom))
+  )
+  (label "ROW3" (at 218.44 113.03 0) (fields_autoplaced)
+    (effects (font (size 1.27 1.27)) (justify left bottom))
   )
   (label "B+" (at 196.85 195.58 180) (fields_autoplaced)
     (effects (font (size 1.27 1.27)) (justify right bottom))
   )
-  (label "KEY5" (at 137.16 205.74 0) (fields_autoplaced)
+  (label "COL6" (at 137.16 218.44 0) (fields_autoplaced)
+    (effects (font (size 1.27 1.27)) (justify left bottom))
+  )
+  (label "COL4" (at 78.74 130.81 0) (fields_autoplaced)
     (effects (font (size 1.27 1.27)) (justify left bottom))
   )
@@
     (effects (font (size 1.524 1.524)) (justify left bottom))
   )
-  (label "KEY12" (at 101.6 203.2 180) (fields_autoplaced)
-    (effects (font (size 1.27 1.27)) (justify right bottom))
+  (label "COL6" (at 22.86 129.54 0) (fields_autoplaced)
+    (effects (font (size 1.27 1.27)) (justify left bottom))
   )
   (label "GND" (at 137.16 193.04 0) (fields_autoplaced)
     (effects (font (size 1.524 1.524)) (justify left bottom))
   )
-  (label "KEY2" (at 101.6 218.44 180) (fields_autoplaced)
-    (effects (font (size 1.27 1.27)) (justify right bottom))
-  )
-  (label "KEY13" (at 101.6 215.9 180) (fields_autoplaced)
-    (effects (font (size 1.27 1.27)) (justify right bottom))
-  )
-  (label "KEY16" (at 137.16 218.44 0) (fields_autoplaced)
-    (effects (font (size 1.27 1.27)) (justify left bottom))
-  )
-  (label "KEY9" (at 101.6 200.66 180) (fields_autoplaced)
-    (effects (font (size 1.27 1.27)) (justify right bottom))
+  (label "COL0" (at 190.5 132.08 0) (fields_autoplaced)
+    (effects (font (size 1.27 1.27)) (justify left bottom))
+  )
+  (label "COL3" (at 106.68 130.81 0) (fields_autoplaced)
+    (effects (font (size 1.27 1.27)) (justify left bottom))
+  )
+  (label "COL5" (at 50.8 129.54 0) (fields_autoplaced)
+    (effects (font (size 1.27 1.27)) (justify left bottom))
   )
   (symbol (lib_id "symbols:ProMicro") (at 119.38 209.55 0) (unit 1)
