File: jlkfs/jlkfs_bottom/jlkfs_bottom.kicad_pcb (KiCad board)
At the start: 2 copper layers, 252 x 178.3 mm, 6 parts, among them U0 NICE!

Commit message: Fixed up the jlkfs bottom plates.
Routing:
- added copper zone on B.Cu, net (none)
- added copper zone on F.Cu, net (none)
Other:
- board size 252 x 178.3 mm -> 133.4 x 118.4 mm
Changed lines of the file:
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@@
   (gr_line (start 75.605 74.400565) (end 74.969999 74.400563)
-    (stroke (width 0.1) (type default)) (layer "Edge.Cuts"))
-  (gr_line (start 324.45157 14.505338) (end 323.885781 14.793622)
     (stroke (width 0.1) (type default)) (layer "Edge.Cuts"))
   (gr_arc (start 74.97 178.533725) (mid 73.173957 177.789779) (end 72.43 175.993726)
@@
     (effects (font (size 2 2) (thickness 0.5) bold))
   )
+  (zone (net 0) (net_name "") (layers "F&B.Cu") (hatch edge 0.5)
+    (connect_pads (clearance 0.508))
+    (min_thickness 0.25) (filled_areas_thickness no)
+    (fill yes (thermal_gap 0.5) (thermal_bridge_width 0.5) (island_removal_mode 1) (island_area_min 10))
+    (polygon
+      (pts
+        (xy 69 70)
+        (xy 209 70)
+        (xy 209 196)
+        (xy 69 196)
+      )
+    )
+  )
 )
