File: jlkfs/jlkfs_bottom_dual/jlkfs_bottom_dual.kicad_pcb (KiCad board)
At the start: 2 copper layers, 309.1 x 149.2 mm, 12 parts, among them U0 NICE!

Commit message: Fixed up the jlkfs bottom plates.
Parts:
- moved H2 15.5 mm to (75.4, 127.8)
- moved H2 15.5 mm to (344.9, 127.8)
- moved H3 15.5 mm to (164.0, 166.9)
- moved H1 15.5 mm to (103.4, 52.0)
- moved U0 15.5 mm to (88.6, 31.9)
- moved RST0 15.5 mm to (315.3, 45.6)
- moved U0 15.5 mm to (331.6, 31.9)
- moved H0 15.5 mm to (232.9, 77.0)
- moved RST0 15.5 mm to (104.9, 45.6)
- moved H0 15.5 mm to (187.4, 77.0)
- moved H3 15.5 mm to (256.3, 166.9)
- moved H1 15.5 mm to (316.8, 52.0)
Routing:
- added copper zone on B.Cu, net (none)
- added copper zone on F.Cu, net (none)
Other:
- outline, holes or cut-outs redrawn
