File: jlkfs_lp/jlkfs_lp.kicad_sch (KiCad schematic)
At the start: 38 parts, among them J0 USB_C_Receptacle_PowerOnly_6P, SW0 SWITCH, SW1 SWITCH, SW10 SWITCH, SW11 SWITCH, SW12 SWITCH, SW13 SWITCH, SW14 SWITCH, SW15 SWITCH, SW16 SWITCH, SW17 SWITCH, SW18 SWITCH, SW19 SWITCH, SW2 SWITCH, SW20 SWITCH, SW21 SWITCH, SW22 SWITCH, SW23 SWITCH, SW24 SWITCH, SW25 SWITCH, SW26 SWITCH, SW27 SWITCH, SW28 SWITCH, SW3 SWITCH, SW4 SWITCH, SW5 SWITCH, SW6 SWITCH, SW7 SWITCH, SW8 SWITCH, SW9 SWITCH, U0 RP2040

Commit message: Updates to jlkfs_lp
Parts:
- SW0: renamed from SW3; footprint footprints:kailh_choc_dual_with_side_diode -> footprints:kailh_choc_dual_with_diode
- SW12: renamed from SW1; footprint footprints:kailh_choc_dual_with_side_diode -> footprints:kailh_choc_dual_with_diode
- SW13: renamed from SW5; footprint footprints:kailh_choc_dual_with_side_diode -> footprints:kailh_choc_dual_with_diode
- SW19: renamed from SW2; footprint footprints:kailh_choc_dual_with_side_diode -> footprints:kailh_choc_dual_with_diode
- SW21: renamed from SW10; footprint footprints:kailh_choc_dual_with_side_diode -> footprints:kailh_choc_dual_with_diode
- SW25: renamed from SW15; footprint footprints:kailh_choc_dual_with_side_diode -> footprints:kailh_choc_dual_with_diode
- SW26: renamed from SW20; footprint footprints:kailh_choc_dual_with_side_diode -> footprints:kailh_choc_dual_with_diode
- SW27: renamed from SW25; footprint footprints:kailh_choc_dual_with_side_diode -> footprints:kailh_choc_dual_with_diode_15
- SW28: footprint footprints:kailh_choc_dual_with_side_diode -> footprints:kailh_choc_dual_with_diode_15
- SW5: renamed from SW0; footprint footprints:kailh_choc_dual_with_side_diode -> footprints:kailh_choc_dual_with_diode
- SW6: renamed from SW4; footprint footprints:kailh_choc_dual_with_side_diode -> footprints:kailh_choc_dual_with_diode
- renumbered SW7 to SW1, SW22 to SW10, SW26 to SW11, SW9 to SW14, SW13 to SW15, SW18 to SW16, SW23 to SW17, SW27 to SW18, SW11 to SW2, SW6 to SW20, SW14 to SW22, SW19 to SW23, SW16 to SW3, SW21 to SW4, SW8 to SW7, SW12 to SW8, SW17 to SW9
Connections:
- net COL0: no longer SW11.1
- net ROW1: now also SW11.3 (K)
- net ROW2: now also SW18.3 (K); no longer SW11.3 (K)
- net ROW3: no longer SW18.3 (K)
- net at SW10.2 (A): now also SW11.1
Other:
- moved on the sheet: SW11, SW18
