File: jlkfs_lp/jlkfs_lower/jlkfs_lower.kicad_pcb (KiCad board)
At the start: 2 copper layers, 142.5 x 133.4 mm, 38 parts, among them J0 USB_C_Receptacle_PowerOnly_6P, SW0 SWITCH, SW1 SWITCH, SW10 SWITCH, SW11 SWITCH, SW12 SWITCH, SW13 SWITCH, SW14 SWITCH, SW15 SWITCH, SW16 SWITCH, SW17 SWITCH, SW18 SWITCH, SW19 SWITCH, SW2 SWITCH, SW20 SWITCH, SW21 SWITCH, SW22 SWITCH, SW23 SWITCH, SW24 SWITCH, SW25 SWITCH, SW26 SWITCH, SW27 SWITCH, SW28 SWITCH, SW3 SWITCH, SW4 SWITCH, SW5 SWITCH, SW6 SWITCH, SW7 SWITCH, SW8 SWITCH, SW9 SWITCH, U0 RP2040

Commit message: Updated jlkfs_lp.
Parts:
- added H4: MountingHole, MountingHole:MountingHole_3.5mm, F.Cu at (240.8, 61.5)
- added H5: MountingHole, MountingHole:MountingHole_3.5mm, F.Cu at (251.7, 76.0)
- R0, R1: footprint Resistor_THT:R_Axial_DIN0204_L3.6mm_D1.6mm_P5.08mm_Horizontal -> Resistor_SMD:R_0805_2012Metric_Pad1.20x1.40mm_HandSolder
- moved H3 137.4 mm to (226.8, 28.7)
- moved H2 128.8 mm to (254.0, 90.4)
- moved RST0 81.1 mm to (205.0, 64.3)
- moved H1 43.4 mm to (228.9, 40.4)
- moved R0 37.6 mm to (202.0, 39.5), turned to 180 degrees
- moved H0 33.3 mm to (237.5, 47.5)
- moved R1 32.5 mm to (201.9, 42.0), turned to 0 degrees
- moved J0 6.85 mm to (186.0, 25.5)
- moved U0 6.85 mm to (206.0, 25.5)
- moved SW1 1.00 mm to (129.0, 48.4)
- moved SW10 1.00 mm to (186.0, 68.8)
- moved SW11 1.00 mm to (205.0, 77.8)
- moved SW14 1.00 mm to (129.0, 84.4)
- moved SW15 1.00 mm to (148.0, 75.5)
- moved SW16 1.00 mm to (167.0, 84.4)
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Connections:
- SW11 pad 1: Net-(SW10-A) -> /COL0
- U0 pad 10: unconnected-(U0-D7-Pad10) -> /ROW1
- U0 pad 11: unconnected-(U0-D8-Pad11) -> /ROW0
- U0 pad 12: /ROW4 -> /COL0
- U0 pad 13: /COL5 -> /COL1
- U0 pad 14: /COL4 -> /COL2
- U0 pad 16: /COL2 -> /COL4
- U0 pad 17: /COL1 -> /COL5
- U0 pad 18: /COL0 -> /COL6
- U0 pad 7: unconnected-(U0-D4-Pad7) -> /ROW4
- U0 pad 8: unconnected-(U0-D5-Pad8) -> /ROW3
- U0 pad 9: unconnected-(U0-D6-Pad9) -> /ROW2
Routing:
- net /COL6: track 39.4 -> 172.9 mm
- net /COL5: track 59.2 -> 162.1 mm
- net /ROW3: track 91.1 -> 182.9 mm
- net /ROW4: track 65.1 -> 152.0 mm
- net /COL4: track 59.2 -> 140.1 mm
- net /ROW2: track 112.1 -> 175.7 mm
- net /COL3: track 78.9 -> 132.0 mm
- net /ROW1: track 112.1 -> 154.7 mm
- net /ROW0: track 71.9 -> 110.8 mm
- net /COL2: track 78.9 -> 112.6 mm
- net /RST: track 0.00 -> 33.7 mm
- net VCC: track 0.00 -> 26.7 mm, vias 0 -> 2
- net /SCL: track 0.00 -> 22.9 mm, vias 0 -> 1
- net /SDA: track 0.00 -> 22.9 mm
- net /COL0: track 64.3 -> 82.5 mm
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Other:
- board size 142.5 x 133.4 mm -> 158.1 x 125.8 mm
