File: jlkfs_lp/jlkfs_lower/jlkfs_lower.kicad_sch (KiCad schematic)
At the start: 38 parts, among them J0 USB_C_Receptacle_PowerOnly_6P, SW0 SWITCH, SW1 SWITCH, SW10 SWITCH, SW11 SWITCH, SW12 SWITCH, SW13 SWITCH, SW14 SWITCH, SW15 SWITCH, SW16 SWITCH, SW17 SWITCH, SW18 SWITCH, SW19 SWITCH, SW2 SWITCH, SW20 SWITCH, SW21 SWITCH, SW22 SWITCH, SW23 SWITCH, SW24 SWITCH, SW25 SWITCH, SW26 SWITCH, SW27 SWITCH, SW28 SWITCH, SW3 SWITCH, SW4 SWITCH, SW5 SWITCH, SW6 SWITCH, SW7 SWITCH, SW8 SWITCH, SW9 SWITCH, U0 RP2040

Commit message: Updated jlkfs_lp.
Parts:
- added H4, H5: MountingHole, MountingHole:MountingHole_3.5mm, symbol Mechanical:MountingHole
- R0, R1: footprint Resistor_THT:R_Axial_DIN0204_L3.6mm_D1.6mm_P5.08mm_Horizontal -> Resistor_SMD:R_0805_2012Metric_Pad1.20x1.40mm_HandSolder
- U0: symbol symbols:elite_pi -> symbols:ProMicro
Connections:
- net COL0: now also SW11.1, U0.12 (B5); no longer U0.18 (A1)
- net COL1: now also U0.13 (B6); no longer U0.17 (A0)
- net COL2: now also U0.14 (B2); no longer U0.16 (D22)
- net COL4: now also U0.16 (B1); no longer U0.14 (D23)
- net COL5: now also U0.17 (F7); no longer U0.13 (D21)
- net COL6: now also U0.18 (F6); no longer U0.29 (D16)
- net ROW0: now also U0.11 (B4); no longer U0.28 (D15)
- net ROW1: now also U0.10 (E6); no longer U0.27 (D14)
- net ROW2: now also U0.9 (D7); no longer U0.26 (D13)
- net ROW3: now also U0.8 (C6); no longer U0.25 (D12)
- net ROW4: now also U0.7 (D4); no longer U0.12 (D9)
- net at SW10.2 (A): no longer SW11.1
