File: jlkfs_lp/jlkfs_upper/jlkfs_upper.kicad_sch (KiCad schematic)
At the start: 38 parts, among them J0 USB_C_Receptacle_PowerOnly_6P, SW0 SWITCH, SW1 SWITCH, SW10 SWITCH, SW11 SWITCH, SW12 SWITCH, SW13 SWITCH, SW14 SWITCH, SW15 SWITCH, SW16 SWITCH, SW17 SWITCH, SW18 SWITCH, SW19 SWITCH, SW2 SWITCH, SW20 SWITCH, SW21 SWITCH, SW22 SWITCH, SW23 SWITCH, SW24 SWITCH, SW25 SWITCH, SW26 SWITCH, SW27 SWITCH, SW28 SWITCH, SW3 SWITCH, SW4 SWITCH, SW5 SWITCH, SW6 SWITCH, SW7 SWITCH, SW8 SWITCH, SW9 SWITCH, U0 RP2040

Commit message: Updated jlkfs_lp.
Parts:
- removed J0: USB_C_Receptacle_PowerOnly_6P, footprints:USB4515, symbol Connector:USB_C_Receptacle_PowerOnly_6P
- removed R0, R1: R, Resistor_THT:R_Axial_DIN0204_L3.6mm_D1.6mm_P5.08mm_Horizontal, symbol Device:R
- removed RST0: SW_Push, footprints:reset_button, symbol Switch:SW_Push
- removed SW0, SW1, SW12, SW13, SW14, SW15, SW19, SW2, SW20, SW21, SW22, SW25, SW5, SW6, SW7, SW8: SWITCH, footprints:kailh_choc_dual_with_diode, symbol symbols:SWITCH_WITH_DIODE
- removed U0: RP2040, footprints:pro_micro_castellated, symbol symbols:elite_pi
