File: jlkws/jlkws_pcb/jlkws_pcb.kicad_pcb (KiCad board)
At the start: 2 copper layers, 133.3 x 118.4 mm, 38 parts, among them J0 Conn_01x02_Socket, SW0 SWITCH, SW1 SWITCH, SW10 SWITCH, SW11 SWITCH, SW12 SWITCH, SW13 SWITCH, SW14 SWITCH, SW15 SWITCH, SW16 SWITCH, SW17 SWITCH, SW18 SWITCH, SW19 SWITCH, SW2 SWITCH, SW20 SWITCH, SW21 SWITCH, SW22 SWITCH, SW23 SWITCH, SW24 SWITCH, SW25 SWITCH, SW26 SWITCH, SW27 SWITCH, SW28 SWITCH, SW29 SWITCH, SW3 SWITCH, SW4 SWITCH, SW5 SWITCH, SW6 SWITCH, SW7 SWITCH, SW8 SWITCH, SW9 SWITCH, U0 NICE!

Commit message: Adding jst inter-board connector to jlkws.
Parts:
- removed PWR0: POWER, footprints:power_switch_1
- J0: value Conn_01x02_Socket -> Conn_01x03; footprint Connector_PinHeader_2.54mm:PinHeader_1x02_P2.54mm_Vertical -> Connector_JST:JST_PH_S3B-PH-K_1x03_P2.00mm_Horizontal
- U0: footprint footprints:nice!nano -> footprints:rp2040_pro_micro
- moved J0 23.4 mm to (209.6, 28.2)
Connections:
- J0 pad 1: GND -> /TX
- J0 pad 2: /B+ -> /GND
- RST0 pad 1: GND -> /GND
- U0 pad 19: unconnected-(U0-F5-Pad19) -> /TX
- U0 pad 23: GND -> /GND
- U0 pad 3: GND -> /GND
- U0 pad 4: GND -> /GND
Routing:
- net /TX: track 0.00 -> 133.0 mm
- net /RAW: track 85.0 -> 128.9 mm
- net /B+: track 25.7 -> 0.00 mm
- net /ROW1: track 197.3 -> 183.0 mm
- net /ROW0: track 117.9 -> 121.0 mm
- net /COL1: track 198.4 -> 197.8 mm
- net /COL0: track 212.8 -> 212.2 mm
- net /COL2: track 175.0 -> 174.4 mm
- net GND: vias 36 -> 0
- net /GND: vias 0 -> 36
- added copper zone on B.Cu, net /GND
- added copper zone on F.Cu, net /GND
- removed copper zone on B.Cu, net GND
- removed copper zone on F.Cu, net GND
Other:
- board size 133.3 x 118.4 mm -> 133.3 x 127.1 mm
