File: olk/olk_pcb/olk_pcb.kicad_pcb (KiCad board)
At the start: 2 copper layers, 266.7 x 95.2 mm, 66 parts, among them SW0 SWITCH, SW1 SWITCH, SW10 SWITCH, SW11 SWITCH, SW12 SWITCH, SW13 SWITCH, SW14 SWITCH, SW15 SWITCH, SW16 SWITCH, SW17 SWITCH, SW18 SWITCH, SW19 SWITCH, SW2 SWITCH, SW20 SWITCH, SW21 SWITCH, SW22 SWITCH, SW23 SWITCH, SW24 SWITCH, SW25 SWITCH, SW26 SWITCH, SW27 SWITCH, SW28 SWITCH, SW29 SWITCH, SW3 SWITCH, SW30 SWITCH, SW31 SWITCH, SW32 SWITCH, SW33 SWITCH, SW34 SWITCH, SW35 SWITCH, SW36 SWITCH, SW37 SWITCH, SW38 SWITCH, SW39 SWITCH, SW4 SWITCH, SW40 SWITCH, SW41 SWITCH, SW42 SWITCH, SW43 SWITCH, SW44 SWITCH, SW45 SWITCH, SW46 SWITCH, SW47 SWITCH, SW48 SWITCH, SW49 SWITCH, SW5 SWITCH, SW50 SWITCH, SW51 SWITCH, SW52 SWITCH, SW53 SWITCH, SW54 SWITCH, SW55 SWITCH, SW6 SWITCH, SW7 SWITCH, SW8 SWITCH, SW9 SWITCH, U0 NICE!

Commit message: Completed a lot of the per-switch routing on olk.
Parts:
- moved H2 5.65 mm to (94.0, 121.9)
- moved H5 5.65 mm to (246.4, 121.9)
- moved H6 5.65 mm to (170.2, 121.9)
- moved H7 5.65 mm to (322.6, 121.9)
- moved SW1 5.65 mm to (89.2, 74.3)
- moved SW14 5.65 mm to (146.4, 74.3)
- moved SW24 5.65 mm to (184.5, 74.3)
- moved SW27 5.65 mm to (198.8, 126.7)
- moved SW29 5.65 mm to (232.1, 74.3)
- moved SW32 5.65 mm to (217.8, 126.7)
- moved SW34 5.65 mm to (251.1, 74.3)
- moved SW39 5.65 mm to (270.2, 74.3)
- moved SW44 5.65 mm to (289.2, 74.3)
- moved SW49 5.65 mm to (308.3, 74.3)
- moved SW0 5.65 mm to (89.2, 55.2)
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Routing:
- net /ROW3: track 0.00 -> 274.3 mm, vias 0 -> 12
- net /ROW0: track 0.00 -> 269.9 mm, vias 0 -> 12
- net /ROW2: track 0.00 -> 268.6 mm, vias 0 -> 12
- net /ROW1: track 0.00 -> 268.0 mm, vias 0 -> 12
- net /ROW4: track 0.00 -> 178.9 mm, vias 0 -> 8
- net /COL5: track 0.00 -> 88.2 mm
- net /COL4: track 0.00 -> 86.2 mm
- net /COL6: track 0.00 -> 84.1 mm
- net /COL7: track 0.00 -> 84.1 mm
- net /COL9: track 0.00 -> 82.1 mm
- net /COL2: track 0.00 -> 82.1 mm
- net /COL8: track 0.00 -> 82.1 mm
- net /COL3: track 0.00 -> 82.1 mm
- net /COL10: track 0.00 -> 59.1 mm
- net /COL1: track 0.00 -> 59.1 mm
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- added copper zone on B.Cu, net /GND
- added copper zone on F.Cu, net /GND
Other:
- outline, holes or cut-outs redrawn

Commit message: Changed the shape of the olk_pcb.
Parts:
- added H8: MountingHole, MountingHole:MountingHole_3.5mm, F.Cu at (193.7, 108.0)
- moved H6 43.4 mm to (127.0, 117.5)
- moved H2 27.7 mm to (79.4, 98.4)
- moved H7 27.7 mm to (308.0, 98.4)
- moved SW13 15.3 mm to (131.8, 50.8)
- moved SW14 15.3 mm to (131.8, 69.8)
- moved SW32 15.3 mm to (203.2, 122.2)
- moved SW33 15.3 mm to (236.5, 50.8)
- moved SW34 15.3 mm to (236.5, 69.8)
- moved SW43 15.3 mm to (274.6, 50.8)
- moved SW44 15.3 mm to (274.6, 69.8)
- moved SW48 15.3 mm to (293.7, 50.8)
- moved SW49 15.3 mm to (293.7, 69.8)
- moved H1 15.3 mm to (303.2, 60.3)
- moved H3 15.3 mm to (227.0, 60.3)
- moved SW12 15.3 mm to (117.5, 127.0)
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Other:
- outline, holes or cut-outs redrawn

Commit message: Changed olk to more ortholinear grid.
Parts:
- moved RST0 35.4 mm to (208.0, 47.0), turned to -90 degrees
- moved H1 4.76 mm to (308.0, 60.3)
- moved H3 4.76 mm to (231.8, 60.3)
- moved H4 4.76 mm to (155.6, 60.3)
- moved SW23 4.76 mm to (165.1, 50.8)
- moved SW24 4.76 mm to (165.1, 69.8)
- moved SW25 4.76 mm to (165.1, 88.9)
- moved SW33 4.76 mm to (241.3, 50.8)
- moved SW34 4.76 mm to (241.3, 69.8)
- moved SW35 4.76 mm to (241.3, 88.9)
- moved SW38 4.76 mm to (260.4, 50.8)
- moved SW39 4.76 mm to (260.4, 69.8)
- moved SW40 4.76 mm to (260.4, 88.9)
- moved H0 4.76 mm to (79.4, 60.3)
- moved SW0 4.76 mm to (69.8, 50.8)
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Routing:
- net /ROW1: track 268.0 -> 274.6 mm
- net /RST: track 0.00 -> 6.67 mm
- net /ROW2: track 268.6 -> 274.6 mm
- net /ROW0: track 269.9 -> 275.1 mm
- net /ROW4: track 178.9 -> 174.3 mm
- net /COL4: track 86.2 -> 83.0 mm
- net /COL5: track 88.2 -> 85.2 mm
- net /COL11: track 59.1 -> 57.1 mm
- net /COL7: track 84.1 -> 82.1 mm
- net /COL1: track 59.1 -> 57.1 mm
- net /COL0: track 59.1 -> 57.1 mm
- net /COL9: track 82.1 -> 80.1 mm
- net /COL8: track 82.1 -> 80.1 mm
- net /COL6: track 84.1 -> 82.1 mm
- net /COL10: track 59.1 -> 57.1 mm
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Other:
- outline, holes or cut-outs redrawn

Commit message: Routed the olk.
Parts:
- moved SW43 2.01 mm to (280.0, 52.7)
- moved SW44 2.01 mm to (280.0, 71.8)
- moved SW45 2.01 mm to (280.0, 90.8)
- moved SW46 2.01 mm to (280.0, 109.9)
- moved SW23 2.01 mm to (165.7, 52.7)
- moved SW24 2.01 mm to (165.7, 71.8)
- moved SW25 2.01 mm to (165.7, 90.8)
- moved SW26 2.01 mm to (165.7, 109.9)
- moved SW32 2.01 mm to (203.8, 124.1)
- moved SW37 2.01 mm to (227.6, 128.9)
- moved SW42 2.01 mm to (251.5, 128.9)
- moved H2 2.01 mm to (80.0, 100.3)
- moved H6 2.01 mm to (127.6, 119.4)
- moved SW0 2.01 mm to (70.5, 52.7)
- moved SW1 2.01 mm to (70.5, 71.8)
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Connections:
- U0 pad 10: unconnected-(U0-E6-Pad10) -> /COL2
- U0 pad 11: unconnected-(U0-B4-Pad11) -> /COL1
- U0 pad 12: unconnected-(U0-B5-Pad12) -> /COL0
- U0 pad 13: unconnected-(U0-B6-Pad13) -> /COL11
- U0 pad 14: unconnected-(U0-B2-Pad14) -> /COL10
- U0 pad 15: unconnected-(U0-B3-Pad15) -> /COL9
- U0 pad 16: unconnected-(U0-B1-Pad16) -> /COL8
- U0 pad 17: unconnected-(U0-F7-Pad17) -> /COL7
- U0 pad 18: unconnected-(U0-F6-Pad18) -> /COL6
- U0 pad 19: unconnected-(U0-F5-Pad19) -> /ROW4
- U0 pad 2: unconnected-(U0-RX-Pad2) -> /ROW1
- U0 pad 20: unconnected-(U0-F4-Pad20) -> /ROW0
- U0 pad 5: unconnected-(U0-SDA-Pad5) -> /ROW2
- U0 pad 6: unconnected-(U0-SCL-Pad6) -> /ROW3
- U0 pad 7: unconnected-(U0-D4-Pad7) -> /COL5
- U0 pad 8: unconnected-(U0-C6-Pad8) -> /COL4
- U0 pad 9: unconnected-(U0-D7-Pad9) -> /COL3
Routing:
- net /COL0: track 57.1 -> 183.6 mm, vias 0 -> 2
- net /COL11: track 57.1 -> 169.4 mm, vias 0 -> 2
- net /COL1: track 57.1 -> 169.3 mm, vias 0 -> 2
- net /COL10: track 57.1 -> 154.9 mm, vias 0 -> 2
- net /COL2: track 80.7 -> 177.5 mm, vias 0 -> 2
- net /COL9: track 80.1 -> 162.8 mm, vias 0 -> 2
- net /COL3: track 80.4 -> 162.0 mm, vias 0 -> 2
- net /ROW4: track 174.3 -> 249.5 mm
- net /COL8: track 80.1 -> 147.6 mm, vias 0 -> 2
- net /COL4: track 83.0 -> 149.5 mm, vias 0 -> 2
- net /ROW3: track 274.6 -> 331.5 mm, vias 12 -> 13
- net /COL7: track 82.1 -> 134.5 mm, vias 0 -> 2
- net /COL5: track 85.2 -> 136.7 mm, vias 0 -> 2
- net /ROW2: track 274.6 -> 315.3 mm, vias 12 -> 13
- net /COL6: track 82.1 -> 119.4 mm, vias 0 -> 2
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
Commit message: Switching olk to castellated pro micro footprint.
Parts:
- U0: footprint footprints:nice!nano -> footprints:pro_micro_castellated
- renumbered H2 to H1, H4 to H2, H6 to H3, H1 to H4, H3 to H5, H5 to H6, SW4 to SW1, SW48 to SW10, SW52 to SW11, SW1 to SW12, SW5 to SW13, SW9 to SW14, SW14 to SW15, SW19 to SW16, SW24 to SW17, SW29 to SW18, SW34 to SW19, SW8 to SW2, SW39 to SW20, SW44 to SW21, SW49 to SW22, SW53 to SW23, SW2 to SW24, SW6 to SW25, SW10 to SW26, SW15 to SW27, SW20 to SW28, SW25 to SW29, SW13 to SW3, SW35 to SW31, SW40 to SW32, SW45 to SW33, SW50 to SW34, SW54 to SW35, SW3 to SW36, SW7 to SW37, SW11 to SW38, SW16 to SW39, SW18 to SW4, SW21 to SW40, SW26 to SW41, SW31 to SW42, SW36 to SW43, SW41 to SW44, SW46 to SW45, SW51 to SW46, SW55 to SW47, SW12 to SW48, SW17 to SW49, SW23 to SW5, SW22 to SW50, SW27 to SW51, SW32 to SW52, SW37 to SW53, SW42 to SW54, SW47 to SW55, SW28 to SW6, SW33 to SW7, SW38 to SW8, SW43 to SW9

Commit message: Moved the keys around again on olk.
Parts:
- moved H8 24.1 mm to (188.9, 133.3)
- moved SW51 21.3 mm to (174.6, 142.9)
- moved SW48 20.4 mm to (103.2, 142.9)
- moved SW49 20.4 mm to (122.2, 142.9)
- moved SW50 20.4 mm to (146.1, 142.9)
- moved SW52 18.7 mm to (203.2, 142.9)
- moved H4 17.3 mm to (298.4, 76.2)
- moved H7 17.3 mm to (298.4, 114.3)
- moved SW20 17.3 mm to (250.8, 85.7)
- moved SW21 17.3 mm to (269.9, 85.7)
- moved SW32 17.3 mm to (250.8, 104.8)
- moved SW33 17.3 mm to (269.9, 104.8)
- moved SW44 17.3 mm to (250.8, 123.8)
- moved SW45 17.3 mm to (269.9, 123.8)
- moved SW8 17.3 mm to (250.8, 66.7)
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Routing:
- net /ROW4: track 249.5 -> 266.0 mm, vias 8 -> 9
- net /COL4: track 149.5 -> 138.0 mm
- net /COL7: track 134.5 -> 123.8 mm
- net /ROW0: track 276.3 -> 266.1 mm
- net /COL5: track 136.7 -> 126.9 mm
- net /ROW3: track 331.5 -> 321.9 mm
- net /ROW2: track 315.3 -> 305.8 mm
- net /ROW1: track 304.1 -> 294.6 mm
- net /COL2: track 177.5 -> 170.2 mm
- net /COL3: track 162.0 -> 155.1 mm
- net /COL6: track 119.4 -> 112.7 mm
- net /COL9: track 162.8 -> 156.0 mm
- net /COL8: track 147.6 -> 140.9 mm
- net /COL1: track 169.3 -> 164.3 mm
- net /COL10: track 154.9 -> 150.2 mm
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Other:
- board size 266.7 x 95.2 mm -> 257.2 x 95.2 mm
