File: olk/olk_pcb/olk_pcb.kicad_pcb (KiCad board)
At the start: 2 copper layers, 257.2 x 95.2 mm, 67 parts, among them SW0 SWITCH, SW1 SWITCH, SW10 SWITCH, SW11 SWITCH, SW12 SWITCH, SW13 SWITCH, SW14 SWITCH, SW15 SWITCH, SW16 SWITCH, SW17 SWITCH, SW18 SWITCH, SW19 SWITCH, SW2 SWITCH, SW20 SWITCH, SW21 SWITCH, SW22 SWITCH, SW23 SWITCH, SW24 SWITCH, SW25 SWITCH, SW26 SWITCH, SW27 SWITCH, SW28 SWITCH, SW29 SWITCH, SW3 SWITCH, SW30 SWITCH, SW31 SWITCH, SW32 SWITCH, SW33 SWITCH, SW34 SWITCH, SW35 SWITCH, SW36 SWITCH, SW37 SWITCH, SW38 SWITCH, SW39 SWITCH, SW4 SWITCH, SW40 SWITCH, SW41 SWITCH, SW42 SWITCH, SW43 SWITCH, SW44 SWITCH, SW45 SWITCH, SW46 SWITCH, SW47 SWITCH, SW48 SWITCH, SW49 SWITCH, SW5 SWITCH, SW50 SWITCH, SW51 SWITCH, SW52 SWITCH, SW53 SWITCH, SW54 SWITCH, SW55 SWITCH, SW6 SWITCH, SW7 SWITCH, SW8 SWITCH, SW9 SWITCH, U0 NICE!

Commit message: Adding option for battery in olk_pcb.
Parts:
- added J0: Conn_01x02_Socket, Connector_PinHeader_2.54mm:PinHeader_1x02_P2.54mm_Vertical, F.Cu at (176.6, 123.8)
- added PWR0: POWER, footprints:power_switch_1, F.Cu at (188.9, 152.4)
- renumbered H2 to H1, H5 to H2, H4 to H3, H1 to H4, H7 to H5, H3 to H6, H8 to H7, H6 to H8
Connections:
- net /GND renamed GND
- U0 pad 24: unconnected-(U0-RAW-Pad24) -> /RAW
Routing:
- net /RAW: track 0.00 -> 91.0 mm
- net /B+: track 0.00 -> 23.6 mm
