File: olk/olk_top/olk_top.kicad_pcb (KiCad board)
At the start: 2 copper layers, 266.7 x 95.2 mm, 64 parts, among them SW0 SWITCH, SW1 SWITCH, SW10 SWITCH, SW11 SWITCH, SW12 SWITCH, SW13 SWITCH, SW14 SWITCH, SW15 SWITCH, SW16 SWITCH, SW17 SWITCH, SW18 SWITCH, SW19 SWITCH, SW2 SWITCH, SW20 SWITCH, SW21 SWITCH, SW22 SWITCH, SW23 SWITCH, SW24 SWITCH, SW25 SWITCH, SW26 SWITCH, SW27 SWITCH, SW28 SWITCH, SW29 SWITCH, SW3 SWITCH, SW30 SWITCH, SW31 SWITCH, SW32 SWITCH, SW33 SWITCH, SW34 SWITCH, SW35 SWITCH, SW36 SWITCH, SW37 SWITCH, SW38 SWITCH, SW39 SWITCH, SW4 SWITCH, SW40 SWITCH, SW41 SWITCH, SW42 SWITCH, SW43 SWITCH, SW44 SWITCH, SW45 SWITCH, SW46 SWITCH, SW47 SWITCH, SW48 SWITCH, SW49 SWITCH, SW5 SWITCH, SW50 SWITCH, SW51 SWITCH, SW52 SWITCH, SW53 SWITCH, SW54 SWITCH, SW55 SWITCH, SW6 SWITCH, SW7 SWITCH, SW8 SWITCH, SW9 SWITCH

Commit message: Adding missing footprint.
Parts:
- moved SW52 8.84 mm to (335.6, 58.4)
- moved SW53 8.84 mm to (335.6, 77.5)
- moved SW54 8.84 mm to (335.6, 96.5)
- moved SW18 8.84 mm to (173.7, 58.4)
- moved SW16 8.84 mm to (149.9, 115.6)
- moved SW19 8.84 mm to (173.7, 77.5)
- moved SW20 8.84 mm to (173.7, 96.5)
- moved SW31 8.84 mm to (245.1, 115.6)
- moved SW36 8.84 mm to (264.2, 115.6)
- moved SW7 8.84 mm to (111.8, 115.6)
- moved SW12 8.84 mm to (140.3, 134.6)
- moved SW17 8.84 mm to (159.4, 134.6)
- moved SW22 8.84 mm to (183.2, 134.6)
- moved SW37 8.84 mm to (249.9, 134.6)
- moved SW42 8.84 mm to (273.7, 134.6)
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Other:
- outline, holes or cut-outs redrawn

Commit message: Adding logo to olk top, and to library.
Parts:
- added REF**: JL Logo, footprints:JL Logo, F.Cu at (209.9, 80.6)
- moved SW18 9.21 mm to (167.0, 52.1)
- moved SW38 9.21 mm to (271.8, 52.1)
- moved SW43 9.21 mm to (290.8, 52.1)
- moved SW48 9.21 mm to (309.9, 52.1)
- moved SW52 9.21 mm to (328.9, 52.1)
- moved H1 9.21 mm to (319.4, 61.6)
- moved SW12 9.21 mm to (133.7, 128.3)
- moved SW16 9.21 mm to (143.2, 109.2)
- moved SW19 9.21 mm to (167.0, 71.1)
- moved SW20 9.21 mm to (167.0, 90.2)
- moved SW26 9.21 mm to (181.3, 109.2)
- moved SW31 9.21 mm to (238.4, 109.2)
- moved SW36 9.21 mm to (257.5, 109.2)
- moved SW39 9.21 mm to (271.8, 71.1)
- moved SW40 9.21 mm to (271.8, 90.2)
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Other:
- outline, holes or cut-outs redrawn

Commit message: Updated the top shape to match the pcb.
Parts:
- added H8: MountingHole, MountingHole:MountingHole_2.2mm_M2_ISO7380_Pad, F.Cu at (203.2, 110.5)
- moved H6 35.3 mm to (136.5, 120.0)
- moved H5 21.9 mm to (269.9, 120.0)
- moved H7 19.0 mm to (317.5, 101.0)
- moved H2 19.0 mm to (88.9, 101.0)
- moved REF** 7.41 mm to (203.2, 77.4)
- moved SW32 6.79 mm to (212.7, 124.8)
- moved H3 6.79 mm to (236.5, 62.9)
- moved SW13 6.79 mm to (141.3, 53.3)
- moved SW23 6.79 mm to (179.4, 53.3)
- moved SW28 6.79 mm to (227.0, 53.3)
- moved SW48 6.79 mm to (303.2, 53.3)
- moved SW52 6.79 mm to (322.3, 53.3)
- moved SW14 6.79 mm to (141.3, 72.4)
- moved SW15 6.79 mm to (141.3, 91.4)
- moved SW21 6.79 mm to (155.6, 110.5)
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Other:
- outline, holes or cut-outs redrawn

Commit message: Changed olk to more ortholinear grid.
Parts:
- moved H1 9.03 mm to (311.1, 54.0)
- moved SW38 9.03 mm to (263.5, 44.5)
- moved SW39 9.03 mm to (263.5, 63.5)
- moved SW40 9.03 mm to (263.5, 82.5)
- moved SW43 9.03 mm to (282.6, 44.5)
- moved SW44 9.03 mm to (282.6, 63.5)
- moved SW45 9.03 mm to (282.6, 82.5)
- moved SW46 9.03 mm to (287.3, 101.6)
- moved SW51 9.03 mm to (306.4, 101.6)
- moved H2 9.03 mm to (87.3, 92.1)
- moved H3 9.03 mm to (234.9, 54.0)
- moved H4 9.03 mm to (168.3, 54.0)
- moved H6 9.03 mm to (134.9, 111.1)
- moved SW0 9.03 mm to (82.5, 44.5)
- moved SW1 9.03 mm to (82.5, 63.5)
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Other:
- board size 266.7 x 95.2 mm -> 266.7 x 95.3 mm

Commit message: Updated olk_top to match the new layout.
Parts:
- moved H8 34.2 mm to (188.9, 133.3)
- moved SW51 32.1 mm to (174.6, 142.9)
- moved SW49 31.4 mm to (122.2, 142.9)
- moved SW48 31.4 mm to (103.2, 142.9)
- moved SW50 31.4 mm to (146.1, 142.9)
- moved REF** 29.6 mm to (188.9, 95.2)
- moved SW44 28.3 mm to (250.8, 123.8)
- moved H7 28.3 mm to (298.4, 114.3)
- moved SW42 28.3 mm to (212.7, 123.8)
- moved SW43 28.3 mm to (231.8, 123.8)
- moved H3 28.3 mm to (117.5, 133.3)
- moved SW45 28.3 mm to (269.9, 123.8)
- moved SW46 28.3 mm to (288.9, 123.8)
- moved SW47 28.3 mm to (308.0, 123.8)
- moved SW52 28.1 mm to (203.2, 142.9)
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- renumbered H2 to H1, H4 to H2, H6 to H3, H1 to H4, H3 to H5, H5 to H6, SW4 to SW1, SW48 to SW10, SW52 to SW11, SW1 to SW12, SW5 to SW13, SW9 to SW14, SW14 to SW15, SW19 to SW16, SW24 to SW17, SW29 to SW18, SW34 to SW19, SW8 to SW2, SW39 to SW20, SW44 to SW21, SW49 to SW22, SW53 to SW23, SW2 to SW24, SW6 to SW25, SW10 to SW26, SW15 to SW27, SW20 to SW28, SW25 to SW29, SW13 to SW3, SW35 to SW31, SW40 to SW32, SW45 to SW33, SW50 to SW34, SW54 to SW35, SW3 to SW36, SW7 to SW37, SW11 to SW38, SW16 to SW39, SW18 to SW4, SW21 to SW40, SW26 to SW41, SW31 to SW42, SW36 to SW43, SW41 to SW44, SW46 to SW45, SW51 to SW46, SW55 to SW47, SW12 to SW48, SW17 to SW49, SW23 to SW5, SW22 to SW50, SW27 to SW51, SW32 to SW52, SW37 to SW53, SW42 to SW54, SW47 to SW55, SW28 to SW6, SW33 to SW7, SW38 to SW8, SW43 to SW9
Routing:
- removed copper zone on B.Cu, net (none)
- removed copper zone on F.Cu, net (none)
Other:
- board size 266.7 x 95.3 mm -> 257.2 x 95.2 mm
