File: olk/olk_bottom/olk_bottom.kicad_pcb (KiCad board)
At the start: 2 copper layers, 257.2 x 95.2 mm, 10 parts

Commit message: Adding option for battery in olk_pcb.
Other:
- board text added: "0"
- board text added: "1"
Changed lines of the file:
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@@
 		(end 107.6 79.375)
 		(stroke
-			(width 0.2)
+			(width 0.5)
 			(type solid)
 		)
@@
 		(end 107.6 135.575)
 		(stroke
-			(width 0.2)
+			(width 0.5)
 			(type solid)
 		)
@@
 		(end 140.9375 154.625)
 		(stroke
-			(width 0.2)
+			(width 0.5)
 			(type solid)
 		)
@@
 		(end 226.1875 79.375)
 		(stroke
-			(width 0.2)
+			(width 0.5)
 			(type solid)
 		)
@@
 		(end 226.1875 154.625)
 		(stroke
-			(width 0.2)
+			(width 0.5)
 			(type solid)
 		)
@@
 		(end 311.4375 154.625)
 		(stroke
-			(width 0.2)
+			(width 0.5)
 			(type solid)
 		)
@@
 		(end 344.775 79.375)
 		(stroke
-			(width 0.2)
+			(width 0.5)
 			(type solid)
 		)
@@
 		(end 344.775 135.575)
 		(stroke
-			(width 0.2)
+			(width 0.5)
 			(type solid)
 		)
@@
 		(layer "Edge.Cuts")
 	)
+	(gr_text "0"
+		(at 215.425 161.625 0)
+		(layer "B.SilkS")
+		(effects
+			(font
+				(size 2 2)
+				(thickness 0.5)
+				(bold yes)
+			)
+			(justify mirror)
+		)
+	)
+	(gr_text "1"
+		(at 224.95 161.625 0)
+		(layer "B.SilkS")
+		(effects
+			(font
+				(size 2 2)
+				(thickness 0.5)
+				(bold yes)
+			)
+			(justify mirror)
+		)
+	)
 	(embedded_fonts no)
