File: jlol/jlol.kicad_sch (KiCad schematic)
At the start: 65 parts, among them SW0 SWITCH, SW1 SWITCH, SW10 SWITCH, SW11 SWITCH, SW12 SWITCH, SW13 SWITCH, SW14 SWITCH, SW15 SWITCH, SW16 SWITCH, SW17 SWITCH, SW18 SWITCH, SW19 SWITCH, SW2 SWITCH, SW20 SWITCH, SW21 SWITCH, SW22 SWITCH, SW23 SWITCH, SW24 SWITCH, SW25 SWITCH, SW26 SWITCH, SW27 SWITCH, SW28 SWITCH, SW29 SWITCH, SW3 SWITCH, SW30 SWITCH, SW31 SWITCH, SW32 SWITCH, SW33 SWITCH, SW34 SWITCH, SW35 SWITCH, SW36 SWITCH, SW37 SWITCH, SW38 SWITCH, SW39 SWITCH, SW4 SWITCH, SW40 SWITCH, SW41 SWITCH, SW42 SWITCH, SW43 SWITCH, SW44 SWITCH, SW45 SWITCH, SW46 SWITCH, SW47 SWITCH, SW48 SWITCH, SW49 SWITCH, SW5 SWITCH, SW50 SWITCH, SW51 SWITCH, SW52 SWITCH, SW53 SWITCH, SW54 SWITCH, SW55 SWITCH, SW6 SWITCH, SW7 SWITCH, SW8 SWITCH, SW9 SWITCH

Commit message: Adding jlol v2.
Parts:
- added J0: Conn_01x02_Socket, footprints:jst_ph, symbol Connector:Conn_01x02_Socket
- added PWR0: POWER, footprints:power_switch_1, symbol Switch:SW_SPDT
- added RST0: RESET, footprints:reset_button, symbol Switch:SW_SPST
- added U0: NICE!, footprints:nice!nano, symbol symbols:ProMicro
- H0: footprint MountingHole:MountingHole_2.2mm_M2_ISO7380_Pad -> MountingHole:MountingHole_3.5mm
- H1: renamed from H2; footprint MountingHole:MountingHole_2.2mm_M2_ISO7380_Pad -> MountingHole:MountingHole_3.5mm
- H2: renamed from H5; footprint MountingHole:MountingHole_2.2mm_M2_ISO7380_Pad -> MountingHole:MountingHole_3.5mm
- H3: renamed from H4; footprint MountingHole:MountingHole_2.2mm_M2_ISO7380_Pad -> MountingHole:MountingHole_3.5mm
- H4: renamed from H1; footprint MountingHole:MountingHole_2.2mm_M2_ISO7380_Pad -> MountingHole:MountingHole_3.5mm
- H5: renamed from H7; footprint MountingHole:MountingHole_2.2mm_M2_ISO7380_Pad -> MountingHole:MountingHole_3.5mm
- H6: renamed from H3; footprint MountingHole:MountingHole_2.2mm_M2_ISO7380_Pad -> MountingHole:MountingHole_3.5mm
- H7: renamed from H8; footprint MountingHole:MountingHole_2.2mm_M2_ISO7380_Pad -> MountingHole:MountingHole_3.5mm
- H8: renamed from H6; footprint MountingHole:MountingHole_2.2mm_M2_ISO7380_Pad -> MountingHole:MountingHole_3.5mm
- SW0, SW1, SW10, SW11, SW12, SW13, SW14, SW15, SW16, SW17, SW18, SW19, SW2, SW20, SW21, SW22, SW23, SW24, SW25, SW26, SW27, SW28, SW29, SW3, SW30, SW31, SW32, SW33, SW34, SW35, SW36, SW37, SW38, SW39, SW4, SW40, SW41, SW42, SW43, SW44, SW45, SW46, SW47, SW48, SW49, SW5, SW50, SW51, SW52, SW53, SW54, SW55, SW6, SW7, SW8, SW9: footprint footprints:cherry_plate -> footprints:cherry_hotswap_with_thru_diode
Connections:
- net COL0: now also U0.13 (B6)
- net COL1: now also U0.14 (B2)
- net COL10: now also U0.11 (B4)
- net COL11: now also U0.12 (B5)
- net COL2: now also U0.15 (B3)
- net COL3: now also U0.16 (B1)
- net COL4: now also U0.17 (F7)
- net COL5: now also U0.18 (F6)
- net COL6: now also U0.7 (D4)
- net COL7: now also U0.8 (C6)
- net COL8: now also U0.9 (D7)
- net COL9: now also U0.10 (E6)
- net ROW0: now also U0.5 (SDA)
- net ROW1: now also U0.2 (RX)
- net ROW2: now also U0.20 (F4)
- net ROW3: now also U0.19 (F5)
- net ROW4: now also U0.6 (SCL)
- new net B+: J0.2 (Pin_2), PWR0.3 (C)
- new net GND: J0.1 (Pin_1), RST0.1 (A), U0.23 (GND), U0.3 (GND), U0.4 (GND)
- new net RAW: PWR0.2 (B), U0.24 (RAW)
- new net RST: RST0.2 (B), U0.22 (RST)
Other:
- moved on the sheet: H0, H1, H2, H3, H4, H5, H6, H7, H8
